File: boards/registers/registers.kicad_pcb (KiCad board)
At the start: 2 copper layers, 100 x 100 mm, 316 parts, among them J1 ALU, J2 CU, J3 IO, J4 5V, SW1 RESET, SW2 STEP, SW3 STEP/RUN, U1 74ACT08, U10 74ACT161, U11 74ACT244, U12 74ACT244, U13 74ACT161, U14 74ACT161, U15 74ACT244, U16 74ACT244, U17 74ACT161, U18 74ACT161, U19 74ACT244, U2 74ACT244, U20 74ACT244, U21 74ACT161, U22 74ACT161, U23 74ACT244, U24 74ACT244, U25 74AC273, U26 74ACT244, U27 74ACT244, U28 74AC273, U29 74ACT244, U3 74AC273, U30 74AC20, U31 28C256, U32 62256-TSOP, U33 74ACT02, U34 74ACT14, U4 74ACT161, U5 74ACT86, U6 74ACT08, U7 74ACT32, U8 74ACT32, U9 74ACT161

Commit message: PCB attempt
Parts:
- H1, H2, H3, H4: value MountingHole_Pad -> MountingHole; footprint MountingHole:MountingHole_3.2mm_M3_DIN965_Pad -> MountingHole:MountingHole_3.2mm_M3_DIN965
- J1, J3, R1, R100, R101, R102, R103, R104, R105, R106, R107, R108, R109, R142, R143, R144, R145, R146, R147, R148, R149, R2, R3, R4, R46, R47, R48, R49, R50, R51, R52, R53, R54, R55, R56, R57, R58, R59, R60, R61, R94, R95, R96, R97, R98, R99: moved to B.Cu
- U25, U28, U3: footprint Package_SO:SOIC-20W_7.5x12.8mm_P1.27mm -> Package_SO:TSSOP-20_4.4x6.5mm_P0.65mm
- moved H1 305.4 mm to (105.0, 55.0)
- moved R105 287.7 mm to (115.9, 87.0)
- moved R103 278.7 mm to (115.9, 93.5)
- moved R107 276.4 mm to (124.2, 93.5)
- moved R104 274.2 mm to (115.9, 90.2)
- moved R106 273.4 mm to (124.2, 96.5)
- moved R95 273.3 mm to (131.9, 93.5)
- moved R109 271.5 mm to (124.2, 87.0)
- moved R94 270.3 mm to (131.9, 96.5)
- moved R97 270.0 mm to (131.9, 87.0)
- moved R102 269.8 mm to (115.9, 96.5)
- moved R108 267.5 mm to (124.2, 90.2)
- moved R96 261.7 mm to (131.9, 90.2)
- moved H3 260.4 mm to (105.0, 145.0)
- moved R101 259.2 mm to (139.9, 87.0)
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Connections:
- H1 pad 1: GND -> (no net)
- H2 pad 1: GND -> (no net)
- H3 pad 1: GND -> (no net)
- H4 pad 1: GND -> (no net)
- J1 pad 10: /alu/a7 -> Net-(J1-Pad10)
- J1 pad 11: /alu_op0 -> Net-(J1-Pad11)
- J1 pad 12: /alu_op1 -> Net-(J1-Pad12)
- J1 pad 13: /alu_op2 -> Net-(J1-Pad13)
- J1 pad 14: /alu_op3 -> Net-(J1-Pad14)
- J1 pad 15: /flags_in0 -> Net-(J1-Pad15)
- J1 pad 16: /flags_in1 -> Net-(J1-Pad16)
- J1 pad 17: /flags_in2 -> Net-(J1-Pad17)
- J1 pad 18: /flags_in3 -> Net-(J1-Pad18)
- J1 pad 19: /di0 -> Net-(J1-Pad19)
- J1 pad 20: /di1 -> Net-(J1-Pad20)
- J1 pad 21: /di2 -> Net-(J1-Pad21)
- J1 pad 22: /di3 -> Net-(J1-Pad22)
- J1 pad 23: /di4 -> /alu_b0
- J1 pad 24: /di5 -> /alu_b4
- J1 pad 25: /di6 -> /alu_b1
- J1 pad 26: /di7 -> /alu_b5
- J1 pad 27: /~oe_alu -> /alu_b2
- J1 pad 28: /alu_invert -> /alu_b6
- J1 pad 29: /flags_out1 -> /alu_b3
- J1 pad 3: /alu/a0 -> Net-(J1-Pad3)
- J1 pad 30: Net-(J1-Pad30) -> /alu_b7
- J1 pad 31: /alu_b0 -> /alu/a0
- J1 pad 32: /alu_b1 -> /alu/a1
- J1 pad 33: /alu_b2 -> /alu/a2
- J1 pad 34: /alu_b3 -> /alu/a3
- J1 pad 35: /alu_b4 -> /alu/a4
- J1 pad 36: /alu_b5 -> /alu/a5
- J1 pad 37: /alu_b6 -> /alu/a6
- J1 pad 38: /alu_b7 -> /alu/a7
- J1 pad 4: /alu/a1 -> Net-(J1-Pad4)
- J1 pad 5: /alu/a2 -> Net-(J1-Pad5)
- J1 pad 6: /alu/a3 -> Net-(J1-Pad6)
- J1 pad 7: /alu/a4 -> Net-(J1-Pad7)
- J1 pad 8: /alu/a5 -> Net-(J1-Pad8)
- J1 pad 9: /alu/a6 -> Net-(J1-Pad9)
- J3 pad 10: /cpu_interface/a7 -> /cpu_interface/a6
- J3 pad 3: /cpu_interface/a0 -> /cpu_interface/a1
- J3 pad 4: /cpu_interface/a1 -> /cpu_interface/a0
- J3 pad 5: /cpu_interface/a2 -> /cpu_interface/a3
- J3 pad 6: /cpu_interface/a3 -> /cpu_interface/a2
- J3 pad 7: /cpu_interface/a4 -> /cpu_interface/a5
- J3 pad 8: /cpu_interface/a5 -> /cpu_interface/a4
- J3 pad 9: /cpu_interface/a6 -> /cpu_interface/a7
- U3 pad 2: /ir_out0 -> /alu_op0
- U3 pad 3: /d0 -> /d3
- U3 pad 4: /d1 -> /d2
- U3 pad 5: /ir_out1 -> /alu_invert
- U3 pad 6: /alu_invert -> /ir_out1
- U3 pad 7: /d2 -> /d1
- U3 pad 8: /d3 -> /d0
- U3 pad 9: /alu_op0 -> /ir_out0
- U32 pad 15: /cpu_interface/a2 -> /cpu_interface/a0
- U32 pad 17: /cpu_interface/a0 -> /cpu_interface/a2
- U32 pad 2: /cpu_interface/a11 -> /cpu_interface/a14
- U32 pad 3: /cpu_interface/a9 -> /cpu_interface/a13
- U32 pad 4: /cpu_interface/a8 -> /cpu_interface/a12
- U32 pad 5: /cpu_interface/a13 -> /cpu_interface/a11
- U32 pad 8: /cpu_interface/a14 -> /cpu_interface/a9
- U32 pad 9: /cpu_interface/a12 -> /cpu_interface/a8
Routing:
- net /cpu_interface/a0: track 0.00 -> 113.9 mm, vias 0 -> 3
- net /cpu_interface/a1: track 0.00 -> 108.6 mm, vias 0 -> 3
- net /cpu_interface/a2: track 0.00 -> 108.3 mm, vias 0 -> 3
- net /cpu_interface/a3: track 0.00 -> 100.5 mm, vias 0 -> 3
- net /cpu_interface/a4: track 0.00 -> 99.3 mm, vias 0 -> 3
- net /cpu_interface/a5: track 0.00 -> 92.0 mm, vias 0 -> 3
- net /alu_b7: track 0.00 -> 89.6 mm
- net /alu_b5: track 0.00 -> 88.1 mm
- net /alu_b6: track 0.00 -> 87.9 mm
- net /alu_b4: track 0.00 -> 87.8 mm
- net /cpu_interface/a6: track 0.00 -> 86.7 mm, vias 0 -> 3
- net /d3: track 0.00 -> 84.3 mm, vias 0 -> 4
- net /d7: track 0.00 -> 80.9 mm, vias 0 -> 4
- net /alu_b1: track 0.00 -> 80.4 mm
- net /alu_b2: track 0.00 -> 80.4 mm
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
Commit message: CPU registers board
Parts:
- removed C1, C12, C13, C14, C15, C16, C17, C2, C20, C21, C22, C23, C24, C25, C27, C29, C33, C5, C7, C8, C9: 0.1u, Capacitor_SMD:C_0805_2012Metric
- removed R1, R100, R101, R102, R103, R104, R105, R106, R107, R108, R109, R110, R111, R112, R113, R114, R115, R116, R117, R134, R135, R136, R137, R138, R139, R140, R141, R142, R143, R144, R145, R146, R147, R148, R149, R158, R159, R160, R161, R162, R163, R164, R165, R2, R3, R38, R39, R4, R40, R41, R42, R43, R44, R45, R46, R47, R48, R49, R5, R50, R51, R52, R53, R54, R55, R56, R57, R58, R59, R6, R60, R61, R62, R63, R64, R65, R66, R67, R68, R69, R7, R8, R86, R87, R88, R89, R90, R91, R92, R93, R94, R95, R96, R97, R98, R99: 1k, Resistor_SMD:R_0805_2012Metric
- C10, C11, C18, C26, C30, C31, C34, C35, C36, C37, C4, C6, R10, R11, R12, R126, R127, R128, R129, R13, R130, R131, R132, R133, R14, R15, R150, R151, R152, R153, R154, R155, R156, R157, R16, R166, R167, R168, R169, R17, R170, R171, R18, R19, R20, R29, R9: moved to B.Cu
- C38: footprint LED_SMD:LED_0805_2012Metric -> Capacitor_SMD:CP_Elec_4x4.5
- SW1, SW2: footprint Button_Switch_THT:SW_TH_Tactile_Omron_B3F-10xx -> Button_Switch_THT:SW_PUSH_6mm
- U11, U12, U15, U16, U19, U2, U20, U23, U24, U26, U27, U29: footprint Package_SO:SO-20_12.8x7.5mm_P1.27mm -> Package_SO:TSSOP-20_4.4x6.5mm_P0.65mm
- moved C32 198.9 mm to (102.8, 135.8), turned to 90 degrees
- moved C28 193.7 mm to (115.8, 80.5)
- moved C31 176.2 mm to (134.2, 75.1), turned to 270 degrees
- moved C30 168.1 mm to (131.2, 141.9), turned to 90 degrees
- moved R27 157.0 mm to (111.0, 95.0), turned to 180 degrees
- moved R157 156.1 mm to (157.8, 83.8)
- moved R152 154.3 mm to (157.8, 73.8)
- moved R155 153.0 mm to (157.8, 79.8)
- moved R154 152.8 mm to (157.8, 77.8)
- moved R23 152.0 mm to (110.8, 109.8), turned to 180 degrees
- moved R151 151.5 mm to (157.8, 71.8)
- moved D56 150.2 mm to (157.8, 73.8)
- moved R25 149.9 mm to (108.1, 113.5), turned to 180 degrees
- moved R26 148.9 mm to (111.0, 97.0), turned to 180 degrees
- moved D59 148.1 mm to (157.8, 79.8)
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Connections:
- C35 pad 1: Net-(C35-Pad1) -> VCC
- C35 pad 2: GND -> Net-(C35-Pad2)
- D62 pad 2: Net-(C35-Pad1) -> Net-(D62-Pad2)
- J1 pad 10: Net-(J1-Pad10) -> /alu_b7
- J1 pad 11: Net-(J1-Pad11) -> /di0
- J1 pad 12: Net-(J1-Pad12) -> /di1
- J1 pad 13: Net-(J1-Pad13) -> /di2
- J1 pad 14: Net-(J1-Pad14) -> /di3
- J1 pad 15: Net-(J1-Pad15) -> /di4
- J1 pad 16: Net-(J1-Pad16) -> /di5
- J1 pad 17: Net-(J1-Pad17) -> /di6
- J1 pad 18: Net-(J1-Pad18) -> /di7
- J1 pad 19: Net-(J1-Pad19) -> /alu/a0
- J1 pad 20: Net-(J1-Pad20) -> /alu/a1
- J1 pad 21: Net-(J1-Pad21) -> /alu/a2
- J1 pad 22: Net-(J1-Pad22) -> /alu/a3
- J1 pad 23: /alu_b0 -> /alu/a4
- J1 pad 24: /alu_b4 -> /alu/a5
- J1 pad 25: /alu_b1 -> /alu/a6
- J1 pad 26: /alu_b5 -> /alu/a7
- J1 pad 27: /alu_b2 -> /alu_op0
- J1 pad 28: /alu_b6 -> /alu_op1
- J1 pad 29: /alu_b3 -> /alu_op2
- J1 pad 3: Net-(J1-Pad3) -> /alu_b0
- J1 pad 30: /alu_b7 -> /alu_op3
- J1 pad 31: /alu/a0 -> /alu_invert
- J1 pad 32: /alu/a1 -> /~oe_alu
- J1 pad 33: /alu/a2 -> /flags_out1
- J1 pad 34: /alu/a3 -> Net-(J1-Pad34)
- J1 pad 35: /alu/a4 -> /flags_in0
- J1 pad 36: /alu/a5 -> /flags_in1
- J1 pad 37: /alu/a6 -> /flags_in2
- J1 pad 38: /alu/a7 -> /flags_in3
- J1 pad 4: Net-(J1-Pad4) -> /alu_b4
- J1 pad 5: Net-(J1-Pad5) -> /alu_b1
- J1 pad 6: Net-(J1-Pad6) -> /alu_b5
- J1 pad 7: Net-(J1-Pad7) -> /alu_b2
- J1 pad 8: Net-(J1-Pad8) -> /alu_b6
- J1 pad 9: Net-(J1-Pad9) -> /alu_b3
- J2 pad 3: /~oe -> Net-(J2-Pad3)
- J2 pad 37: Net-(J2-Pad37) -> /~oe
- J2 pad 38: Net-(J2-Pad38) -> /~we
- J2 pad 4: /~we -> Net-(J2-Pad4)
- J3 pad 10: /cpu_interface/a6 -> /d6
- J3 pad 11: /d0 -> /d5
- J3 pad 12: /d1 -> /d4
- J3 pad 13: /d2 -> /d3
- J3 pad 14: /d3 -> /d2
- J3 pad 15: /d4 -> /d1
- J3 pad 16: /d5 -> /d0
- J3 pad 17: /d6 -> /cpu_interface/a0
- J3 pad 18: /d7 -> /cpu_interface/a1
- J3 pad 19: /clk -> /cpu_interface/a2
- J3 pad 20: /cpu_interface/~io_cs -> /cpu_interface/a3
- J3 pad 21: /~oe -> /cpu_interface/a4
- J3 pad 22: /~rst -> /cpu_interface/a5
- J3 pad 23: /~we -> /cpu_interface/a6
- J3 pad 24: /cpu_interface/~io_rdy -> /cpu_interface/a7
- J3 pad 3: /cpu_interface/a1 -> /cpu_interface/~io_rdy
- J3 pad 4: /cpu_interface/a0 -> /cpu_interface/~io_cs
- J3 pad 5: /cpu_interface/a3 -> /~oe
- J3 pad 6: /cpu_interface/a2 -> /~we
- J3 pad 7: /cpu_interface/a5 -> /clk
- J3 pad 8: /cpu_interface/a4 -> /~rst
- J3 pad 9: /cpu_interface/a7 -> /d7
- R166 pad 1: GND -> Net-(C35-Pad2)
- R166 pad 2: Net-(C35-Pad1) -> VCC
- R169 pad 2: Net-(C35-Pad1) -> Net-(C35-Pad2)
- SW1 pad 1: VCC -> GND
- SW1 pad 2: Net-(C35-Pad1) -> Net-(C35-Pad2)
- SW2 pad 1: VCC -> GND
- U11 pad 12: Net-(R41-Pad2) -> /cpu_interface/a3
- U11 pad 14: Net-(R40-Pad2) -> /cpu_interface/a2
- U11 pad 16: Net-(R39-Pad2) -> /cpu_interface/a1
- U11 pad 18: Net-(R38-Pad2) -> /cpu_interface/a0
- U11 pad 3: Net-(R42-Pad2) -> /cpu_interface/a4
- U11 pad 5: Net-(R43-Pad2) -> /cpu_interface/a5
- U11 pad 7: Net-(R44-Pad2) -> /cpu_interface/a6
- U11 pad 9: Net-(R45-Pad2) -> /cpu_interface/a7
- U12 pad 12: Net-(R49-Pad2) -> /alu_b3
- U12 pad 14: Net-(R48-Pad2) -> /alu_b2
- U12 pad 16: Net-(R47-Pad2) -> /alu_b1
- U12 pad 18: Net-(R46-Pad2) -> /alu_b0
- U12 pad 3: Net-(R50-Pad2) -> /alu_b4
- U12 pad 5: Net-(R51-Pad2) -> /alu_b5
- U12 pad 7: Net-(R52-Pad2) -> /alu_b6
- U12 pad 9: Net-(R53-Pad2) -> /alu_b7
- U15 pad 12: Net-(R57-Pad2) -> /alu_b3
- U15 pad 14: Net-(R56-Pad2) -> /alu_b2
- U15 pad 16: Net-(R55-Pad2) -> /alu_b1
- U15 pad 18: Net-(R54-Pad2) -> /alu_b0
- U15 pad 3: Net-(R58-Pad2) -> /alu_b4
- U15 pad 5: Net-(R59-Pad2) -> /alu_b5
- U15 pad 7: Net-(R60-Pad2) -> /alu_b6
- U15 pad 9: Net-(R61-Pad2) -> /alu_b7
- U16 pad 12: Net-(R65-Pad2) -> /cpu_interface/a11
- U16 pad 14: Net-(R64-Pad2) -> /cpu_interface/a10
- U16 pad 16: Net-(R63-Pad2) -> /cpu_interface/a9
- U16 pad 18: Net-(R62-Pad2) -> /cpu_interface/a8
- U16 pad 3: Net-(R66-Pad2) -> /cpu_interface/a12
- U16 pad 5: Net-(R67-Pad2) -> /cpu_interface/a13
- U16 pad 7: Net-(R68-Pad2) -> /cpu_interface/a14
- U16 pad 9: Net-(R69-Pad2) -> /cpu_interface/a15
- U19 pad 12: Net-(R89-Pad2) -> /cpu_interface/a3
- U19 pad 14: Net-(R88-Pad2) -> /cpu_interface/a2
- U19 pad 16: Net-(R87-Pad2) -> /cpu_interface/a1
- U19 pad 18: Net-(R86-Pad2) -> /cpu_interface/a0
- U19 pad 3: Net-(R90-Pad2) -> /cpu_interface/a4
- U19 pad 5: Net-(R91-Pad2) -> /cpu_interface/a5
- U19 pad 7: Net-(R92-Pad2) -> /cpu_interface/a6
- U19 pad 9: Net-(R93-Pad2) -> /cpu_interface/a7
- U2 pad 12: Net-(R4-Pad2) -> /di3
- U2 pad 14: Net-(R3-Pad2) -> /di2
- U2 pad 16: Net-(R2-Pad2) -> /di1
- U2 pad 18: Net-(R1-Pad2) -> /di0
- U2 pad 3: Net-(R5-Pad2) -> /di4
- U2 pad 5: Net-(R6-Pad2) -> /di5
- U2 pad 7: Net-(R7-Pad2) -> /di6
- U2 pad 9: Net-(R8-Pad2) -> /di7
- U20 pad 12: Net-(R97-Pad2) -> /alu_b3
- U20 pad 14: Net-(R96-Pad2) -> /alu_b2
- U20 pad 16: Net-(R95-Pad2) -> /alu_b1
- U20 pad 18: Net-(R94-Pad2) -> /alu_b0
- U20 pad 3: Net-(R98-Pad2) -> /alu_b4
- U20 pad 5: Net-(R99-Pad2) -> /alu_b5
- U20 pad 7: Net-(R100-Pad2) -> /alu_b6
- U20 pad 9: Net-(R101-Pad2) -> /alu_b7
- U23 pad 12: Net-(R105-Pad2) -> /alu_b3
- U23 pad 14: Net-(R104-Pad2) -> /alu_b2
- U23 pad 16: Net-(R103-Pad2) -> /alu_b1
- U23 pad 18: Net-(R102-Pad2) -> /alu_b0
- U23 pad 3: Net-(R106-Pad2) -> /alu_b4
- U23 pad 5: Net-(R107-Pad2) -> /alu_b5
- U23 pad 7: Net-(R108-Pad2) -> /alu_b6
- U23 pad 9: Net-(R109-Pad2) -> /alu_b7
- U24 pad 12: Net-(R113-Pad2) -> /cpu_interface/a11
- U24 pad 14: Net-(R112-Pad2) -> /cpu_interface/a10
- U24 pad 16: Net-(R111-Pad2) -> /cpu_interface/a9
- U24 pad 18: Net-(R110-Pad2) -> /cpu_interface/a8
- U24 pad 3: Net-(R114-Pad2) -> /cpu_interface/a12
- U24 pad 5: Net-(R115-Pad2) -> /cpu_interface/a13
- U24 pad 7: Net-(R116-Pad2) -> /cpu_interface/a14
- U24 pad 9: Net-(R117-Pad2) -> /cpu_interface/a15
- U25 pad 12: /gp_reg_b/d4 -> /gp_reg_b/d7
- U25 pad 13: /di4 -> /di7
- U25 pad 14: /di5 -> /di6
- U25 pad 15: /gp_reg_b/d5 -> /gp_reg_b/d6
- U25 pad 16: /gp_reg_b/d6 -> /gp_reg_b/d5
- U25 pad 17: /di6 -> /di5
- U25 pad 18: /di7 -> /di4
- U25 pad 19: /gp_reg_b/d7 -> /gp_reg_b/d4
- U26 pad 12: Net-(R137-Pad2) -> /d3
- U26 pad 14: Net-(R136-Pad2) -> /d2
- U26 pad 16: Net-(R135-Pad2) -> /d1
- U26 pad 18: Net-(R134-Pad2) -> /d0
- U26 pad 3: Net-(R138-Pad2) -> /d4
- U26 pad 5: Net-(R139-Pad2) -> /d5
- U26 pad 7: Net-(R140-Pad2) -> /d6
- U26 pad 9: Net-(R141-Pad2) -> /d7
- U27 pad 12: Net-(R145-Pad2) -> /alu_b3
- U27 pad 14: Net-(R144-Pad2) -> /alu_b2
- U27 pad 16: Net-(R143-Pad2) -> /alu_b1
- U27 pad 18: Net-(R142-Pad2) -> /alu_b0
- U27 pad 3: Net-(R146-Pad2) -> /alu_b4
- U27 pad 5: Net-(R147-Pad2) -> /alu_b5
- U27 pad 7: Net-(R148-Pad2) -> /alu_b6
- U27 pad 9: Net-(R149-Pad2) -> /alu_b7
- U29 pad 12: Net-(R161-Pad2) -> /d3
- U29 pad 14: Net-(R160-Pad2) -> /d2
- U29 pad 16: Net-(R159-Pad2) -> /d1
- U29 pad 18: Net-(R158-Pad2) -> /d0
- U29 pad 3: Net-(R162-Pad2) -> /d4
- U29 pad 5: Net-(R163-Pad2) -> /d5
- U29 pad 7: Net-(R164-Pad2) -> /d6
- U29 pad 9: Net-(R165-Pad2) -> /d7
- U32 pad 18: /d0 -> /d7
- U32 pad 19: /d1 -> /d6
- U32 pad 20: /d2 -> /d5
- U32 pad 22: /d3 -> /d4
- U32 pad 23: /d4 -> /d3
- U32 pad 24: /d5 -> /d2
- U32 pad 25: /d6 -> /d1
- U32 pad 26: /d7 -> /d0
- U34 pad 12: Net-(U34-Pad12) -> /~rst
- U34 pad 13: GND -> Net-(D62-Pad2)
- U34 pad 8: /~rst -> Net-(D62-Pad2)
Routing:
- net GND: track 0.00 -> 1207.4 mm, vias 0 -> 79
- net VCC: track 0.00 -> 755.2 mm, vias 0 -> 62
- net /~rst: track 0.00 -> 352.1 mm, vias 0 -> 16
- net /~clk: track 0.00 -> 241.8 mm, vias 0 -> 14
- net /di7: track 0.00 -> 210.5 mm, vias 0 -> 8
- net /di5: track 0.00 -> 205.3 mm, vias 0 -> 8
- net /di6: track 0.00 -> 204.7 mm, vias 0 -> 8
- net /di3: track 0.00 -> 200.0 mm, vias 0 -> 8
- net /di4: track 0.00 -> 196.9 mm, vias 0 -> 8
- net /di2: track 0.00 -> 193.4 mm, vias 0 -> 8
- net /di1: track 0.00 -> 193.1 mm, vias 0 -> 8
- net /di0: track 0.00 -> 187.8 mm, vias 0 -> 8
- net /alu_invert: track 0.00 -> 183.7 mm, vias 0 -> 2
- net /pointer_pair/reg_a/~oe_dl: track 0.00 -> 182.9 mm, vias 0 -> 5
- net /pointer_pair/reg_a/cnt: track 0.00 -> 177.9 mm, vias 0 -> 7
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- added copper zone on B.Cu, net GND
- added copper zone on F.Cu, net VCC
Other:
- net class Power: trace_width 0.4 -> 0.22; via_dia 0.8 -> 0.6; via_drill 0.5 -> 0.4
- board text added: "0"
- board text added: "15"
- board text added: "7"
- board text added: "A"
- board text added: "B"
- board text added: "C"
- board text added: "IR"
- board text added: "O"
- board text added: "P0"
- board text added: "P1"
- board text added: "RESET"
- board text added: "S"
- board text added: "STEP"
- board text added: "Z"

Commit message: Fixed some footprints
Parts:
- C37: footprint LED_SMD:LED_0805_2012Metric -> Capacitor_SMD:C_0805_2012Metric
Routing:
- net GND: track 1207.4 -> 1206.2 mm
- net /alu_op0: track 165.6 -> 164.9 mm
