File: boards/registers/registers.kicad_pcb (KiCad board)
At the start: 2 copper layers, 100 x 100 mm, 192 parts, among them J1 SSW-120-02-G-D-RA, J2 SSW-120-02-G-D-RA, J4 5V, J5 SSW-120-02-G-D-RA, SW1 RESET, SW2 STEP, SW3 OS102011MS2QN1, U1 SN74ACT08PW, U10 MC74ACT161DG, U11 SN74ACT244PW, U12 SN74ACT244PW, U13 MC74ACT161DG, U14 MC74ACT161DG, U15 SN74ACT244PW, U16 SN74ACT244PW, U17 MC74ACT161DG, U18 MC74ACT161DG, U19 SN74ACT244PW, U2 SN74ACT244PW, U20 SN74ACT244PW, U21 MC74ACT161DG, U22 MC74ACT161DG, U23 SN74ACT244PW, U24 SN74ACT244PW, U25 MC74AC273DTR2G, U26 SN74ACT244PW, U27 SN74ACT244PW, U28 MC74AC273DTR2G, U29 SN74ACT244PW, U3 MC74AC273DTR2G, U34 74ACT14MTCX, U4 MC74ACT161DG, U5 MC74ACT86DG, U6 SN74ACT08PW, U7 SN74ACT32PWR, U8 SN74ACT32PWR, U9 MC74ACT161DG

Commit message: Power supply plus sign
Other:
- board text added: "+"
Changed lines of the file:
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@@
   (general
     (thickness 1.6)
-    (drawings 28)
+    (drawings 29)
     (tracks 5700)
     (zones 0)
@@
     )
   )
+  (gr_text + (at 178.9 59.2) (layer F.SilkS)
+    (effects (font (size 1 1) (thickness 0.15)))
+  )
   (gr_text "P sel" (at 178.5 105) (layer F.SilkS)
