File: boards/registers/cpu_interface.sch (KiCad schematic (older format))
At the start: 1 part, among them J5 CU

Commit message: Part names
Parts:
- J5: value CU -> SSW-120-02-G-D-RA
Changed lines of the file:
@@
 AR Path="/5EC337E5/6056FC88" Ref="J5"  Part="1"
 F 0 "J5" H 5900 3517 50  0000 C CNN
-F 1 "CU" H 5900 3426 50  0000 C CNN
+F 1 "SSW-120-02-G-D-RA" H 5900 3426 50  0000 C CNN
 F 2 "Connector_PinSocket_2.54mm:PinSocket_2x20_P2.54mm_Horizontal" H 5850 2400 50  0001 C CNN
 F 3 "~" H 5850 2400 50  0001 C CNN

Commit message: Registers: new clock and reset
Connections:
- net labels added: rdy
- net labels removed: ~rdy
Changed lines of the file:
@@
 Sheet 9 10
 Title "CPU interface"
-Date "2020-01-27"
+Date "2021-01-18"
 Rev "2"
 Comp ""
@@
 ~we
 Text HLabel 1500 1900 0    50   Output ~ 0
-~rdy
+rdy
 Text HLabel 1500 2000 0    50   Input ~ 0
 clk
@@
 ~rst
 Text Label 1850 1900 2    50   ~ 0
-~rdy
+rdy
 Wire Bus Line
 	2800 1200 1500 1200
@@
 ~we
 Text Label 5650 1700 2    50   ~ 0
-~rdy
+rdy
 Text Label 5650 1600 2    50   ~ 0
 clk

Commit message: Registers board rev. 2
Implement RDY mechanism by suspending clock signal
Take caution against crosstalk on sensitive line
Add proper decoupling capacitors
Connections:
- no-connect marks 7 -> 8
Changed lines of the file:
@@
 Text Label 5650 1700 2    50   ~ 0
 rdy
-Text Label 5650 1600 2    50   ~ 0
-clk
 Text Label 6150 1600 0    50   ~ 0
 ~rst
@@
 NoConn ~ 5650 1900
 NoConn ~ 6150 1700
+NoConn ~ 5650 1600
 Wire Bus Line
 	4500 1300 4500 2350
