File: boards/registers/gp_reg.sch (KiCad schematic (older format))
At the start: 38 parts, among them U25 74AC273, U26 74ACT244, U27 74ACT244

Commit message: PCB attempt
Parts:
- U25: footprint Package_SO:SOIC-20W_7.5x12.8mm_P1.27mm -> Package_SO:TSSOP-20_4.4x6.5mm_P0.65mm
Changed lines of the file:
@@
 F 0 "U25" H 4700 1100 50  0000 C CNN
 F 1 "74AC273" H 4650 1000 50  0000 C CNN
-F 2 "Package_SO:SOIC-20W_7.5x12.8mm_P1.27mm" H 4300 1650 50  0001 C CNN
+F 2 "Package_SO:TSSOP-20_4.4x6.5mm_P0.65mm" H 4300 1650 50  0001 C CNN
 F 3 "https://assets.nexperia.com/documents/data-sheet/74HC_HCT273.pdf" H 4300 1650 50  0001 C CNN
 	1    4300 1650

Commit message: CPU registers board
Parts:
- removed C25, C27: 0.1u, Capacitor_SMD:C_0805_2012Metric, symbol Device:C
- removed R134, R135, R136, R137, R138, R139, R140, R141, R142, R143, R144, R145, R146, R147, R148, R149: 1k, Resistor_SMD:R_0805_2012Metric, symbol Device:R
- U26, U27: footprint Package_SO:SO-20_12.8x7.5mm_P1.27mm -> Package_SO:TSSOP-20_4.4x6.5mm_P0.65mm
Connections:
- net d4: now also U25.19 (Q7); no longer U25.12 (Q4)
- net d5: now also U25.16 (Q6); no longer U25.15 (Q5)
- net d6: now also U25.15 (Q5); no longer U25.16 (Q6)
- net d7: now also U25.12 (Q4); no longer U25.19 (Q7)
- net di4: now also U25.18 (D7); no longer U25.13 (D4)
- net di5: now also U25.17 (D6); no longer U25.14 (D5)
- net di6: now also U25.14 (D5); no longer U25.17 (D6)
- net di7: now also U25.13 (D4); no longer U25.18 (D7)
- net doa0: now also U26.18 (1Y0)
- net doa1: now also U26.16 (1Y1)
- net doa2: now also U26.14 (1Y2)
- net doa3: now also U26.12 (1Y3)
- net doa4: now also U26.3 (2Y0)
- net doa5: now also U26.5 (2Y1)
- net doa6: now also U26.7 (2Y2)
- net doa7: now also U26.9 (2Y3)
- net dob0: now also U27.18 (1Y0)
- net dob1: now also U27.16 (1Y1)
- net dob2: now also U27.14 (1Y2)
- net dob3: now also U27.12 (1Y3)
- net dob4: now also U27.3 (2Y0)
- net dob5: now also U27.5 (2Y1)
- net dob6: now also U27.7 (2Y2)
- net dob7: now also U27.9 (2Y3)

Commit message: LEDs and LED resistors
Parts:
- D46, D47, D48, D49, D50, D51, D52, D53: value LED -> KP-2012EC
- R126, R127, R128, R129, R130, R131, R132, R133: value LED -> 620
Changed lines of the file:
@@
 AR Path="/5E7CA397/5E7690D3" Ref="D46"  Part="1"
 F 0 "D46" H 3700 3250 50  0000 C CNN
-F 1 "LED" H 4643 3375 50  0001 C CNN
+F 1 "KP-2012EC" H 4643 3375 50  0001 C CNN
 F 2 "LED_SMD:LED_0805_2012Metric" H 4650 3250 50  0001 C CNN
 F 3 "~" H 4650 3250 50  0001 C CNN
@@
 AR Path="/5E7CA397/5E769EED" Ref="R126"  Part="1"
 F 0 "R126" V 4350 2050 50  0000 C CNN
-F 1 "LED" V 4350 2400 50  0000 C CNN
+F 1 "620" V 4350 2400 50  0000 C CNN
 F 2 "Resistor_SMD:R_0805_2012Metric" V 4280 3250 50  0001 C CNN
 F 3 "~" H 4350 3250 50  0001 C CNN
@@
 AR Path="/5E7CA397/5E76BFE9" Ref="D47"  Part="1"
 F 0 "D47" H 3700 3350 50  0000 C CNN
-F 1 "LED" H 4643 3475 50  0001 C CNN
+F 1 "KP-2012EC" H 4643 3475 50  0001 C CNN
 F 2 "LED_SMD:LED_0805_2012Metric" H 4650 3350 50  0001 C CNN
 F 3 "~" H 4650 3350 50  0001 C CNN
@@
 AR Path="/5E7CA397/5E76BFEF" Ref="R127"  Part="1"
 F 0 "R127" V 4350 2150 50  0000 C CNN
-F 1 "LED" V 4350 2500 50  0000 C CNN
+F 1 "620" V 4350 2500 50  0000 C CNN
 F 2 "Resistor_SMD:R_0805_2012Metric" V 4280 3350 50  0001 C CNN
 F 3 "~" H 4350 3350 50  0001 C CNN
@@
 AR Path="/5E7CA397/5E76E132" Ref="D48"  Part="1"
 F 0 "D48" H 3700 3450 50  0000 C CNN
-F 1 "LED" H 4643 3575 50  0001 C CNN
+F 1 "KP-2012EC" H 4643 3575 50  0001 C CNN
 F 2 "LED_SMD:LED_0805_2012Metric" H 4650 3450 50  0001 C CNN
 F 3 "~" H 4650 3450 50  0001 C CNN
@@
 AR Path="/5E7CA397/5E76E138" Ref="R128"  Part="1"
 F 0 "R128" V 4350 2250 50  0000 C CNN
-F 1 "LED" V 4350 2600 50  0000 C CNN
+F 1 "620" V 4350 2600 50  0000 C CNN
 F 2 "Resistor_SMD:R_0805_2012Metric" V 4280 3450 50  0001 C CNN
 F 3 "~" H 4350 3450 50  0001 C CNN
@@
 AR Path="/5E7CA397/5E76FA9B" Ref="D49"  Part="1"
 F 0 "D49" H 3700 3550 50  0000 C CNN
-F 1 "LED" H 4643 3675 50  0001 C CNN
+F 1 "KP-2012EC" H 4643 3675 50  0001 C CNN
 F 2 "LED_SMD:LED_0805_2012Metric" H 4650 3550 50  0001 C CNN
 F 3 "~" H 4650 3550 50  0001 C CNN
@@
 AR Path="/5E7CA397/5E76FAA1" Ref="R129"  Part="1"
 F 0 "R129" V 4350 2350 50  0000 C CNN
-F 1 "LED" V 4350 2700 50  0000 C CNN
+F 1 "620" V 4350 2700 50  0000 C CNN
 F 2 "Resistor_SMD:R_0805_2012Metric" V 4280 3550 50  0001 C CNN
 F 3 "~" H 4350 3550 50  0001 C CNN
@@
 AR Path="/5E7CA397/5E771404" Ref="D50"  Part="1"
 F 0 "D50" H 3700 3650 50  0000 C CNN
-F 1 "LED" H 4643 3775 50  0001 C CNN
+F 1 "KP-2012EC" H 4643 3775 50  0001 C CNN
 F 2 "LED_SMD:LED_0805_2012Metric" H 4650 3650 50  0001 C CNN
 F 3 "~" H 4650 3650 50  0001 C CNN
@@
 AR Path="/5E7CA397/5E77140A" Ref="R130"  Part="1"
 F 0 "R130" V 4350 2450 50  0000 C CNN
-F 1 "LED" V 4350 2800 50  0000 C CNN
+F 1 "620" V 4350 2800 50  0000 C CNN
 F 2 "Resistor_SMD:R_0805_2012Metric" V 4280 3650 50  0001 C CNN
 F 3 "~" H 4350 3650 50  0001 C CNN
@@
 AR Path="/5E7CA397/5E772D6D" Ref="D51"  Part="1"
 F 0 "D51" H 3700 3750 50  0000 C CNN
-F 1 "LED" H 4643 3875 50  0001 C CNN
+F 1 "KP-2012EC" H 4643 3875 50  0001 C CNN
 F 2 "LED_SMD:LED_0805_2012Metric" H 4650 3750 50  0001 C CNN
 F 3 "~" H 4650 3750 50  0001 C CNN
@@
 AR Path="/5E7CA397/5E772D73" Ref="R131"  Part="1"
 F 0 "R131" V 4350 2550 50  0000 C CNN
-F 1 "LED" V 4350 2900 50  0000 C CNN
+F 1 "620" V 4350 2900 50  0000 C CNN
 F 2 "Resistor_SMD:R_0805_2012Metric" V 4280 3750 50  0001 C CNN
 F 3 "~" H 4350 3750 50  0001 C CNN
@@
 AR Path="/5E7CA397/5E7746D6" Ref="D52"  Part="1"
 F 0 "D52" H 3700 3850 50  0000 C CNN
-F 1 "LED" H 4643 3975 50  0001 C CNN
+F 1 "KP-2012EC" H 4643 3975 50  0001 C CNN
 F 2 "LED_SMD:LED_0805_2012Metric" H 4650 3850 50  0001 C CNN
 F 3 "~" H 4650 3850 50  0001 C CNN
@@
 AR Path="/5E7CA397/5E7746DC" Ref="R132"  Part="1"
 F 0 "R132" V 4350 2650 50  0000 C CNN
-F 1 "LED" V 4350 3000 50  0000 C CNN
+F 1 "620" V 4350 3000 50  0000 C CNN
 F 2 "Resistor_SMD:R_0805_2012Metric" V 4280 3850 50  0001 C CNN
 F 3 "~" H 4350 3850 50  0001 C CNN
@@
 AR Path="/5E7CA397/5E7762B5" Ref="D53"  Part="1"
 F 0 "D53" H 3700 3950 50  0000 C CNN
-F 1 "LED" H 4643 4075 50  0001 C CNN
+F 1 "KP-2012EC" H 4643 4075 50  0001 C CNN
 F 2 "LED_SMD:LED_0805_2012Metric" H 4650 3950 50  0001 C CNN
 F 3 "~" H 4650 3950 50  0001 C CNN
@@
 AR Path="/5E7CA397/5E7762BB" Ref="R133"  Part="1"
 F 0 "R133" V 4350 2750 50  0000 C CNN
-F 1 "LED" V 4350 3100 50  0000 C CNN
+F 1 "620" V 4350 3100 50  0000 C CNN
 F 2 "Resistor_SMD:R_0805_2012Metric" V 4280 3950 50  0001 C CNN
 F 3 "~" H 4350 3950 50  0001 C CNN

Commit message: Part names
Parts:
- U25: value 74AC273 -> MC74AC273DTR2G
- U26, U27: value 74ACT244 -> SN74ACT244PW
Changed lines of the file:
@@
 AR Path="/5E7CA397/5E73BC4E" Ref="U26"  Part="1"
 F 0 "U26" H 7200 1100 50  0000 C CNN
-F 1 "74ACT244" H 7100 1000 50  0000 C CNN
+F 1 "SN74ACT244PW" H 7100 1000 50  0000 C CNN
 F 2 "Package_SO:TSSOP-20_4.4x6.5mm_P0.65mm" H 6800 1650 50  0001 C CNN
 F 3 "https://assets.nexperia.com/documents/data-sheet/74HC_HCT244.pdf" H 6800 1650 50  0001 C CNN
@@
 AR Path="/5E7CA397/5E74CA38" Ref="U27"  Part="1"
 F 0 "U27" H 7200 3300 50  0000 C CNN
-F 1 "74ACT244" H 7100 3200 50  0000 C CNN
+F 1 "SN74ACT244PW" H 7100 3200 50  0000 C CNN
 F 2 "Package_SO:TSSOP-20_4.4x6.5mm_P0.65mm" H 6800 3850 50  0001 C CNN
 F 3 "https://assets.nexperia.com/documents/data-sheet/74HC_HCT244.pdf" H 6800 3850 50  0001 C CNN
@@
 AR Path="/5E7CA397/5E755BB1" Ref="U25"  Part="1"
 F 0 "U25" H 4700 1100 50  0000 C CNN
-F 1 "74AC273" H 4650 1000 50  0000 C CNN
+F 1 "MC74AC273DTR2G" H 4650 1000 50  0000 C CNN
 F 2 "Package_SO:TSSOP-20_4.4x6.5mm_P0.65mm" H 4300 1650 50  0001 C CNN
 F 3 "https://assets.nexperia.com/documents/data-sheet/74HC_HCT273.pdf" H 4300 1650 50  0001 C CNN

Commit message: Registers: more decoupling capacitors
Parts:
- added C29, C30: 0.1u, Capacitor_SMD:C_0805_2012Metric, symbol Device:C
Connections:
- net GND: now also C29.2, C30.2
- net VCC: now also C29.1, C30.1
Changed lines of the file:
@@
 Text Label 3600 1650 0    50   ~ 0
 di6
+$Comp
+L Device:C C?
+U 1 1 60138FE9
+P 7700 2350
+AR Path="/60138FE9" Ref="C?"  Part="1"
+AR Path="/5E7CA397/60138FE9" Ref="C30"  Part="1"
+F 0 "C30" H 7815 2396 50  0000 L CNN
+F 1 "0.1u" H 7815 2305 50  0000 L CNN
+F 2 "Capacitor_SMD:C_0805_2012Metric" H 7738 2200 50  0001 C CNN
+F 3 "~" H 7700 2350 50  0001 C CNN
+	1    7700 2350
+	1    0    0    -1
+$EndComp
+$Comp
+L power:VCC #PWR?
+U 1 1 60138FEF
+P 7700 2200
+AR Path="/60138FEF" Ref="#PWR?"  Part="1"
+AR Path="/5E7CA397/60138FEF" Ref="#PWR0222"  Part="1"
+F 0 "#PWR0222" H 7700 2050 50  0001 C CNN
+F 1 "VCC" H 7717 2373 50  0000 C CNN
+F 2 "" H 7700 2200 50  0001 C CNN
+F 3 "" H 7700 2200 50  0001 C CNN
+	1    7700 2200
+	1    0    0    -1
+$EndComp
+$Comp
+L power:GND #PWR?
+U 1 1 60138FF5
+P 7700 2500
+AR Path="/60138FF5" Ref="#PWR?"  Part="1"
+AR Path="/5E7CA397/60138FF5" Ref="#PWR0224"  Part="1"
+F 0 "#PWR0224" H 7700 2250 50  0001 C CNN
+F 1 "GND" H 7705 2327 50  0000 C CNN
+F 2 "" H 7700 2500 50  0001 C CNN
+F 3 "" H 7700 2500 50  0001 C CNN
+	1    7700 2500
+	1    0    0    -1
+$EndComp
+$Comp
+L Device:C C?
+U 1 1 6013E427
+P 5350 2150
+AR Path="/6013E427" Ref="C?"  Part="1"
+AR Path="/5E7CA397/6013E427" Ref="C29"  Part="1"
+F 0 "C29" H 5465 2196 50  0000 L CNN
+F 1 "0.1u" H 5465 2105 50  0000 L CNN
+F 2 "Capacitor_SMD:C_0805_2012Metric" H 5388 2000 50  0001 C CNN
+F 3 "~" H 5350 2150 50  0001 C CNN
+	1    5350 2150
+	1    0    0    -1
+$EndComp
+$Comp
+L power:VCC #PWR?
+U 1 1 6013E42D
+P 5350 2000
+AR Path="/6013E42D" Ref="#PWR?"  Part="1"
+AR Path="/5E7CA397/6013E42D" Ref="#PWR0218"  Part="1"
+F 0 "#PWR0218" H 5350 1850 50  0001 C CNN
+F 1 "VCC" H 5367 2173 50  0000 C CNN
+F 2 "" H 5350 2000 50  0001 C CNN
+F 3 "" H 5350 2000 50  0001 C CNN
+	1    5350 2000
+	1    0    0    -1
+$EndComp
+$Comp
+L power:GND #PWR?
+U 1 1 6013E433
+P 5350 2300
+AR Path="/6013E433" Ref="#PWR?"  Part="1"
+AR Path="/5E7CA397/6013E433" Ref="#PWR0219"  Part="1"
+F 0 "#PWR0219" H 5350 2050 50  0001 C CNN
+F 1 "GND" H 5355 2127 50  0000 C CNN
+F 2 "" H 5350 2300 50  0001 C CNN
+F 3 "" H 5350 2300 50  0001 C CNN
+	1    5350 2300
+	1    0    0    -1
+$EndComp
 Wire Bus Line
 	8000 3100 8000 3950

Commit message: Registers: change logic family to HC and LV-A
Parts:
- U25: value MC74AC273DTR2G -> MC74HC273ADT
- U26, U27: value SN74ACT244PW -> MC74HC244ADT
Changed lines of the file:
@@
 AR Path="/5E7CA397/5E73BC4E" Ref="U26"  Part="1"
 F 0 "U26" H 7200 1100 50  0000 C CNN
-F 1 "SN74ACT244PW" H 7100 1000 50  0000 C CNN
+F 1 "MC74HC244ADT" H 7100 1000 50  0000 C CNN
 F 2 "Package_SO:TSSOP-20_4.4x6.5mm_P0.65mm" H 6800 1650 50  0001 C CNN
-F 3 "https://assets.nexperia.com/documents/data-sheet/74HC_HCT244.pdf" H 6800 1650 50  0001 C CNN
+F 3 "http://www.farnell.com/datasheets/1878565.pdf" H 6800 1650 50  0001 C CNN
 	1    6800 1650
 	1    0    0    -1
@@
 AR Path="/5E7CA397/5E74CA38" Ref="U27"  Part="1"
 F 0 "U27" H 7200 3300 50  0000 C CNN
-F 1 "SN74ACT244PW" H 7100 3200 50  0000 C CNN
+F 1 "MC74HC244ADT" H 7100 3200 50  0000 C CNN
 F 2 "Package_SO:TSSOP-20_4.4x6.5mm_P0.65mm" H 6800 3850 50  0001 C CNN
-F 3 "https://assets.nexperia.com/documents/data-sheet/74HC_HCT244.pdf" H 6800 3850 50  0001 C CNN
+F 3 "http://www.farnell.com/datasheets/1878565.pdf" H 6800 3850 50  0001 C CNN
 	1    6800 3850
 	1    0    0    -1
@@
 AR Path="/5E7CA397/5E755BB1" Ref="U25"  Part="1"
 F 0 "U25" H 4700 1100 50  0000 C CNN
-F 1 "MC74AC273DTR2G" H 4650 1000 50  0000 C CNN
+F 1 "MC74HC273ADT" H 4650 1000 50  0000 C CNN
 F 2 "Package_SO:TSSOP-20_4.4x6.5mm_P0.65mm" H 4300 1650 50  0001 C CNN
-F 3 "https://assets.nexperia.com/documents/data-sheet/74HC_HCT273.pdf" H 4300 1650 50  0001 C CNN
+F 3 "http://www.farnell.com/datasheets/1878567.pdf" H 4300 1650 50  0001 C CNN
 	1    4300 1650
 	1    0    0    -1

Commit message: Registers board rev. 2
Implement RDY mechanism by suspending clock signal
Take caution against crosstalk on sensitive line
Add proper decoupling capacitors
Connections:
- net d0: now also U27.17 (2A0); no longer U27.2 (1A0)
- net d1: now also U27.15 (2A1); no longer U27.4 (1A1)
- net d2: now also U27.13 (2A2); no longer U27.6 (1A2)
- net d3: now also U27.11 (2A3); no longer U27.8 (1A3)
- net d4: now also U27.2 (1A0); no longer U27.17 (2A0)
- net d5: now also U27.4 (1A1); no longer U27.15 (2A1)
- net d6: now also U27.6 (1A2); no longer U27.13 (2A2)
- net d7: now also U27.8 (1A3); no longer U27.11 (2A3)
- net dob0: now also U27.3 (2Y0); no longer U27.18 (1Y0)
- net dob1: now also U27.5 (2Y1); no longer U27.16 (1Y1)
- net dob2: now also U27.7 (2Y2); no longer U27.14 (1Y2)
- net dob3: now also U27.9 (2Y3); no longer U27.12 (1Y3)
- net dob4: now also U27.18 (1Y0); no longer U27.3 (2Y0)
- net dob5: now also U27.16 (1Y1); no longer U27.5 (2Y1)
- net dob6: now also U27.14 (1Y2); no longer U27.7 (2Y2)
- net dob7: now also U27.12 (1Y3); no longer U27.9 (2Y3)
Changed lines of the file:
@@
 	5950 4150 6050 4050
 Wire Wire Line
+	6050 3650 6300 3650
+Wire Wire Line
+	6300 3550 6050 3550
+Wire Wire Line
+	6050 3450 6300 3450
+Wire Wire Line
+	6300 3350 6050 3350
+Wire Wire Line
 	6050 4050 6300 4050
 Wire Wire Line
@@
 Wire Wire Line
 	6300 3750 6050 3750
-Wire Wire Line
-	6050 3650 6300 3650
-Wire Wire Line
-	6300 3550 6050 3550
-Wire Wire Line
-	6050 3450 6300 3450
-Wire Wire Line
-	6300 3350 6050 3350
 Entry Wire Line
 	7900 3350 8000 3250
@@
 Entry Wire Line
 	7900 4050 8000 3950
+Text Label 6050 3750 0    50   ~ 0
+d0
+Text Label 6050 3850 0    50   ~ 0
+d1
+Text Label 6050 3950 0    50   ~ 0
+d2
+Text Label 6050 4050 0    50   ~ 0
+d3
 Text Label 6050 3350 0    50   ~ 0
-d0
+d4
 Text Label 6050 3450 0    50   ~ 0
-d1
+d5
 Text Label 6050 3550 0    50   ~ 0
-d2
+d6
 Text Label 6050 3650 0    50   ~ 0
-d3
-Text Label 6050 3750 0    50   ~ 0
-d4
-Text Label 6050 3850 0    50   ~ 0
-d5
-Text Label 6050 3950 0    50   ~ 0
-d6
-Text Label 6050 4050 0    50   ~ 0
 d7
 $Comp
@@
 Text Label 7650 1850 0    50   ~ 0
 doa7
+Text Label 7650 3750 0    50   ~ 0
+dob0
+Text Label 7650 3850 0    50   ~ 0
+dob1
+Text Label 7650 3950 0    50   ~ 0
+dob2
+Text Label 7650 4050 0    50   ~ 0
+dob3
 Text Label 7650 3350 0    50   ~ 0
-dob0
+dob4
 Text Label 7650 3450 0    50   ~ 0
-dob1
+dob5
 Text Label 7650 3550 0    50   ~ 0
-dob2
+dob6
 Text Label 7650 3650 0    50   ~ 0
-dob3
-Text Label 7650 3750 0    50   ~ 0
-dob4
-Text Label 7650 3850 0    50   ~ 0
-dob5
-Text Label 7650 3950 0    50   ~ 0
-dob6
-Text Label 7650 4050 0    50   ~ 0
 dob7
 Wire Bus Line
@@
 	7300 1850 7900 1850
 Wire Wire Line
+	7300 3750 7900 3750
+Wire Wire Line
+	7300 3850 7900 3850
+Wire Wire Line
+	7300 3950 7900 3950
+Wire Wire Line
+	7300 4050 7900 4050
+Wire Wire Line
 	7300 3350 7900 3350
 Wire Wire Line
@@
 Wire Wire Line
 	7300 3650 7900 3650
-Wire Wire Line
-	7300 3750 7900 3750
-Wire Wire Line
-	7300 3850 7900 3850
-Wire Wire Line
-	7300 3950 7900 3950
-Wire Wire Line
-	7300 4050 7900 4050
 Text Label 3600 1650 0    50   ~ 0
 di6
