File: boards/registers/pwr_and_clk.sch (KiCad schematic (older format))
At the start: 21 parts, among them SW1 RESET, SW2 STEP, SW3 OS102011MS2QN1, U30 74LS74, U31 74AHC1G86, U34 74ACT14MTCX

Commit message: Registers: change logic family to HC and LV-A
Parts:
- U30: value 74LS74 -> 74HC74PW; footprint (none) -> Package_SO:TSSOP-14_4.4x5mm_P0.65mm
- U31: value 74AHC1G86 -> SN74AHC1G86DBVR; footprint (none) -> Package_TO_SOT_SMD:SOT-23-5
- U34: value 74ACT14MTCX -> SN74LV14APW
Changed lines of the file:
@@
 P 3550 1750
 F 0 "U34" H 3550 2067 50  0000 C CNN
-F 1 "74ACT14MTCX" H 3550 1976 50  0000 C CNN
+F 1 "SN74LV14APW" H 3550 1976 50  0000 C CNN
 F 2 "Package_SO:TSSOP-14_4.4x5mm_P0.65mm" H 3550 1750 50  0001 C CNN
-F 3 "http://www.ti.com/lit/gpn/sn74HC14" H 3550 1750 50  0001 C CNN
+F 3 "https://www.ti.com/lit/ds/symlink/sn74lv14a.pdf" H 3550 1750 50  0001 C CNN
 	1    3550 1750
 	1    0    0    -1
@@
 P 3550 3000
 F 0 "U34" H 3550 3317 50  0000 C CNN
-F 1 "74ACT14MTCX" H 3550 3226 50  0000 C CNN
+F 1 "SN74LV14APW" H 3550 3226 50  0000 C CNN
 F 2 "Package_SO:TSSOP-14_4.4x5mm_P0.65mm" H 3550 3000 50  0001 C CNN
-F 3 "http://www.ti.com/lit/gpn/sn74HC14" H 3550 3000 50  0001 C CNN
+F 3 "https://www.ti.com/lit/ds/symlink/sn74lv14a.pdf" H 3550 3000 50  0001 C CNN
 	2    3550 3000
 	1    0    0    -1
@@
 P 4800 3000
 F 0 "U34" H 4800 3317 50  0000 C CNN
-F 1 "74ACT14MTCX" H 4800 3226 50  0000 C CNN
+F 1 "SN74LV14APW" H 4800 3226 50  0000 C CNN
 F 2 "Package_SO:TSSOP-14_4.4x5mm_P0.65mm" H 4800 3000 50  0001 C CNN
-F 3 "http://www.ti.com/lit/gpn/sn74HC14" H 4800 3000 50  0001 C CNN
+F 3 "https://www.ti.com/lit/ds/symlink/sn74lv14a.pdf" H 4800 3000 50  0001 C CNN
 	3    4800 3000
 	1    0    0    -1
@@
 P 3550 4400
 F 0 "U34" H 3550 4717 50  0000 C CNN
-F 1 "74ACT14MTCX" H 3550 4626 50  0000 C CNN
+F 1 "SN74LV14APW" H 3550 4626 50  0000 C CNN
 F 2 "Package_SO:TSSOP-14_4.4x5mm_P0.65mm" H 3550 4400 50  0001 C CNN
-F 3 "http://www.ti.com/lit/gpn/sn74HC14" H 3550 4400 50  0001 C CNN
+F 3 "https://www.ti.com/lit/ds/symlink/sn74lv14a.pdf" H 3550 4400 50  0001 C CNN
 	4    3550 4400
 	1    0    0    -1
@@
 P 4800 3550
 F 0 "U34" H 4800 3867 50  0000 C CNN
-F 1 "74ACT14MTCX" H 4800 3776 50  0000 C CNN
+F 1 "SN74LV14APW" H 4800 3776 50  0000 C CNN
 F 2 "Package_SO:TSSOP-14_4.4x5mm_P0.65mm" H 4800 3550 50  0001 C CNN
-F 3 "http://www.ti.com/lit/gpn/sn74HC14" H 4800 3550 50  0001 C CNN
+F 3 "https://www.ti.com/lit/ds/symlink/sn74lv14a.pdf" H 4800 3550 50  0001 C CNN
 	5    4800 3550
 	1    0    0    -1
@@
 P 9450 2850
 F 0 "U34" H 9450 3167 50  0000 C CNN
-F 1 "74ACT14MTCX" H 9450 3076 50  0000 C CNN
+F 1 "SN74LV14APW" H 9450 3076 50  0000 C CNN
 F 2 "Package_SO:TSSOP-14_4.4x5mm_P0.65mm" H 9450 2850 50  0001 C CNN
-F 3 "http://www.ti.com/lit/gpn/sn74HC14" H 9450 2850 50  0001 C CNN
+F 3 "https://www.ti.com/lit/ds/symlink/sn74lv14a.pdf" H 9450 2850 50  0001 C CNN
 	6    9450 2850
 	1    0    0    -1
@@
 P 3050 6450
 F 0 "U34" H 3280 6496 50  0000 L CNN
-F 1 "74ACT14MTCX" H 3280 6405 50  0000 L CNN
+F 1 "SN74LV14APW" H 3280 6405 50  0000 L CNN
 F 2 "Package_SO:TSSOP-14_4.4x5mm_P0.65mm" H 3050 6450 50  0001 C CNN
-F 3 "http://www.ti.com/lit/gpn/sn74HC14" H 3050 6450 50  0001 C CNN
+F 3 "https://www.ti.com/lit/ds/symlink/sn74lv14a.pdf" H 3050 6450 50  0001 C CNN
 	7    3050 6450
 	1    0    0    -1
@@
 P 5750 1750
 F 0 "U30" H 6100 1500 50  0000 C CNN
-F 1 "74LS74" H 6050 1400 50  0000 C CNN
-F 2 "" H 5750 1750 50  0001 C CNN
-F 3 "74xx/74hc_hct74.pdf" H 5750 1750 50  0001 C CNN
+F 1 "74HC74PW" H 6050 1400 50  0000 C CNN
+F 2 "Package_SO:TSSOP-14_4.4x5mm_P0.65mm" H 5750 1750 50  0001 C CNN
+F 3 "http://www.farnell.com/datasheets/1648944.pdf" H 5750 1750 50  0001 C CNN
 	1    5750 1750
 	1    0    0    -1
@@
 P 9900 4000
 F 0 "U30" H 9900 4481 50  0000 C CNN
-F 1 "74LS74" H 9900 4390 50  0000 C CNN
-F 2 "" H 9900 4000 50  0001 C CNN
-F 3 "74xx/74hc_hct74.pdf" H 9900 4000 50  0001 C CNN
+F 1 "74HC74PW" H 9900 4390 50  0000 C CNN
+F 2 "Package_SO:TSSOP-14_4.4x5mm_P0.65mm" H 9900 4000 50  0001 C CNN
+F 3 "http://www.farnell.com/datasheets/1648944.pdf" H 9900 4000 50  0001 C CNN
 	2    9900 4000
 	1    0    0    -1
@@
 P 4150 6450
 F 0 "U30" H 4380 6496 50  0000 L CNN
-F 1 "74LS74" H 4380 6405 50  0000 L CNN
-F 2 "" H 4150 6450 50  0001 C CNN
-F 3 "74xx/74hc_hct74.pdf" H 4150 6450 50  0001 C CNN
+F 1 "74HC74PW" H 4380 6405 50  0000 L CNN
+F 2 "Package_SO:TSSOP-14_4.4x5mm_P0.65mm" H 4150 6450 50  0001 C CNN
+F 3 "http://www.farnell.com/datasheets/1648944.pdf" H 4150 6450 50  0001 C CNN
 	3    4150 6450
 	1    0    0    -1
@@
 P 5750 1000
 F 0 "U31" H 5725 733 50  0000 C CNN
-F 1 "74AHC1G86" H 5725 824 50  0000 C CNN
-F 2 "" H 5750 1000 50  0001 C CNN
-F 3 "http://www.ti.com/lit/sg/scyt129e/scyt129e.pdf" H 5750 1000 50  0001 C CNN
+F 1 "SN74AHC1G86DBVR" H 5725 824 50  0000 C CNN
+F 2 "Package_TO_SOT_SMD:SOT-23-5" H 5750 1000 50  0001 C CNN
+F 3 "https://www.ti.com/lit/ds/symlink/sn74ahc1g86.pdf" H 5750 1000 50  0001 C CNN
 	1    5750 1000
 	-1   0    0    1

Commit message: Registers: new board started
Parts:
- C38: footprint Capacitor_SMD:CP_Elec_4x4.5 -> Capacitor_Tantalum_SMD:CP_EIA-3528-21_Kemet-B_Pad1.50x2.35mm_HandSolder
Changed lines of the file:
@@
 F 0 "C38" H 9118 1396 50  0000 L CNN
 F 1 "100u" H 9118 1305 50  0000 L CNN
-F 2 "Capacitor_SMD:CP_Elec_4x4.5" H 9038 1200 50  0001 C CNN
+F 2 "Capacitor_Tantalum_SMD:CP_EIA-3528-21_Kemet-B_Pad1.50x2.35mm_HandSolder" H 9038 1200 50  0001 C CNN
 F 3 "~" H 9000 1350 50  0001 C CNN
 	1    9000 1350

Commit message: Registers: add a pull-up on RDY
Parts:
- added R3: 10k, Resistor_SMD:R_0805_2012Metric, symbol Device:R
Connections:
- wire segments 31 -> 32
Changed lines of the file:
@@
 mem_rdy
 Wire Wire Line
-	6650 950  6050 950
+	6650 950  6450 950
 $Comp
 L power:VCC #PWR082
@@
 	1    0    0    -1
 $EndComp
+$Comp
+L Device:R R3
+U 1 1 600B21B7
+P 6450 800
+F 0 "R3" H 6700 750 50  0000 R CNN
+F 1 "10k" H 6700 850 50  0000 R CNN
+F 2 "Resistor_SMD:R_0805_2012Metric" V 6380 800 50  0001 C CNN
+F 3 "~" H 6450 800 50  0001 C CNN
+	1    6450 800
+	-1   0    0    1
+$EndComp
+Connection ~ 6450 950
+Wire Wire Line
+	6450 950  6050 950
+$Comp
+L power:VCC #PWR08
+U 1 1 600B2FB1
+P 6450 650
+F 0 "#PWR08" H 6450 500 50  0001 C CNN
+F 1 "VCC" H 6550 750 50  0000 C CNN
+F 2 "" H 6450 650 50  0001 C CNN
+F 3 "" H 6450 650 50  0001 C CNN
+	1    6450 650
+	1    0    0    -1
+$EndComp
