File: boards/control/control.sch (KiCad schematic (older format))
At the start: 53 parts, among them U1 74ACT08, U2 74ACT139, U3 74ACT74, U4 74ACT86, U5 74ACT32, U6 28C256, U7 28C256, U8 28C256

Commit message: AT28C256-PLCC symbol
Parts:
- removed U6, U7, U8: 28C256, Package_LCC:PLCC-28_SMD-Socket, symbol Memory_EEPROM:28C256
- added U? (x3): AT28C256-PLCC32, symbol missing:AT28C256-PLCC32
Changed lines of the file:
@@
 NoConn ~ 5700 9500
 NoConn ~ 5700 8950
-$Comp
-L Memory_EEPROM:28C256 U6
-U 1 1 6002A9FF
-P 7650 2600
-F 0 "U6" H 8050 1650 50  0000 C CNN
-F 1 "28C256" H 8000 1550 50  0000 C CNN
-F 2 "Package_LCC:PLCC-28_SMD-Socket" H 7650 2600 50  0001 C CNN
-F 3 "http://ww1.microchip.com/downloads/en/DeviceDoc/doc0006.pdf" H 7650 2600 50  0001 C CNN
-	1    7650 2600
-	1    0    0    -1
-$EndComp
 Text Label 7250 1700 2    50   ~ 0
 ir0
@@
 L power:GND #PWR031
 U 1 1 60036651
+P 7250 3300
+F 0 "#PWR031" H 7250 3050 50  0001 C CNN
+F 1 "GND" V 7255 3172 50  0000 R CNN
+F 2 "" H 7250 3300 50  0001 C CNN
+F 3 "" H 7250 3300 50  0001 C CNN
+	1    7250 3300
+	0    1    1    0
+$EndComp
+$Comp
+L power:VCC #PWR030
+U 1 1 60037061
 P 7250 3400
-F 0 "#PWR031" H 7250 3150 50  0001 C CNN
-F 1 "GND" V 7255 3272 50  0000 R CNN
+F 0 "#PWR030" H 7250 3250 50  0001 C CNN
+F 1 "VCC" V 7268 3527 50  0000 L CNN
 F 2 "" H 7250 3400 50  0001 C CNN
 F 3 "" H 7250 3400 50  0001 C CNN
 	1    7250 3400
-	0    1    1    0
-$EndComp
-$Comp
-L power:VCC #PWR030
-U 1 1 60037061
-P 7250 3300
-F 0 "#PWR030" H 7250 3150 50  0001 C CNN
-F 1 "VCC" V 7268 3427 50  0000 L CNN
-F 2 "" H 7250 3300 50  0001 C CNN
-F 3 "" H 7250 3300 50  0001 C CNN
-	1    7250 3300
 	0    -1   -1   0
 $EndComp
@@
 F 3 "" H 7650 3700 50  0001 C CNN
 	1    7650 3700
-	1    0    0    -1
-$EndComp
-$Comp
-L Memory_EEPROM:28C256 U7
-U 1 1 6003DC84
-P 10150 2600
-F 0 "U7" H 10550 1650 50  0000 C CNN
-F 1 "28C256" H 10500 1550 50  0000 C CNN
-F 2 "Package_LCC:PLCC-28_SMD-Socket" H 10150 2600 50  0001 C CNN
-F 3 "http://ww1.microchip.com/downloads/en/DeviceDoc/doc0006.pdf" H 10150 2600 50  0001 C CNN
-	1    10150 2600
 	1    0    0    -1
 $EndComp
@@
 L power:GND #PWR042
 U 1 1 6003DCAE
+P 9750 3300
+F 0 "#PWR042" H 9750 3050 50  0001 C CNN
+F 1 "GND" V 9755 3172 50  0000 R CNN
+F 2 "" H 9750 3300 50  0001 C CNN
+F 3 "" H 9750 3300 50  0001 C CNN
+	1    9750 3300
+	0    1    1    0
+$EndComp
+$Comp
+L power:VCC #PWR041
+U 1 1 6003DCB4
 P 9750 3400
-F 0 "#PWR042" H 9750 3150 50  0001 C CNN
-F 1 "GND" V 9755 3272 50  0000 R CNN
+F 0 "#PWR041" H 9750 3250 50  0001 C CNN
+F 1 "VCC" V 9768 3527 50  0000 L CNN
 F 2 "" H 9750 3400 50  0001 C CNN
 F 3 "" H 9750 3400 50  0001 C CNN
 	1    9750 3400
-	0    1    1    0
-$EndComp
-$Comp
-L power:VCC #PWR041
-U 1 1 6003DCB4
-P 9750 3300
-F 0 "#PWR041" H 9750 3150 50  0001 C CNN
-F 1 "VCC" V 9768 3427 50  0000 L CNN
-F 2 "" H 9750 3300 50  0001 C CNN
-F 3 "" H 9750 3300 50  0001 C CNN
-	1    9750 3300
 	0    -1   -1   0
 $EndComp
@@
 F 3 "" H 10150 3700 50  0001 C CNN
 	1    10150 3700
-	1    0    0    -1
-$EndComp
-$Comp
-L Memory_EEPROM:28C256 U8
-U 1 1 60041836
-P 12400 2600
-F 0 "U8" H 12800 1650 50  0000 C CNN
-F 1 "28C256" H 12750 1550 50  0000 C CNN
-F 2 "Package_LCC:PLCC-28_SMD-Socket" H 12400 2600 50  0001 C CNN
-F 3 "http://ww1.microchip.com/downloads/en/DeviceDoc/doc0006.pdf" H 12400 2600 50  0001 C CNN
-	1    12400 2600
 	1    0    0    -1
 $EndComp
@@
 L power:GND #PWR052
 U 1 1 60041860
+P 12000 3300
+F 0 "#PWR052" H 12000 3050 50  0001 C CNN
+F 1 "GND" V 12005 3172 50  0000 R CNN
+F 2 "" H 12000 3300 50  0001 C CNN
+F 3 "" H 12000 3300 50  0001 C CNN
+	1    12000 3300
+	0    1    1    0
+$EndComp
+$Comp
+L power:VCC #PWR051
+U 1 1 60041866
 P 12000 3400
-F 0 "#PWR052" H 12000 3150 50  0001 C CNN
-F 1 "GND" V 12005 3272 50  0000 R CNN
+F 0 "#PWR051" H 12000 3250 50  0001 C CNN
+F 1 "VCC" V 12018 3527 50  0000 L CNN
 F 2 "" H 12000 3400 50  0001 C CNN
 F 3 "" H 12000 3400 50  0001 C CNN
 	1    12000 3400
-	0    1    1    0
-$EndComp
-$Comp
-L power:VCC #PWR051
-U 1 1 60041866
-P 12000 3300
-F 0 "#PWR051" H 12000 3150 50  0001 C CNN
-F 1 "VCC" V 12018 3427 50  0000 L CNN
-F 2 "" H 12000 3300 50  0001 C CNN
-F 3 "" H 12000 3300 50  0001 C CNN
-	1    12000 3300
 	0    -1   -1   0
 $EndComp
@@
 Wire Bus Line
 	3750 1150 3750 1950
+$Comp
+L missing:AT28C256-PLCC32 U?
+U 1 1 60136676
+P 7650 2600
+F 0 "U?" H 8050 1750 50  0000 C CNN
+F 1 "AT28C256-PLCC32" H 8350 1650 50  0000 C CNN
+F 2 "" H 7900 2950 50  0001 C CNN
+F 3 "http://ww1.microchip.com/downloads/en/DeviceDoc/doc0006.pdf" H 7900 2950 50  0001 C CNN
+	1    7650 2600
+	1    0    0    -1
+$EndComp
+$Comp
+L missing:AT28C256-PLCC32 U?
+U 1 1 60139786
+P 10150 2600
+F 0 "U?" H 10550 1750 50  0000 C CNN
+F 1 "AT28C256-PLCC32" H 10850 1650 50  0000 C CNN
+F 2 "" H 10400 2950 50  0001 C CNN
+F 3 "http://ww1.microchip.com/downloads/en/DeviceDoc/doc0006.pdf" H 10400 2950 50  0001 C CNN
+	1    10150 2600
+	1    0    0    -1
+$EndComp
+$Comp
+L missing:AT28C256-PLCC32 U?
+U 1 1 6013B3C2
+P 12400 2600
+F 0 "U?" H 12800 1750 50  0000 C CNN
+F 1 "AT28C256-PLCC32" H 13100 1650 50  0000 C CNN
+F 2 "" H 12650 2950 50  0001 C CNN
+F 3 "http://ww1.microchip.com/downloads/en/DeviceDoc/doc0006.pdf" H 12650 2950 50  0001 C CNN
+	1    12400 2600
+	1    0    0    -1
+$EndComp
 $EndSCHEMATC

Commit message: Control unit board
Parts:
- removed D2: LED, LED_SMD:LED_0805_2012Metric, symbol Device:LED
- removed R2: LED, Resistor_SMD:R_0805_2012Metric, symbol Device:R
- added H1, H2, H3, H4: MountingHole, MountingHole:MountingHole_3.2mm_M3, symbol Mechanical:MountingHole
- U6, U7, U8: renamed from U?; footprint (none) -> missing:PLCC-32_SMD_Socket
Connections:
- no-connect marks 11 -> 12
Changed lines of the file:
@@
 condition_result
-$Comp
-L Device:LED D2
-U 1 1 600FD3DA
-P 6050 5650
-F 0 "D2" H 6050 5500 50  0000 C CNN
-F 1 "LED" H 6043 5775 50  0001 C CNN
-F 2 "LED_SMD:LED_0805_2012Metric" H 6050 5650 50  0001 C CNN
-F 3 "~" H 6050 5650 50  0001 C CNN
-	1    6050 5650
-	1    0    0    -1
-$EndComp
-$Comp
-L Device:R R2
-U 1 1 600FF980
-P 6350 5650
-F 0 "R2" V 6500 5650 50  0000 C CNN
-F 1 "LED" V 6600 5650 50  0000 C CNN
-F 2 "Resistor_SMD:R_0805_2012Metric" V 6280 5650 50  0001 C CNN
-F 3 "~" H 6350 5650 50  0001 C CNN
-	1    6350 5650
-	0    1    1    0
-$EndComp
-$Comp
-L power:VCC #PWR026
-U 1 1 601003F3
-P 6500 5650
-F 0 "#PWR026" H 6500 5500 50  0001 C CNN
-F 1 "VCC" V 6517 5778 50  0000 L CNN
-F 2 "" H 6500 5650 50  0001 C CNN
-F 3 "" H 6500 5650 50  0001 C CNN
-	1    6500 5650
-	0    1    1    0
-$EndComp
-Wire Wire Line
-	5550 5650 5900 5650
 $Comp
 L Device:LED D1
@@
 	1    0    0    -1
 $EndComp
+$Comp
+L missing:AT28C256-PLCC32 U6
+U 1 1 60136676
+P 7650 2600
+F 0 "U6" H 8050 1750 50  0000 C CNN
+F 1 "AT28C256-PLCC32" H 8350 1650 50  0000 C CNN
+F 2 "missing:PLCC-32_SMD_Socket" H 7900 2950 50  0001 C CNN
+F 3 "http://ww1.microchip.com/downloads/en/DeviceDoc/doc0006.pdf" H 7900 2950 50  0001 C CNN
+	1    7650 2600
+	1    0    0    -1
+$EndComp
+$Comp
+L missing:AT28C256-PLCC32 U7
+U 1 1 60139786
+P 10150 2600
+F 0 "U7" H 10550 1750 50  0000 C CNN
+F 1 "AT28C256-PLCC32" H 10850 1650 50  0000 C CNN
+F 2 "missing:PLCC-32_SMD_Socket" H 10400 2950 50  0001 C CNN
+F 3 "http://ww1.microchip.com/downloads/en/DeviceDoc/doc0006.pdf" H 10400 2950 50  0001 C CNN
+	1    10150 2600
+	1    0    0    -1
+$EndComp
+$Comp
+L missing:AT28C256-PLCC32 U8
+U 1 1 6013B3C2
+P 12400 2600
+F 0 "U8" H 12800 1750 50  0000 C CNN
+F 1 "AT28C256-PLCC32" H 13100 1650 50  0000 C CNN
+F 2 "missing:PLCC-32_SMD_Socket" H 12650 2950 50  0001 C CNN
+F 3 "http://ww1.microchip.com/downloads/en/DeviceDoc/doc0006.pdf" H 12650 2950 50  0001 C CNN
+	1    12400 2600
+	1    0    0    -1
+$EndComp
+$Comp
+L Mechanical:MountingHole H2
+U 1 1 6026AC94
+P 850 650
+F 0 "H2" H 950 696 50  0000 L CNN
+F 1 "MountingHole" H 950 605 50  0000 L CNN
+F 2 "MountingHole:MountingHole_3.2mm_M3" H 850 650 50  0001 C CNN
+F 3 "~" H 850 650 50  0001 C CNN
+	1    850  650
+	1    0    0    -1
+$EndComp
+$Comp
+L Mechanical:MountingHole H3
+U 1 1 6026B403
+P 15150 750
+F 0 "H3" H 15250 796 50  0000 L CNN
+F 1 "MountingHole" H 15250 705 50  0000 L CNN
+F 2 "MountingHole:MountingHole_3.2mm_M3" H 15150 750 50  0001 C CNN
+F 3 "~" H 15150 750 50  0001 C CNN
+	1    15150 750
+	1    0    0    -1
+$EndComp
+$Comp
+L Mechanical:MountingHole H4
+U 1 1 6026B9D0
+P 15150 9550
+F 0 "H4" H 15250 9596 50  0000 L CNN
+F 1 "MountingHole" H 15250 9505 50  0000 L CNN
+F 2 "MountingHole:MountingHole_3.2mm_M3" H 15150 9550 50  0001 C CNN
+F 3 "~" H 15150 9550 50  0001 C CNN
+	1    15150 9550
+	1    0    0    -1
+$EndComp
+$Comp
+L Mechanical:MountingHole H1
+U 1 1 6026C0CF
+P 750 11000
+F 0 "H1" H 850 11046 50  0000 L CNN
+F 1 "MountingHole" H 850 10955 50  0000 L CNN
+F 2 "MountingHole:MountingHole_3.2mm_M3" H 750 11000 50  0001 C CNN
+F 3 "~" H 750 11000 50  0001 C CNN
+	1    750  11000
+	1    0    0    -1
+$EndComp
+NoConn ~ 5550 5650
 Wire Bus Line
 	3750 2050 3750 2650
 Wire Bus Line
 	3750 1150 3750 1950
-$Comp
-L missing:AT28C256-PLCC32 U?
-U 1 1 60136676
-P 7650 2600
-F 0 "U?" H 8050 1750 50  0000 C CNN
-F 1 "AT28C256-PLCC32" H 8350 1650 50  0000 C CNN
-F 2 "" H 7900 2950 50  0001 C CNN
-F 3 "http://ww1.microchip.com/downloads/en/DeviceDoc/doc0006.pdf" H 7900 2950 50  0001 C CNN
-	1    7650 2600
-	1    0    0    -1
-$EndComp
-$Comp
-L missing:AT28C256-PLCC32 U?
-U 1 1 60139786
-P 10150 2600
-F 0 "U?" H 10550 1750 50  0000 C CNN
-F 1 "AT28C256-PLCC32" H 10850 1650 50  0000 C CNN
-F 2 "" H 10400 2950 50  0001 C CNN
-F 3 "http://ww1.microchip.com/downloads/en/DeviceDoc/doc0006.pdf" H 10400 2950 50  0001 C CNN
-	1    10150 2600
-	1    0    0    -1
-$EndComp
-$Comp
-L missing:AT28C256-PLCC32 U?
-U 1 1 6013B3C2
-P 12400 2600
-F 0 "U?" H 12800 1750 50  0000 C CNN
-F 1 "AT28C256-PLCC32" H 13100 1650 50  0000 C CNN
-F 2 "" H 12650 2950 50  0001 C CNN
-F 3 "http://ww1.microchip.com/downloads/en/DeviceDoc/doc0006.pdf" H 12650 2950 50  0001 C CNN
-	1    12400 2600
-	1    0    0    -1
-$EndComp
 $EndSCHEMATC

Commit message: Add a 2-bit state for the future expansion
Parts:
- added C7: 0.1u, Capacitor_SMD:C_0805_2012Metric, symbol Device:C
- added D2, D21: LED, LED_SMD:LED_0805_2012Metric, symbol Device:LED
- added R2, R21, R23, R24: 0, Resistor_SMD:R_0805_2012Metric, symbol Device:R
- added R22, R25: LED, Resistor_SMD:R_0805_2012Metric, symbol Device:R
- added U9: 74ACT74, Package_SO:SOIC-14_3.9x8.7mm_P1.27mm, symbol 74xx:74HC74
Connections:
- net GND: now also C7.2, U9.7 (GND); no longer U6.3 (A12), U6.30 (A13), U7.3 (A12), U7.30 (A13), U8.3 (A12), U8.30 (A13)
- net VCC: now also C7.1, R22.1, R25.1, U9.10 (~S), U9.14 (VCC), U9.4 (~S)
- net clk: now also R2.2, R23.2
- net ~clk: now also R21.2, R24.2
- net ~oe_a_d: now also U7.18 (IO3); no longer U7.19 (IO4)
- net ~oe_b_d: now also U7.19 (IO4); no longer U7.20 (IO5)
- net ~rst: now also U9.1 (~R), U9.13 (~R)
- net ~we_flags: now also U7.20 (IO5); no longer U7.21 (IO6)
- net s2_d: now reaches U7.22 (IO7)
- net s2_d: now also U9.12 (D)
- new net: R2.1, R21.1, U9.3 (C)
- new net: D2.1 (K), U9.6 (~Q)
- new net: R23.1, R24.1, U9.11 (C)
- new net: D21.1 (K), U9.8 (~Q)
- new net: D2.2 (A), R22.2
- new net: D21.2 (A), R25.2
- new net s1: U6.3 (A12), U7.3 (A12), U8.3 (A12), U9.5 (Q)
- new net s1_d: U7.21 (IO6), U9.2 (D)
- new net s2: U6.30 (A13), U7.30 (A13), U8.30 (A13), U9.9 (Q)
- no-connect marks 12 -> 10
Other:
- note added: "Install one of resistors to select clock source"

Commit message: LEDs and LED resistors
Parts:
- D1, D2, D21: value LED -> KP-2012CGCK
- D10, D11, D12, D13, D14, D15, D16, D17, D18, D19, D20, D3, D4, D5, D6, D7, D8, D9: value LED -> KP-2012EC
- R1, R22, R25: value LED -> 600
- R10, R11, R12, R13, R14, R15, R16, R17, R18, R19, R20, R3, R4, R5, R6, R7, R8, R9: value LED -> 620
Changed lines of the file:
@@
 P 14200 1050
 F 0 "D3" H 15100 1050 50  0000 C CNN
-F 1 "LED" H 14193 1175 50  0001 C CNN
+F 1 "KP-2012EC" H 14193 1175 50  0001 C CNN
 F 2 "LED_SMD:LED_0805_2012Metric" H 14200 1050 50  0001 C CNN
 F 3 "~" H 14200 1050 50  0001 C CNN
@@
 P 14200 1250
 F 0 "D4" H 15100 1250 50  0000 C CNN
-F 1 "LED" H 14193 1375 50  0001 C CNN
+F 1 "KP-2012EC" H 14193 1375 50  0001 C CNN
 F 2 "LED_SMD:LED_0805_2012Metric" H 14200 1250 50  0001 C CNN
 F 3 "~" H 14200 1250 50  0001 C CNN
@@
 P 14200 2250
 F 0 "D9" H 15100 2250 50  0000 C CNN
-F 1 "LED" H 14193 2375 50  0001 C CNN
+F 1 "KP-2012EC" H 14193 2375 50  0001 C CNN
 F 2 "LED_SMD:LED_0805_2012Metric" H 14200 2250 50  0001 C CNN
 F 3 "~" H 14200 2250 50  0001 C CNN
@@
 P 14200 2450
 F 0 "D10" H 15100 2450 50  0000 C CNN
-F 1 "LED" H 14193 2575 50  0001 C CNN
+F 1 "KP-2012EC" H 14193 2575 50  0001 C CNN
 F 2 "LED_SMD:LED_0805_2012Metric" H 14200 2450 50  0001 C CNN
 F 3 "~" H 14200 2450 50  0001 C CNN
@@
 P 14200 3050
 F 0 "D13" H 15100 3050 50  0000 C CNN
-F 1 "LED" H 14193 3175 50  0001 C CNN
+F 1 "KP-2012EC" H 14193 3175 50  0001 C CNN
 F 2 "LED_SMD:LED_0805_2012Metric" H 14200 3050 50  0001 C CNN
 F 3 "~" H 14200 3050 50  0001 C CNN
@@
 P 14200 3250
 F 0 "D14" H 15100 3250 50  0000 C CNN
-F 1 "LED" H 14193 3375 50  0001 C CNN
+F 1 "KP-2012EC" H 14193 3375 50  0001 C CNN
 F 2 "LED_SMD:LED_0805_2012Metric" H 14200 3250 50  0001 C CNN
 F 3 "~" H 14200 3250 50  0001 C CNN
@@
 P 14200 3450
 F 0 "D15" H 15100 3450 50  0000 C CNN
-F 1 "LED" H 14193 3575 50  0001 C CNN
+F 1 "KP-2012EC" H 14193 3575 50  0001 C CNN
 F 2 "LED_SMD:LED_0805_2012Metric" H 14200 3450 50  0001 C CNN
 F 3 "~" H 14200 3450 50  0001 C CNN
@@
 P 14200 3650
 F 0 "D16" H 15100 3650 50  0000 C CNN
-F 1 "LED" H 14193 3775 50  0001 C CNN
+F 1 "KP-2012EC" H 14193 3775 50  0001 C CNN
 F 2 "LED_SMD:LED_0805_2012Metric" H 14200 3650 50  0001 C CNN
 F 3 "~" H 14200 3650 50  0001 C CNN
@@
 P 14200 3850
 F 0 "D17" H 15100 3850 50  0000 C CNN
-F 1 "LED" H 14193 3975 50  0001 C CNN
+F 1 "KP-2012EC" H 14193 3975 50  0001 C CNN
 F 2 "LED_SMD:LED_0805_2012Metric" H 14200 3850 50  0001 C CNN
 F 3 "~" H 14200 3850 50  0001 C CNN
@@
 P 14200 4050
 F 0 "D18" H 15100 4050 50  0000 C CNN
-F 1 "LED" H 14193 4175 50  0001 C CNN
+F 1 "KP-2012EC" H 14193 4175 50  0001 C CNN
 F 2 "LED_SMD:LED_0805_2012Metric" H 14200 4050 50  0001 C CNN
 F 3 "~" H 14200 4050 50  0001 C CNN
@@
 P 14200 4250
 F 0 "D19" H 15100 4250 50  0000 C CNN
-F 1 "LED" H 14193 4375 50  0001 C CNN
+F 1 "KP-2012EC" H 14193 4375 50  0001 C CNN
 F 2 "LED_SMD:LED_0805_2012Metric" H 14200 4250 50  0001 C CNN
 F 3 "~" H 14200 4250 50  0001 C CNN
@@
 P 14200 4450
 F 0 "D20" H 15100 4450 50  0000 C CNN
-F 1 "LED" H 14193 4575 50  0001 C CNN
+F 1 "KP-2012EC" H 14193 4575 50  0001 C CNN
 F 2 "LED_SMD:LED_0805_2012Metric" H 14200 4450 50  0001 C CNN
 F 3 "~" H 14200 4450 50  0001 C CNN
@@
 P 14200 2850
 F 0 "D12" H 13300 2850 50  0000 C CNN
-F 1 "LED" H 14193 2975 50  0001 C CNN
+F 1 "KP-2012EC" H 14193 2975 50  0001 C CNN
 F 2 "LED_SMD:LED_0805_2012Metric" H 14200 2850 50  0001 C CNN
 F 3 "~" H 14200 2850 50  0001 C CNN
@@
 P 14200 2650
 F 0 "D11" H 13300 2650 50  0000 C CNN
-F 1 "LED" H 14193 2775 50  0001 C CNN
+F 1 "KP-2012EC" H 14193 2775 50  0001 C CNN
 F 2 "LED_SMD:LED_0805_2012Metric" H 14200 2650 50  0001 C CNN
 F 3 "~" H 14200 2650 50  0001 C CNN
@@
 P 14200 2050
 F 0 "D8" H 13300 2050 50  0000 C CNN
-F 1 "LED" H 14193 2175 50  0001 C CNN
+F 1 "KP-2012EC" H 14193 2175 50  0001 C CNN
 F 2 "LED_SMD:LED_0805_2012Metric" H 14200 2050 50  0001 C CNN
 F 3 "~" H 14200 2050 50  0001 C CNN
@@
 P 14200 1850
 F 0 "D7" H 13300 1850 50  0000 C CNN
-F 1 "LED" H 14193 1975 50  0001 C CNN
+F 1 "KP-2012EC" H 14193 1975 50  0001 C CNN
 F 2 "LED_SMD:LED_0805_2012Metric" H 14200 1850 50  0001 C CNN
 F 3 "~" H 14200 1850 50  0001 C CNN
@@
 P 14200 1650
 F 0 "D6" H 13300 1650 50  0000 C CNN
-F 1 "LED" H 14193 1775 50  0001 C CNN
+F 1 "KP-2012EC" H 14193 1775 50  0001 C CNN
 F 2 "LED_SMD:LED_0805_2012Metric" H 14200 1650 50  0001 C CNN
 F 3 "~" H 14200 1650 50  0001 C CNN
@@
 P 14200 1450
 F 0 "D5" H 13300 1450 50  0000 C CNN
-F 1 "LED" H 14193 1575 50  0001 C CNN
+F 1 "KP-2012EC" H 14193 1575 50  0001 C CNN
 F 2 "LED_SMD:LED_0805_2012Metric" H 14200 1450 50  0001 C CNN
 F 3 "~" H 14200 1450 50  0001 C CNN
@@
 P 14500 1050
 F 0 "R3" V 14500 1850 50  0000 C CNN
-F 1 "LED" V 14500 2050 50  0000 C CNN
+F 1 "620" V 14500 2050 50  0000 C CNN
 F 2 "Resistor_SMD:R_0805_2012Metric" V 14430 1050 50  0001 C CNN
 F 3 "~" H 14500 1050 50  0001 C CNN
@@
 P 14500 1250
 F 0 "R4" V 14500 2050 50  0000 C CNN
-F 1 "LED" V 14500 2250 50  0000 C CNN
+F 1 "620" V 14500 2250 50  0000 C CNN
 F 2 "Resistor_SMD:R_0805_2012Metric" V 14430 1250 50  0001 C CNN
 F 3 "~" H 14500 1250 50  0001 C CNN
@@
 P 14500 1450
 F 0 "R5" V 14500 2250 50  0000 C CNN
-F 1 "LED" V 14500 2450 50  0000 C CNN
+F 1 "620" V 14500 2450 50  0000 C CNN
 F 2 "Resistor_SMD:R_0805_2012Metric" V 14430 1450 50  0001 C CNN
 F 3 "~" H 14500 1450 50  0001 C CNN
@@
 P 14500 1650
 F 0 "R6" V 14500 2450 50  0000 C CNN
-F 1 "LED" V 14500 2650 50  0000 C CNN
+F 1 "620" V 14500 2650 50  0000 C CNN
 F 2 "Resistor_SMD:R_0805_2012Metric" V 14430 1650 50  0001 C CNN
 F 3 "~" H 14500 1650 50  0001 C CNN
@@
 P 14500 1850
 F 0 "R7" V 14500 2650 50  0000 C CNN
-F 1 "LED" V 14500 2850 50  0000 C CNN
+F 1 "620" V 14500 2850 50  0000 C CNN
 F 2 "Resistor_SMD:R_0805_2012Metric" V 14430 1850 50  0001 C CNN
 F 3 "~" H 14500 1850 50  0001 C CNN
@@
 P 14500 2050
 F 0 "R8" V 14500 2850 50  0000 C CNN
-F 1 "LED" V 14500 3050 50  0000 C CNN
+F 1 "620" V 14500 3050 50  0000 C CNN
 F 2 "Resistor_SMD:R_0805_2012Metric" V 14430 2050 50  0001 C CNN
 F 3 "~" H 14500 2050 50  0001 C CNN
@@
 P 14500 2250
 F 0 "R9" V 14500 3050 50  0000 C CNN
-F 1 "LED" V 14500 3250 50  0000 C CNN
+F 1 "620" V 14500 3250 50  0000 C CNN
 F 2 "Resistor_SMD:R_0805_2012Metric" V 14430 2250 50  0001 C CNN
 F 3 "~" H 14500 2250 50  0001 C CNN
@@
 P 14500 2450
 F 0 "R10" V 14500 3250 50  0000 C CNN
-F 1 "LED" V 14500 3450 50  0000 C CNN
+F 1 "620" V 14500 3450 50  0000 C CNN
 F 2 "Resistor_SMD:R_0805_2012Metric" V 14430 2450 50  0001 C CNN
 F 3 "~" H 14500 2450 50  0001 C CNN
@@
 P 14500 2650
 F 0 "R11" V 14500 3450 50  0000 C CNN
-F 1 "LED" V 14500 3650 50  0000 C CNN
+F 1 "620" V 14500 3650 50  0000 C CNN
 F 2 "Resistor_SMD:R_0805_2012Metric" V 14430 2650 50  0001 C CNN
 F 3 "~" H 14500 2650 50  0001 C CNN
@@
 P 14500 2850
 F 0 "R12" V 14500 3650 50  0000 C CNN
-F 1 "LED" V 14500 3850 50  0000 C CNN
+F 1 "620" V 14500 3850 50  0000 C CNN
 F 2 "Resistor_SMD:R_0805_2012Metric" V 14430 2850 50  0001 C CNN
 F 3 "~" H 14500 2850 50  0001 C CNN
@@
 P 14500 3050
 F 0 "R13" V 14500 3850 50  0000 C CNN
-F 1 "LED" V 14500 4050 50  0000 C CNN
+F 1 "620" V 14500 4050 50  0000 C CNN
 F 2 "Resistor_SMD:R_0805_2012Metric" V 14430 3050 50  0001 C CNN
 F 3 "~" H 14500 3050 50  0001 C CNN
@@
 P 14500 3250
 F 0 "R14" V 14500 4050 50  0000 C CNN
-F 1 "LED" V 14500 4250 50  0000 C CNN
+F 1 "620" V 14500 4250 50  0000 C CNN
 F 2 "Resistor_SMD:R_0805_2012Metric" V 14430 3250 50  0001 C CNN
 F 3 "~" H 14500 3250 50  0001 C CNN
@@
 P 14500 3450
 F 0 "R15" V 14500 4250 50  0000 C CNN
-F 1 "LED" V 14500 4450 50  0000 C CNN
+F 1 "620" V 14500 4450 50  0000 C CNN
 F 2 "Resistor_SMD:R_0805_2012Metric" V 14430 3450 50  0001 C CNN
 F 3 "~" H 14500 3450 50  0001 C CNN
@@
 P 14500 3650
 F 0 "R16" V 14500 4450 50  0000 C CNN
-F 1 "LED" V 14500 4650 50  0000 C CNN
+F 1 "620" V 14500 4650 50  0000 C CNN
 F 2 "Resistor_SMD:R_0805_2012Metric" V 14430 3650 50  0001 C CNN
 F 3 "~" H 14500 3650 50  0001 C CNN
@@
 P 14500 3850
 F 0 "R17" V 14500 4650 50  0000 C CNN
-F 1 "LED" V 14500 4850 50  0000 C CNN
+F 1 "620" V 14500 4850 50  0000 C CNN
 F 2 "Resistor_SMD:R_0805_2012Metric" V 14430 3850 50  0001 C CNN
 F 3 "~" H 14500 3850 50  0001 C CNN
@@
 P 14500 4050
 F 0 "R18" V 14500 4850 50  0000 C CNN
-F 1 "LED" V 14500 5050 50  0000 C CNN
+F 1 "620" V 14500 5050 50  0000 C CNN
 F 2 "Resistor_SMD:R_0805_2012Metric" V 14430 4050 50  0001 C CNN
 F 3 "~" H 14500 4050 50  0001 C CNN
@@
 P 14500 4250
 F 0 "R19" V 14500 5050 50  0000 C CNN
-F 1 "LED" V 14500 5250 50  0000 C CNN
+F 1 "620" V 14500 5250 50  0000 C CNN
 F 2 "Resistor_SMD:R_0805_2012Metric" V 14430 4250 50  0001 C CNN
 F 3 "~" H 14500 4250 50  0001 C CNN
@@
 P 14500 4450
 F 0 "R20" V 14500 5250 50  0000 C CNN
-F 1 "LED" V 14500 5450 50  0000 C CNN
+F 1 "620" V 14500 5450 50  0000 C CNN
 F 2 "Resistor_SMD:R_0805_2012Metric" V 14430 4450 50  0001 C CNN
 F 3 "~" H 14500 4450 50  0001 C CNN
@@
 P 2950 5650
 F 0 "D1" H 2950 5500 50  0000 C CNN
-F 1 "LED" H 2943 5775 50  0001 C CNN
+F 1 "KP-2012CGCK" H 2943 5775 50  0001 C CNN
 F 2 "LED_SMD:LED_0805_2012Metric" H 2950 5650 50  0001 C CNN
 F 3 "~" H 2950 5650 50  0001 C CNN
@@
 P 3250 5650
 F 0 "R1" V 3400 5650 50  0000 C CNN
-F 1 "LED" V 3500 5650 50  0000 C CNN
+F 1 "600" V 3500 5650 50  0000 C CNN
 F 2 "Resistor_SMD:R_0805_2012Metric" V 3180 5650 50  0001 C CNN
 F 3 "~" H 3250 5650 50  0001 C CNN
@@
 P 10550 8100
 F 0 "D2" H 10550 7950 50  0000 C CNN
-F 1 "LED" H 10543 8225 50  0001 C CNN
+F 1 "KP-2012CGCK" H 10543 8225 50  0001 C CNN
 F 2 "LED_SMD:LED_0805_2012Metric" H 10550 8100 50  0001 C CNN
 F 3 "~" H 10550 8100 50  0001 C CNN
@@
 P 10550 8400
 F 0 "R22" V 10700 8400 50  0000 C CNN
-F 1 "LED" V 10800 8400 50  0000 C CNN
+F 1 "600" V 10800 8400 50  0000 C CNN
 F 2 "Resistor_SMD:R_0805_2012Metric" V 10480 8400 50  0001 C CNN
 F 3 "~" H 10550 8400 50  0001 C CNN
@@
 P 12500 8100
 F 0 "D21" H 12500 7950 50  0000 C CNN
-F 1 "LED" H 12493 8225 50  0001 C CNN
+F 1 "KP-2012CGCK" H 12493 8225 50  0001 C CNN
 F 2 "LED_SMD:LED_0805_2012Metric" H 12500 8100 50  0001 C CNN
 F 3 "~" H 12500 8100 50  0001 C CNN
@@
 P 12500 8400
 F 0 "R25" V 12650 8400 50  0000 C CNN
-F 1 "LED" V 12750 8400 50  0000 C CNN
+F 1 "600" V 12750 8400 50  0000 C CNN
 F 2 "Resistor_SMD:R_0805_2012Metric" V 12430 8400 50  0001 C CNN
 F 3 "~" H 12500 8400 50  0001 C CNN
