File: boards/control/control.sch (KiCad schematic (older format))
At the start: 65 parts, among them U1 74ACT08, U2 74ACT139, U3 74ACT74, U4 74ACT86, U5 74ACT32, U6 AT28C256-PLCC32, U7 AT28C256-PLCC32, U8 AT28C256-PLCC32, U9 74ACT74

Commit message: Part names
Parts:
- U1: value 74ACT08 -> SN74ACT08PW
- U2: value 74ACT139 -> MC74ACT139DG
- U3, U9: value 74ACT74 -> SN74ACT74D
- U4: value 74ACT86 -> MC74ACT86DG
- U5: value 74ACT32 -> SN74ACT32PW
Changed lines of the file:
@@
 P 2150 5550
 F 0 "U3" H 2400 5200 50  0000 C CNN
-F 1 "74ACT74" H 2400 5300 50  0000 C CNN
+F 1 "SN74ACT74D" H 2400 5300 50  0000 C CNN
 F 2 "Package_SO:SOIC-14_3.9x8.7mm_P1.27mm" H 2150 5550 50  0001 C CNN
 F 3 "74xx/74hc_hct74.pdf" H 2150 5550 50  0001 C CNN
@@
 P 5250 5550
 F 0 "U3" H 5500 5200 50  0000 C CNN
-F 1 "74ACT74" H 5500 5300 50  0000 C CNN
+F 1 "SN74ACT74D" H 5500 5300 50  0000 C CNN
 F 2 "Package_SO:SOIC-14_3.9x8.7mm_P1.27mm" H 5250 5550 50  0001 C CNN
 F 3 "74xx/74hc_hct74.pdf" H 5250 5550 50  0001 C CNN
@@
 P 4400 5450
 F 0 "U4" H 4400 5775 50  0000 C CNN
-F 1 "74ACT86" H 4400 5684 50  0000 C CNN
+F 1 "MC74ACT86DG" H 4400 5684 50  0000 C CNN
 F 2 "Package_SO:SOIC-14_3.9x8.7mm_P1.27mm" H 4400 5450 50  0001 C CNN
 F 3 "http://www.ti.com/lit/gpn/sn74HC86" H 4400 5450 50  0001 C CNN
@@
 P 2450 4250
 F 0 "U4" H 2450 4575 50  0000 C CNN
-F 1 "74ACT86" H 2450 4484 50  0000 C CNN
+F 1 "MC74ACT86DG" H 2450 4484 50  0000 C CNN
 F 2 "Package_SO:SOIC-14_3.9x8.7mm_P1.27mm" H 2450 4250 50  0001 C CNN
 F 3 "http://www.ti.com/lit/gpn/sn74HC86" H 2450 4250 50  0001 C CNN
@@
 P 1800 6350
 F 0 "U1" H 1800 6033 50  0000 C CNN
-F 1 "74ACT08" H 1800 6124 50  0000 C CNN
+F 1 "SN74ACT08PW" H 1800 6124 50  0000 C CNN
 F 2 "Package_SO:TSSOP-14_4.4x5mm_P0.65mm" H 1800 6350 50  0001 C CNN
 F 3 "http://www.ti.com/lit/gpn/sn74LS08" H 1800 6350 50  0001 C CNN
@@
 P 1600 8250
 F 0 "U1" H 1830 8296 50  0000 L CNN
-F 1 "74ACT08" H 1830 8205 50  0000 L CNN
+F 1 "SN74ACT08PW" H 1830 8205 50  0000 L CNN
 F 2 "Package_SO:TSSOP-14_4.4x5mm_P0.65mm" H 1600 8250 50  0001 C CNN
 F 3 "http://www.ti.com/lit/gpn/sn74LS08" H 1600 8250 50  0001 C CNN
@@
 P 2450 8250
 F 0 "U4" H 2680 8296 50  0000 L CNN
-F 1 "74ACT86" H 2680 8205 50  0000 L CNN
+F 1 "MC74ACT86DG" H 2680 8205 50  0000 L CNN
 F 2 "Package_SO:SOIC-14_3.9x8.7mm_P1.27mm" H 2450 8250 50  0001 C CNN
 F 3 "http://www.ti.com/lit/gpn/sn74HC86" H 2450 8250 50  0001 C CNN
@@
 P 3300 8250
 F 0 "U3" H 3530 8296 50  0000 L CNN
-F 1 "74ACT74" H 3530 8205 50  0000 L CNN
+F 1 "SN74ACT74D" H 3530 8205 50  0000 L CNN
 F 2 "Package_SO:SOIC-14_3.9x8.7mm_P1.27mm" H 3300 8250 50  0001 C CNN
 F 3 "74xx/74hc_hct74.pdf" H 3300 8250 50  0001 C CNN
@@
 P 11600 5250
 F 0 "U1" H 11600 5575 50  0000 C CNN
-F 1 "74ACT08" H 11600 5484 50  0000 C CNN
+F 1 "SN74ACT08PW" H 11600 5484 50  0000 C CNN
 F 2 "Package_SO:TSSOP-14_4.4x5mm_P0.65mm" H 11600 5250 50  0001 C CNN
 F 3 "http://www.ti.com/lit/gpn/sn74LS08" H 11600 5250 50  0001 C CNN
@@
 P 11600 6350
 F 0 "U1" H 11600 6675 50  0000 C CNN
-F 1 "74ACT08" H 11600 6584 50  0000 C CNN
+F 1 "SN74ACT08PW" H 11600 6584 50  0000 C CNN
 F 2 "Package_SO:TSSOP-14_4.4x5mm_P0.65mm" H 11600 6350 50  0001 C CNN
 F 3 "http://www.ti.com/lit/gpn/sn74LS08" H 11600 6350 50  0001 C CNN
@@
 P 12400 5750
 F 0 "U1" H 12400 6075 50  0000 C CNN
-F 1 "74ACT08" H 12400 5984 50  0000 C CNN
+F 1 "SN74ACT08PW" H 12400 5984 50  0000 C CNN
 F 2 "Package_SO:TSSOP-14_4.4x5mm_P0.65mm" H 12400 5750 50  0001 C CNN
 F 3 "http://www.ti.com/lit/gpn/sn74LS08" H 12400 5750 50  0001 C CNN
@@
 P 9250 5550
 F 0 "U2" H 9250 5917 50  0000 C CNN
-F 1 "74ACT139" H 9250 5826 50  0000 C CNN
+F 1 "MC74ACT139DG" H 9250 5826 50  0000 C CNN
 F 2 "Package_SO:SOIC-16_3.9x9.9mm_P1.27mm" H 9250 5550 50  0001 C CNN
 F 3 "http://www.ti.com/lit/gpn/sn74LS139" H 9250 5550 50  0001 C CNN
@@
 P 6850 9150
 F 0 "U2" H 6850 9517 50  0000 C CNN
-F 1 "74ACT139" H 6850 9426 50  0000 C CNN
+F 1 "MC74ACT139DG" H 6850 9426 50  0000 C CNN
 F 2 "Package_SO:SOIC-16_3.9x9.9mm_P1.27mm" H 6850 9150 50  0001 C CNN
 F 3 "http://www.ti.com/lit/gpn/sn74LS139" H 6850 9150 50  0001 C CNN
@@
 P 2000 9600
 F 0 "U2" H 2230 9646 50  0000 L CNN
-F 1 "74ACT139" H 2230 9555 50  0000 L CNN
+F 1 "MC74ACT139DG" H 2230 9555 50  0000 L CNN
 F 2 "Package_SO:SOIC-16_3.9x9.9mm_P1.27mm" H 2000 9600 50  0001 C CNN
 F 3 "http://www.ti.com/lit/gpn/sn74LS139" H 2000 9600 50  0001 C CNN
@@
 P 10750 4950
 F 0 "U5" H 10750 5275 50  0000 C CNN
-F 1 "74ACT32" H 10750 5184 50  0000 C CNN
+F 1 "SN74ACT32PW" H 10750 5184 50  0000 C CNN
 F 2 "Package_SO:TSSOP-14_4.4x5mm_P0.65mm" H 10750 4950 50  0001 C CNN
 F 3 "http://www.ti.com/lit/gpn/sn74LS32" H 10750 4950 50  0001 C CNN
@@
 P 10750 5500
 F 0 "U5" H 10750 5825 50  0000 C CNN
-F 1 "74ACT32" H 10750 5734 50  0000 C CNN
+F 1 "SN74ACT32PW" H 10750 5734 50  0000 C CNN
 F 2 "Package_SO:TSSOP-14_4.4x5mm_P0.65mm" H 10750 5500 50  0001 C CNN
 F 3 "http://www.ti.com/lit/gpn/sn74LS32" H 10750 5500 50  0001 C CNN
@@
 P 10750 6050
 F 0 "U5" H 10750 6375 50  0000 C CNN
-F 1 "74ACT32" H 10750 6284 50  0000 C CNN
+F 1 "SN74ACT32PW" H 10750 6284 50  0000 C CNN
 F 2 "Package_SO:TSSOP-14_4.4x5mm_P0.65mm" H 10750 6050 50  0001 C CNN
 F 3 "http://www.ti.com/lit/gpn/sn74LS32" H 10750 6050 50  0001 C CNN
@@
 P 10750 6600
 F 0 "U5" H 10750 6925 50  0000 C CNN
-F 1 "74ACT32" H 10750 6834 50  0000 C CNN
+F 1 "SN74ACT32PW" H 10750 6834 50  0000 C CNN
 F 2 "Package_SO:TSSOP-14_4.4x5mm_P0.65mm" H 10750 6600 50  0001 C CNN
 F 3 "http://www.ti.com/lit/gpn/sn74LS32" H 10750 6600 50  0001 C CNN
@@
 P 2900 9600
 F 0 "U5" H 3130 9646 50  0000 L CNN
-F 1 "74ACT32" H 3130 9555 50  0000 L CNN
+F 1 "SN74ACT32PW" H 3130 9555 50  0000 L CNN
 F 2 "Package_SO:TSSOP-14_4.4x5mm_P0.65mm" H 2900 9600 50  0001 C CNN
 F 3 "http://www.ti.com/lit/gpn/sn74LS32" H 2900 9600 50  0001 C CNN
@@
 P 2450 10550
 F 0 "U9" H 2680 10596 50  0000 L CNN
-F 1 "74ACT74" H 2680 10505 50  0000 L CNN
+F 1 "SN74ACT74D" H 2680 10505 50  0000 L CNN
 F 2 "Package_SO:SOIC-14_3.9x8.7mm_P1.27mm" H 2450 10550 50  0001 C CNN
 F 3 "74xx/74hc_hct74.pdf" H 2450 10550 50  0001 C CNN
@@
 P 10250 7600
 F 0 "U9" H 10000 7200 50  0000 C CNN
-F 1 "74ACT74" H 10100 7050 50  0000 C CNN
+F 1 "SN74ACT74D" H 10100 7050 50  0000 C CNN
 F 2 "Package_SO:SOIC-14_3.9x8.7mm_P1.27mm" H 10250 7600 50  0001 C CNN
 F 3 "74xx/74hc_hct74.pdf" H 10250 7600 50  0001 C CNN
@@
 P 5400 9500
 F 0 "U4" H 5400 9825 50  0000 C CNN
-F 1 "74ACT86" H 5400 9734 50  0000 C CNN
+F 1 "MC74ACT86DG" H 5400 9734 50  0000 C CNN
 F 2 "Package_SO:SOIC-14_3.9x8.7mm_P1.27mm" H 5400 9500 50  0001 C CNN
 F 3 "http://www.ti.com/lit/gpn/sn74HC86" H 5400 9500 50  0001 C CNN
@@
 P 12200 7600
 F 0 "U9" H 11800 7250 50  0000 C CNN
-F 1 "74ACT74" H 11900 7100 50  0000 C CNN
+F 1 "SN74ACT74D" H 11900 7100 50  0000 C CNN
 F 2 "Package_SO:SOIC-14_3.9x8.7mm_P1.27mm" H 12200 7600 50  0001 C CNN
 F 3 "74xx/74hc_hct74.pdf" H 12200 7600 50  0001 C CNN
@@
 P 5400 8950
 F 0 "U4" H 5400 9275 50  0000 C CNN
-F 1 "74ACT86" H 5400 9184 50  0000 C CNN
+F 1 "MC74ACT86DG" H 5400 9184 50  0000 C CNN
 F 2 "Package_SO:SOIC-14_3.9x8.7mm_P1.27mm" H 5400 8950 50  0001 C CNN
 F 3 "http://www.ti.com/lit/gpn/sn74HC86" H 5400 8950 50  0001 C CNN

Commit message: Logic-based control unit
Parts:
- removed C3, C4, C5: 0.1u, Capacitor_SMD:C_0805_2012Metric, symbol Device:C
- removed D2, D21: KP-2012CGCK, LED_SMD:LED_0805_2012Metric, symbol Device:LED
- removed R2, R21, R23, R24: 0, Resistor_SMD:R_0805_2012Metric, symbol Device:R
- removed R22, R25: 600, Resistor_SMD:R_0805_2012Metric, symbol Device:R
- removed U6, U7, U8: AT28C256-PLCC32, missing:PLCC-32_SMD_Socket, symbol missing:AT28C256-PLCC32
- added U10, U15: MC74ACT139DG, Package_SO:SOIC-16_3.9x9.9mm_P1.27mm, symbol 74xx:74LS139
- added U11, U12: SN74ACT08PW, Package_SO:TSSOP-14_4.4x5mm_P0.65mm, symbol 74xx:74LS08
- added U13, U16, U8: SN74ACT32PW, Package_SO:TSSOP-14_4.4x5mm_P0.65mm, symbol 74xx:74LS32
- added U14, U9: 74HC00, symbol 74xx:74HC00
- added U7: 74AHCT04, symbol 74xx:74AHCT04
- renumbered C7 to C3, D11 to D10, D12 to D11, D13 to D12, D14 to D13, D15 to D14, D16 to D15, D17 to D16, D18 to D17, D19 to D18, D20 to D19, D3 to D2, D4 to D3, D5 to D4, D6 to D5, D7 to D6, D8 to D7, D9 to D8, D10 to D9, H4 to H3, H3 to H4, R11 to R10, R12 to R11, R13 to R12, R14 to R13, R15 to R14, R16 to R15, R17 to R16, R18 to R17, R19 to R18, R20 to R19, R3 to R2, R4 to R3, R5 to R4, R6 to R5, R7 to R6, R8 to R7, R9 to R8, R10 to R9, U4 to U3, U3 to U4, U9 to U4, U3 to U6, U9 to U6
Connections:
- net labels added: flag_set, op_alu, op_jmp, op_ldi, supercycle, we_cycle, ~clear_we_cycle, ~ir2, ~is_alu, ~oe_alu_di, ~oe_d_di_a, ~oe_d_di_b, ~op_jmp, ~op_ld, ~op_ldi, ~op_st, ~rst_supercycle, ~set_we_cycle, ~supercycle, ~we_a, ~we_b, ~we_cycle
- net labels removed: s1, s1_d, s2, s2_d, ~mem_rdy, ~oe_alu, ~reset_cycle
- wire segments 56 -> 118
- no-connect marks 10 -> 14
Other:
- note removed: "A"
- note removed: "B"
- note removed: "C"
- note removed: "Install one of resistors to select clock source"
- moved on the sheet: C1, C2, C3, D1, D10, D11, D12, D13, D14, D15, D16, D17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

Commit message: New control unit schematics
Parts:
- added C10, C5, C6, C7, C8, C9: 0.1u, Capacitor_SMD:C_0805_2012Metric, symbol Device:C
- added D20, D21, D22: KP-2012CGCK, LED_SMD:LED_0805_2012Metric, symbol Device:LED
- added R20, R21, R22: 600, Resistor_SMD:R_0805_2012Metric, symbol Device:R
- U14, U9: value 74HC00 -> 74ACT00MTCX; footprint (none) -> Package_SO:TSSOP-14_4.4x5mm_P0.65mm
- U7: value 74AHCT04 -> 74ACT04MTCX; footprint (none) -> Package_SO:TSSOP-14_4.4x5mm_P0.65mm
Connections:
- net labels added: ~p_selector
- wire segments 118 -> 122
- no-connect marks 14 -> 13
Other:
- moved on the sheet: C1, C2, C3, D10, D11, D12, D13, D14, D15, D16, D17, D18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

Commit message: Board adjustments
Parts:
- U7: value 74ACT04MTCX -> SN74ACT04PW
Changed lines of the file:
@@
 P 5250 1000
 F 0 "U7" H 5250 1317 50  0000 C CNN
-F 1 "74ACT04MTCX" H 5250 1226 50  0000 C CNN
+F 1 "SN74ACT04PW" H 5250 1226 50  0000 C CNN
 F 2 "Package_SO:TSSOP-14_4.4x5mm_P0.65mm" H 5250 1000 50  0001 C CNN
 F 3 "https://assets.nexperia.com/documents/data-sheet/74AHC_AHCT04.pdf" H 5250 1000 50  0001 C CNN
@@
 P 6200 2450
 F 0 "U7" H 6200 2767 50  0000 C CNN
-F 1 "74ACT04MTCX" H 6200 2676 50  0000 C CNN
+F 1 "SN74ACT04PW" H 6200 2676 50  0000 C CNN
 F 2 "Package_SO:TSSOP-14_4.4x5mm_P0.65mm" H 6200 2450 50  0001 C CNN
 F 3 "https://assets.nexperia.com/documents/data-sheet/74AHC_AHCT04.pdf" H 6200 2450 50  0001 C CNN
@@
 P 6200 2950
 F 0 "U7" H 6200 3267 50  0000 C CNN
-F 1 "74ACT04MTCX" H 6200 3176 50  0000 C CNN
+F 1 "SN74ACT04PW" H 6200 3176 50  0000 C CNN
 F 2 "Package_SO:TSSOP-14_4.4x5mm_P0.65mm" H 6200 2950 50  0001 C CNN
 F 3 "https://assets.nexperia.com/documents/data-sheet/74AHC_AHCT04.pdf" H 6200 2950 50  0001 C CNN
@@
 P 7800 8450
 F 0 "U7" H 7800 8767 50  0000 C CNN
-F 1 "74ACT04MTCX" H 7800 8676 50  0000 C CNN
+F 1 "SN74ACT04PW" H 7800 8676 50  0000 C CNN
 F 2 "Package_SO:TSSOP-14_4.4x5mm_P0.65mm" H 7800 8450 50  0001 C CNN
 F 3 "https://assets.nexperia.com/documents/data-sheet/74AHC_AHCT04.pdf" H 7800 8450 50  0001 C CNN
@@
 P 12200 8250
 F 0 "U7" H 12200 8567 50  0000 C CNN
-F 1 "74ACT04MTCX" H 12200 8476 50  0000 C CNN
+F 1 "SN74ACT04PW" H 12200 8476 50  0000 C CNN
 F 2 "Package_SO:TSSOP-14_4.4x5mm_P0.65mm" H 12200 8250 50  0001 C CNN
 F 3 "https://assets.nexperia.com/documents/data-sheet/74AHC_AHCT04.pdf" H 12200 8250 50  0001 C CNN
@@
 P 2450 4150
 F 0 "U7" H 2450 4467 50  0000 C CNN
-F 1 "74ACT04MTCX" H 2450 4376 50  0000 C CNN
+F 1 "SN74ACT04PW" H 2450 4376 50  0000 C CNN
 F 2 "Package_SO:TSSOP-14_4.4x5mm_P0.65mm" H 2450 4150 50  0001 C CNN
 F 3 "https://assets.nexperia.com/documents/data-sheet/74AHC_AHCT04.pdf" H 2450 4150 50  0001 C CNN
@@
 P 4200 15200
 F 0 "U7" H 4430 15246 50  0000 L CNN
-F 1 "74ACT04MTCX" H 4430 15155 50  0000 L CNN
+F 1 "SN74ACT04PW" H 4430 15155 50  0000 L CNN
 F 2 "Package_SO:TSSOP-14_4.4x5mm_P0.65mm" H 4200 15200 50  0001 C CNN
 F 3 "https://assets.nexperia.com/documents/data-sheet/74AHC_AHCT04.pdf" H 4200 15200 50  0001 C CNN
