File: boards/control/interface.sch (KiCad schematic (older format))
At the start: 2 parts, among them J2 CU

Commit message: Part names
Parts:
- J2: value CU -> 61304021021
Changed lines of the file:
@@
 P 5850 3700
 F 0 "J2" H 5900 4817 50  0000 C CNN
-F 1 "CU" H 5900 4726 50  0000 C CNN
+F 1 "61304021021" H 5900 4726 50  0000 C CNN
 F 2 "Connector_PinHeader_2.54mm:PinHeader_2x20_P2.54mm_Horizontal" H 5850 3700 50  0001 C CNN
 F 3 "~" H 5850 3700 50  0001 C CNN

Commit message: Logic-based control unit
Parts:
- renumbered C6 to C4, J2 to J1
Connections:
- net ~mem_rdy: no longer names the net of J1.26 (Pin_26)
- no-connect marks 3 -> 4
Changed lines of the file:
@@
 Text HLabel 4700 3550 0    50   Output ~ 0
 flags[0..3]
-Text HLabel 6250 4000 2    50   Output ~ 0
-~mem_rdy
 Text HLabel 6250 4600 2    50   Input ~ 0
 ~we_mem
@@
 ~oe_b_alu
 $Comp
-L Connector_Generic:Conn_02x20_Odd_Even J2
+L Connector_Generic:Conn_02x20_Odd_Even J1
 U 1 1 5EDA71CD
 P 5850 3700
-F 0 "J2" H 5900 4817 50  0000 C CNN
+F 0 "J1" H 5900 4817 50  0000 C CNN
 F 1 "61304021021" H 5900 4726 50  0000 C CNN
 F 2 "Connector_PinHeader_2.54mm:PinHeader_2x20_P2.54mm_Horizontal" H 5850 3700 50  0001 C CNN
@@
 $EndComp
 $Comp
-L power:VCC #PWR0190
+L power:VCC #PWR060
 U 1 1 5EDAB67E
 P 5650 2800
-F 0 "#PWR0190" H 5650 2650 50  0001 C CNN
+F 0 "#PWR060" H 5650 2650 50  0001 C CNN
 F 1 "VCC" V 5668 2927 50  0000 L CNN
 F 2 "" H 5650 2800 50  0001 C CNN
@@
 $EndComp
 $Comp
-L power:VCC #PWR0193
+L power:VCC #PWR063
 U 1 1 5EDABE71
 P 6150 4700
-F 0 "#PWR0193" H 6150 4550 50  0001 C CNN
+F 0 "#PWR063" H 6150 4550 50  0001 C CNN
 F 1 "VCC" V 6167 4828 50  0000 L CNN
 F 2 "" H 6150 4700 50  0001 C CNN
@@
 $EndComp
 $Comp
-L power:GND #PWR0191
+L power:GND #PWR061
 U 1 1 5EDAC68A
 P 5650 4700
-F 0 "#PWR0191" H 5650 4450 50  0001 C CNN
+F 0 "#PWR061" H 5650 4450 50  0001 C CNN
 F 1 "GND" V 5655 4572 50  0000 R CNN
 F 2 "" H 5650 4700 50  0001 C CNN
@@
 $EndComp
 $Comp
-L power:GND #PWR0192
+L power:GND #PWR062
 U 1 1 5EDACBD5
 P 6150 2800
-F 0 "#PWR0192" H 6150 2550 50  0001 C CNN
+F 0 "#PWR062" H 6150 2550 50  0001 C CNN
 F 1 "GND" V 6155 2672 50  0000 R CNN
 F 2 "" H 6150 2800 50  0001 C CNN
@@
 $EndComp
 $Comp
-L power:GND #PWR079
+L power:GND #PWR067
 U 1 1 5FFEF396
 P 8550 3100
-F 0 "#PWR079" H 8550 2850 50  0001 C CNN
+F 0 "#PWR067" H 8550 2850 50  0001 C CNN
 F 1 "GND" V 8555 2972 50  0000 R CNN
 F 2 "" H 8550 3100 50  0001 C CNN
@@
 $EndComp
 $Comp
-L power:VCC #PWR076
+L power:VCC #PWR064
 U 1 1 5FFEFB40
 P 8100 3100
-F 0 "#PWR076" H 8100 2950 50  0001 C CNN
+F 0 "#PWR064" H 8100 2950 50  0001 C CNN
 F 1 "VCC" V 8118 3227 50  0000 L CNN
 F 2 "" H 8100 3100 50  0001 C CNN
@@
 $EndComp
 $Comp
-L Device:CP C6
+L Device:CP C4
 U 1 1 5FFF064D
 P 8200 3950
-F 0 "C6" H 8318 3996 50  0000 L CNN
+F 0 "C4" H 8318 3996 50  0000 L CNN
 F 1 "10u 6.3v" H 8318 3905 50  0000 L CNN
 F 2 "Capacitor_SMD:CP_Elec_4x4.5" H 8238 3800 50  0001 C CNN
@@
 $EndComp
 $Comp
-L power:GND #PWR078
+L power:GND #PWR066
 U 1 1 5FFF0D8B
 P 8200 4100
-F 0 "#PWR078" H 8200 3850 50  0001 C CNN
+F 0 "#PWR066" H 8200 3850 50  0001 C CNN
 F 1 "GND" V 8205 3972 50  0000 R CNN
 F 2 "" H 8200 4100 50  0001 C CNN
@@
 $EndComp
 $Comp
-L power:VCC #PWR077
+L power:VCC #PWR065
 U 1 1 5FFF1304
 P 8200 3800
-F 0 "#PWR077" H 8200 3650 50  0001 C CNN
+F 0 "#PWR065" H 8200 3650 50  0001 C CNN
 F 1 "VCC" V 8218 3927 50  0000 L CNN
 F 2 "" H 8200 3800 50  0001 C CNN
@@
 	1    0    0    -1
 $EndComp
+NoConn ~ 6250 4000
 Wire Bus Line
 	4800 3700 4800 3850

Commit message: Change control unit schematics to support wait cycles (not checked)
Connections:
- net ~mem_rdy: now reaches J1.26 (Pin_26)
- no-connect marks 4 -> 3
Changed lines of the file:
@@
 Sheet 2 2
 Title "Interface connector"
-Date "2020-01-25"
-Rev "1"
+Date "2020-11-29"
+Rev "3"
 Comp ""
 Comment1 "Licensed under the TAPR Open Hardware License (www.tapr.org/OHL)"
@@
 	4800 3550 4800 3600
 Wire Wire Line
-	6250 4000 6150 4000
-Wire Wire Line
 	6150 4100 6250 4100
 NoConn ~ 5650 4000
@@
 	1    0    0    -1
 $EndComp
-NoConn ~ 6250 4000
+Text HLabel 6250 4000 2    50   Output ~ 0
+~mem_rdy
+Wire Wire Line
+	6150 4000 6250 4000
 Wire Bus Line
 	4800 3700 4800 3850

Commit message: Control: change big capacitor footprint
Parts:
- C4: value 10u 6.3v -> TPSB336K010T0425; footprint Capacitor_SMD:CP_Elec_4x4.5 -> Capacitor_Tantalum_SMD:CP_EIA-3528-21_Kemet-B_Pad1.50x2.35mm_HandSolder
Changed lines of the file:
@@
 P 8200 3950
 F 0 "C4" H 8318 3996 50  0000 L CNN
-F 1 "10u 6.3v" H 8318 3905 50  0000 L CNN
-F 2 "Capacitor_SMD:CP_Elec_4x4.5" H 8238 3800 50  0001 C CNN
+F 1 "TPSB336K010T0425" H 8318 3905 50  0000 L CNN
+F 2 "Capacitor_Tantalum_SMD:CP_EIA-3528-21_Kemet-B_Pad1.50x2.35mm_HandSolder" H 8238 3800 50  0001 C CNN
 F 3 "~" H 8200 3950 50  0001 C CNN
 	1    8200 3950
