File: boards/alu/interface.sch (KiCad schematic (older format))
At the start: 1 part, among them J1 ALU

Commit message: Part names
Parts:
- J1: value ALU -> 61304021021
Changed lines of the file:
@@
 AR Path="/5FC3F1F0/5FC3FB3E" Ref="J1"  Part="1"
 F 0 "J1" H 5300 4417 50  0000 C CNN
-F 1 "ALU" H 5300 4326 50  0000 C CNN
+F 1 "61304021021" H 5300 4326 50  0000 C CNN
 F 2 "Connector_PinHeader_2.54mm:PinHeader_2x20_P2.54mm_Horizontal" H 5250 3300 50  0001 C CNN
 F 3 "~" H 5250 3300 50  0001 C CNN
