File: boards/alu/adder.sch (KiCad schematic (older format))
At the start: 20 parts, among them U22 74HC86, U23 74HC86, U24 74HC86, U25 74HC86, U26 74HC86, U27 74HC86, U28 74HC86, U29 74HC86, U30 74LS08, U31 74LS08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

Commit message: Footprints and part names
Parts:
- C4, C5, C6, C7, C8, C9: footprint (none) -> Capacitor_SMD:C_0805_2012Metric
- U22, U23, U24, U25, U26, U27, U28, U29: value 74HC86 -> MC74ACT86DG; footprint (none) -> Package_SO:SOIC-14_3.9x8.7mm_P1.27mm
- U30, U31, U32, U33: value 74LS08 -> SN74ACT08PW; footprint (none) -> Package_SO:TSSOP-14_4.4x5mm_P0.65mm
- U34, U35: value 74LS32 -> 74ACT32MTCX; footprint (none) -> Package_SO:TSSOP-14_4.4x5mm_P0.65mm
