File: boards/alu/alu.sch (KiCad schematic (older format))
At the start: 80 parts, among them U1 AT28C256-PLCC32, U2 SN74ACT08PW, U3 AT28C256-PLCC32, U4 74ACT00MTCX, U5 MC74ACT02DTR2G

Commit message: ALU model + sch
Parts:
- removed C1, C2: 0.1u, Capacitor_SMD:C_0805_2012Metric, symbol Device:C
- removed U1, U3: AT28C256-PLCC32, missing:PLCC-32_SMD_Socket, symbol missing:AT28C256-PLCC32
- removed U4: 74ACT00MTCX, Package_SO:TSSOP-14_4.4x5mm_P0.65mm, symbol 74xx:74HC00
- added U1, U15, U38: SN74ACT08PW, Package_SO:TSSOP-14_4.4x5mm_P0.65mm, symbol 74xx:74LS08
- added U10, U16, U17, U18, U19, U20, U3: 74ACT244MTC, symbol 74xx:74HC244
- added U11, U8, U9: 74LS32, symbol 74xx:74LS32
- added U12: 74LS138, symbol 74xx:74LS138
- added unit 1 of U13
- added unit 2 of U13
- added unit 3 of U2
- added unit 4 of U2
- added unit 5 of U2
- added U21: SN74ACT240PWR, symbol 74xx:74HC240
- added U36: 74HC86, symbol 74xx:74HC86
- added U37: MC74ACT02DTR2G, Package_SO:TSSOP-14_4.4x5mm_P0.65mm, symbol 74xx:74LS02
- added U4, U5, U6, U7: MC74AC157DR2G, symbol 74xx:74LS157
- renumbered C3 to C1, C4 to C2, C5 to C3, D29 to D25, D30 to D26, D31 to D27, D32 to D28, D33 to D29, D25 to D30, D26 to D31, D27 to D32, D28 to D33, R29 to R25, R30 to R26, R31 to R27, R32 to R28, R33 to R29, R25 to R30, R26 to R31, R27 to R32, R28 to R33, U2 to U13, U5 to U14
Connections:
- net GND: now also U1.7 (GND), U10.10 (GND), U11.7 (GND), U12.8 (GND), U15.7 (GND), U16.10 (GND), U17.10 (GND), U18.10 (GND), U18.2 (1A0), U19.10 (GND), U2.7 (GND), U20.10 (GND), U21.10 (GND), U3.10 (GND), U36.7 (GND), U37.7 (GND), U38.7 (GND), U4.8 (GND), U5.8 (GND), U6.8 (GND), U7.8 (GND), U8.7 (GND), U9.7 (GND)
- net VCC: now also U1.14 (VCC), U10.20 (VCC), U11.14 (VCC), U12.16 (VCC), U12.6 (E3), U15.14 (VCC), U16.20 (VCC), U17.20 (VCC), U18.20 (VCC), U19.20 (VCC), U2.14 (VCC), U20.20 (VCC), U21.20 (VCC), U3.20 (VCC), U36.10, U36.13, U36.14 (VCC), U37.14 (VCC), U38.14 (VCC), U4.16 (VCC), U5.16 (VCC), U6.16 (VCC), U7.16 (VCC), U8.14 (VCC), U9.14 (VCC)
- net a0: now also U4.2 (I0a), U6.3 (I1a)
- net a1: now also U4.5 (I0b), U6.6 (I1b)
- net a2: now also U4.11 (I0c), U6.10 (I1c)
- net a3: now also U4.14 (I0d), U6.13 (I1d)
- net a4: now also U5.2 (I0a), U7.3 (I1a)
- net a5: now also U5.5 (I0b), U7.6 (I1b)
- net a6: now also U5.11 (I0c), U7.10 (I1c)
- net a7: now also U5.14 (I0d), U7.13 (I1d)
- net b0: now also U4.3 (I1a), U6.2 (I0a)
- net b1: now also U4.6 (I1b), U6.5 (I0b)
- net b2: now also U4.10 (I1c), U6.11 (I0c)
- net b3: now also U4.13 (I1d), U6.14 (I0d)
- net b4: now also U5.3 (I1a), U7.2 (I0a)
- net b5: now also U5.6 (I1b), U7.5 (I0b)
- net b6: now also U5.10 (I1c), U7.11 (I0c)
- net b7: now also U5.13 (I1d), U7.14 (I0d)
- net carry_in: now also U13.1, U20.11 (2A3), U20.13 (2A2), U20.15 (2A1), U20.17 (2A0), U20.2 (1A0), U20.4 (1A1), U20.6 (1A2), U20.8 (1A3)
- net flags0: now also U13.6
- net flags1: now also U11.8
- net flags2: now also U10.9 (2Y3), U16.9 (2Y3), U17.9 (2Y3), U18.9 (2Y3), U19.9 (2Y3), U20.9 (2Y3), U21.9 (2Y3), U3.9 (2Y3)
- net flags3: now also U36.6
- net invert: now also U36.1
- net op0: now also U12.1 (A0), U15.1, U37.2, U37.6
- net op1: now also U12.2 (A1), U15.2, U37.3, U37.8, U37.9
- net op3: now also U12.5 (E2), U15.13, U36.9, U38.10; no longer U2.1
- net r0: now also U10.18 (1Y0), U16.18 (1Y0), U17.18 (1Y0), U18.18 (1Y0), U19.18 (1Y0), U20.18 (1Y0), U21.18 (1Y0), U3.18 (1Y0)
- net r1: now also U10.16 (1Y1), U16.16 (1Y1), U17.16 (1Y1), U18.16 (1Y1), U19.16 (1Y1), U20.16 (1Y1), U21.16 (1Y1), U3.16 (1Y1)
- net r2: now also U10.14 (1Y2), U16.14 (1Y2), U17.14 (1Y2), U18.14 (1Y2), U19.14 (1Y2), U20.14 (1Y2), U21.14 (1Y2), U3.14 (1Y2)
- net r3: now also U10.12 (1Y3), U16.12 (1Y3), U17.12 (1Y3), U18.12 (1Y3), U19.12 (1Y3), U20.12 (1Y3), U21.12 (1Y3), U3.12 (1Y3)
- net r4: now also U10.3 (2Y0), U16.3 (2Y0), U17.3 (2Y0), U18.3 (2Y0), U19.3 (2Y0), U20.3 (2Y0), U21.3 (2Y0), U3.3 (2Y0)
- net r5: now also U10.5 (2Y1), U16.5 (2Y1), U17.5 (2Y1), U18.5 (2Y1), U19.5 (2Y1), U20.5 (2Y1), U21.5 (2Y1), U3.5 (2Y1)
- net r6: now also U10.7 (2Y2), U16.7 (2Y2), U17.7 (2Y2), U18.7 (2Y2), U19.7 (2Y2), U20.7 (2Y2), U21.7 (2Y2), U3.7 (2Y2)
- net z03: now also U13.4
- net z47: now also U13.5
- net ~oe: now also U11.5, U12.4 (E1)
- net ~op3: now also U11.4, U36.8; no longer U2.4
- net from_hi: no longer names the net of U2.3
- net from_hi: now also U3.17 (2A0)
- net from_lo: no longer names the net of U2.6
- net from_lo: now also U3.15 (2A1)
- net op2 renamed adder_sub
- net adder_sub: now also U12.3 (A2), U15.9
- net to_hi renamed adder_b5
- net adder_b5: now also U21.15 (2A1), U7.7 (Zb), U9.5
- net to_lo renamed adder_b4
- net adder_b4: now also U21.17 (2A0), U7.4 (Za), U9.2
- new net: U15.6, U19.11 (2A3)
- new net: U1.3, U3.2 (1A0)
- new net: U1.6, U3.4 (1A1)
- new net: U1.8, U3.6 (1A2)
- new net: U1.11, U3.8 (1A3)
- new net: U2.8, U3.13 (2A2)
- new net: U2.11, U3.11 (2A3)
- new net: U10.11 (2A3), U9.11
- new net: U10.13 (2A2), U9.8
- new net: U10.15 (2A1), U9.6
- new net: U10.17 (2A0), U9.3
- new net: U10.2 (1A0), U8.3
- new net: U10.4 (1A1), U8.6
- new net: U10.6 (1A2), U8.8
- new net: U10.8 (1A3), U8.11
- new net: U12.7 (O7), U38.13
- new net adder_b0: U11.3
- new net adder_b1: U1.5, U21.4 (1A1), U6.7 (Zb), U8.5
- new net adder_b2: U1.10, U21.6 (1A2), U6.9 (Zc), U8.10
- new net adder_b3: U1.13, U21.8 (1A3), U6.12 (Zd), U8.13
- new net adder_b6: U2.10, U21.13 (2A2), U7.9 (Zc), U9.10
- new net adder_b7: U2.13, U21.11 (2A3), U7.12 (Zd), U9.13
- new net adder_b_one: U11.1, U15.12, U15.3
- new net adder_c6_out: U36.4
- new net adder_c_in: U13.3
- new net adder_c_out: U36.5, U38.9
- new net adder_carry_ena: U13.2, U37.4
- new net adder_r0: U16.2 (1A0)
- new net adder_r1: U16.4 (1A1)
- new net adder_r2: U16.6 (1A2)
- new net adder_r3: U16.8 (1A3)
- new net adder_r4: U16.17 (2A0)
- new net adder_r5: U16.15 (2A1)
- new net adder_r6: U16.13 (2A2)
- new net adder_r7: U16.11 (2A3)
- new net c_adder: U11.9, U38.8
- new net c_sh: U11.10, U11.11
- new net c_shl: U11.13, U38.6
- new net c_shr: U11.12, U38.3
- new net int_swap: U15.8, U36.2
- new net sa0: U1.1, U18.4 (1A1), U38.2, U4.4 (Za), U8.1
- new net sa1: U1.4, U18.6 (1A2), U19.2 (1A0), U4.7 (Zb), U8.4
- new net sa2: U1.9, U18.8 (1A3), U19.4 (1A1), U4.9 (Zc), U8.9
- new net sa3: U1.12, U18.17 (2A0), U19.6 (1A2), U4.12 (Zd), U8.12
- new net sa4: U18.15 (2A1), U19.8 (1A3), U2.1, U5.4 (Za), U9.1
- new net sa5: U18.13 (2A2), U19.17 (2A0), U2.4, U5.7 (Zb), U9.4
- new net sa6: U18.11 (2A3), U19.15 (2A1), U2.9, U5.9 (Zc), U9.9
- new net sa7: U15.5, U19.13 (2A2), U2.12, U38.5, U5.12 (Zd), U9.12
- new net sar_ena: U12.9 (O6), U15.4, U38.12
- new net sb0: U1.2, U11.2, U21.2 (1A0), U6.4 (Za), U8.2
- new net shl_oe: U37.13, U38.4
- new net shr_oe: U36.11, U38.1
- new net swap: U36.3, U4.1 (S), U5.1 (S), U6.1 (S), U7.1 (S)
- new net xor_r0: U17.2 (1A0)
- new net xor_r1: U17.4 (1A1)
- new net xor_r2: U17.6 (1A2)
- new net xor_r3: U17.8 (1A3)
- new net xor_r4: U17.17 (2A0)
- new net xor_r5: U17.15 (2A1)
- new net xor_r6: U17.13 (2A2)
- new net xor_r7: U17.11 (2A3)
- new net ~adder_oe: U11.6, U16.1 (1OE), U16.19 (2OE)
- new net ~and_oe: U12.14 (O1), U3.1 (1OE), U3.19 (2OE)
- new net ~exp_oe: U12.15 (O0), U20.1 (1OE), U20.19 (2OE)
- new net ~not_oe: U12.11 (O4), U21.1 (1OE), U21.19 (2OE)
- new net ~op1: U37.10, U37.5
- new net ~or_oe: U10.1 (1OE), U10.19 (2OE), U12.13 (O2)
- new net ~sa_ena: U15.10, U37.1, U4.15 (E), U5.15 (E)
- new net ~sb_ena: U15.11, U6.15 (E), U7.15 (E)
- new net ~shl_oe: U12.12 (O3), U18.1 (1OE), U18.19 (2OE), U37.11, U37.12
- new net ~shr_oe: U19.1 (1OE), U19.19 (2OE), U36.12, U38.11
- new net ~xor_oe: U12.10 (O5), U17.1 (1OE), U17.19 (2OE)
- no-connect marks 3 -> 0
Other:
- moved on the sheet: C1, C2, C3, D1, D10, D11, D12, D13, D14, D15, D16, D17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

Commit message: Footprints and part names
Parts:
- added C? (x2): 0.1u, Capacitor_SMD:C_0805_2012Metric, symbol Device:C
- U10, U16, U17, U18, U19, U20, U21, U3: footprint (none) -> Package_SO:TSSOP-20_4.4x6.5mm_P0.65mm
- U11, U8, U9: value 74LS32 -> 74ACT32MTCX; footprint (none) -> Package_SO:TSSOP-14_4.4x5mm_P0.65mm
- U12: value 74LS138 -> MC74ACT138DTR2G; footprint (none) -> Package_SO:TSSOP-16_4.4x5mm_P0.65mm
- U36: value 74HC86 -> MC74ACT86DG; footprint (none) -> Package_SO:SOIC-14_3.9x8.7mm_P1.27mm
- U4, U5, U6, U7: footprint (none) -> Package_SO:SOIC-16_3.9x9.9mm_P1.27mm
Connections:
- net GND: now also C?.2, C?.2
- net VCC: now also C?.1, C?.1

Commit message: ALU board started
Parts:
- removed D1, D10, D11, D12, D13, D14, D15, D16, D2, D3, D4, D5, D6, D7, D8, D9: KP-2012CGCK, LED_SMD:LED_0805_2012Metric, symbol Device:LED
- removed D17, D18, D19, D20, D21, D22, D23, D24: KP-2012EC, LED_SMD:LED_0805_2012Metric, symbol Device:LED
- removed R1, R10, R11, R12, R13, R14, R15, R16, R2, R3, R4, R5, R6, R7, R8, R9: 600, Resistor_SMD:R_0805_2012Metric, symbol Device:R
- removed R17, R18, R19, R20, R21, R22, R23, R24: 620, Resistor_SMD:R_0805_2012Metric, symbol Device:R
- gave numbers to parts that had none: 2
Connections:
- net a0: now also U6.6 (I1b); no longer U6.3 (I1a)
- net a1: now also U6.3 (I1a); no longer U6.6 (I1b)
- net a2: now also U6.13 (I1d); no longer U6.10 (I1c)
- net a3: now also U6.10 (I1c); no longer U6.13 (I1d)
- net a4: now also U7.6 (I1b); no longer U7.3 (I1a)
- net a5: now also U7.3 (I1a); no longer U7.6 (I1b)
- net a6: now also U7.13 (I1d); no longer U7.10 (I1c)
- net a7: now also U7.10 (I1c); no longer U7.13 (I1d)
- net adder_b1: now also U2.5, U21.15 (2A1), U6.4 (Za), U9.5; no longer U1.5, U21.4 (1A1), U6.7 (Zb), U8.5
- net adder_b2: now also U2.10, U21.13 (2A2), U6.12 (Zd), U9.10; no longer U1.10, U21.6 (1A2), U6.9 (Zc), U8.10
- net adder_b3: now also U2.13, U21.11 (2A3), U6.9 (Zc), U9.13; no longer U1.13, U21.8 (1A3), U6.12 (Zd), U8.13
- net adder_b4: now also U1.2, U21.2 (1A0), U7.7 (Zb), U8.2; no longer U2.2, U21.17 (2A0), U7.4 (Za), U9.2
- net adder_b5: now also U1.5, U21.4 (1A1), U7.4 (Za), U8.5; no longer U2.5, U21.15 (2A1), U7.7 (Zb), U9.5
- net adder_b6: now also U1.10, U21.6 (1A2), U7.12 (Zd), U8.10; no longer U2.10, U21.13 (2A2), U7.9 (Zc), U9.10
- net adder_b7: now also U1.13, U21.8 (1A3), U7.9 (Zc), U8.13; no longer U2.13, U21.11 (2A3), U7.12 (Zd), U9.13
- net adder_r0: now also U16.17 (2A0); no longer U16.2 (1A0)
- net adder_r1: now also U16.15 (2A1); no longer U16.4 (1A1)
- net adder_r2: now also U16.13 (2A2); no longer U16.6 (1A2)
- net adder_r3: now also U16.11 (2A3); no longer U16.8 (1A3)
- net adder_r4: now also U16.2 (1A0); no longer U16.17 (2A0)
- net adder_r5: now also U16.4 (1A1); no longer U16.15 (2A1)
- net adder_r6: now also U16.6 (1A2); no longer U16.13 (2A2)
- net adder_r7: now also U16.8 (1A3); no longer U16.11 (2A3)
- net b0: now also U6.5 (I0b); no longer U6.2 (I0a)
- net b1: now also U6.2 (I0a); no longer U6.5 (I0b)
- net b2: now also U6.14 (I0d); no longer U6.11 (I0c)
- net b3: now also U6.11 (I0c); no longer U6.14 (I0d)
- net b4: now also U7.5 (I0b); no longer U7.2 (I0a)
- net b5: now also U7.2 (I0a); no longer U7.5 (I0b)
- net b6: now also U7.14 (I0d); no longer U7.11 (I0c)
- net b7: now also U7.11 (I0c); no longer U7.14 (I0d)
- net flags2: now also U10.12 (1Y3), U14.6, U16.12 (1Y3), U19.12 (1Y3), U21.12 (1Y3), U3.12 (1Y3); no longer U10.9 (2Y3), U14.12, U16.9 (2Y3), U19.9 (2Y3), U21.9 (2Y3), U3.9 (2Y3)
- net nor01: now also U14.10; no longer U14.1
- net nor23: now also U14.13; no longer U14.4
- net nor45: now also U13.13, U14.1; no longer U13.12, U14.10
- net nor67: now also U13.12, U14.4; no longer U13.13, U14.13
- net r0: now also U10.3 (2Y0), U14.8, U16.3 (2Y0), U19.3 (2Y0), U21.3 (2Y0), U3.3 (2Y0); no longer U10.18 (1Y0), U14.2, U16.18 (1Y0), U19.18 (1Y0), U21.18 (1Y0), U3.18 (1Y0)
- net r1: now also U10.5 (2Y1), U14.9, U16.5 (2Y1), U19.5 (2Y1), U21.5 (2Y1), U3.5 (2Y1); no longer U10.16 (1Y1), U14.3, U16.16 (1Y1), U19.16 (1Y1), U21.16 (1Y1), U3.16 (1Y1)
- net r2: now also U10.7 (2Y2), U14.11, U16.7 (2Y2), U19.7 (2Y2), U21.7 (2Y2), U3.7 (2Y2); no longer U10.14 (1Y2), U14.5, U16.14 (1Y2), U19.14 (1Y2), U21.14 (1Y2), U3.14 (1Y2)
- net r3: now also U10.9 (2Y3), U14.12, U16.9 (2Y3), U19.9 (2Y3), U21.9 (2Y3), U3.9 (2Y3); no longer U10.12 (1Y3), U14.6, U16.12 (1Y3), U19.12 (1Y3), U21.12 (1Y3), U3.12 (1Y3)
- net r4: now also U10.18 (1Y0), U14.2, U16.18 (1Y0), U19.18 (1Y0), U21.18 (1Y0), U3.18 (1Y0); no longer U10.3 (2Y0), U14.8, U16.3 (2Y0), U19.3 (2Y0), U21.3 (2Y0), U3.3 (2Y0)
- net r5: now also U10.16 (1Y1), U14.3, U16.16 (1Y1), U19.16 (1Y1), U21.16 (1Y1), U3.16 (1Y1); no longer U10.5 (2Y1), U14.9, U16.5 (2Y1), U19.5 (2Y1), U21.5 (2Y1), U3.5 (2Y1)
- net r6: now also U10.14 (1Y2), U14.5, U16.14 (1Y2), U19.14 (1Y2), U21.14 (1Y2), U3.14 (1Y2); no longer U10.7 (2Y2), U14.11, U16.7 (2Y2), U19.7 (2Y2), U21.7 (2Y2), U3.7 (2Y2)
- net sa0: now also U2.1, U9.1; no longer U1.1, U8.1
- net sa1: now also U19.17 (2A0), U2.4, U9.4; no longer U1.4, U19.2 (1A0), U8.4
- net sa2: now also U19.15 (2A1), U2.9, U9.9; no longer U1.9, U19.4 (1A1), U8.9
- net sa3: now also U19.13 (2A2), U2.12, U9.12; no longer U1.12, U19.6 (1A2), U8.12
- net sa4: now also U1.1, U19.11 (2A3), U8.1; no longer U19.8 (1A3), U2.1, U9.1
- net sa5: now also U1.4, U19.2 (1A0), U8.4; no longer U19.17 (2A0), U2.4, U9.4
- net sa6: now also U1.9, U19.4 (1A1), U8.9; no longer U19.15 (2A1), U2.9, U9.9
- net sa7: now also U1.12, U19.6 (1A2), U8.12; no longer U19.13 (2A2), U2.12, U9.12
- net sb0: now also U2.2, U21.17 (2A0), U6.7 (Zb), U9.2; no longer U1.2, U21.2 (1A0), U6.4 (Za), U8.2
- net z03: now also U13.5; no longer U13.4
- net z47: now also U13.4; no longer U13.5
- net at U15.6: now also U19.8 (1A3); no longer U19.11 (2A3)
Other:
- moved on the sheet: U15B

Commit message: VCC and GND tracks
Parts:
- removed D26, D27, D28: KP-2012EC, LED_SMD:LED_0805_2012Metric, symbol Device:LED
- removed D29, D30, D31, D32, D33: KP-2012CGCK, LED_SMD:LED_0805_2012Metric, symbol Device:LED
- removed R26, R27, R28: 620, Resistor_SMD:R_0805_2012Metric, symbol Device:R
- removed R29, R30, R31, R32, R33: 600, Resistor_SMD:R_0805_2012Metric, symbol Device:R
- added D1, D2, D3, D4, D5, D6, D7: KP-2012EC, LED_SMD:LED_0805_2012Metric, symbol Device:LED
- added R1, R2, R3, R4, R5, R6, R7: 620, Resistor_SMD:R_0805_2012Metric, symbol Device:R
- renumbered D25 to D8, R25 to R8
Connections:
- net GND: no longer R8.1
- net VCC: now also R8.1, R1.1, R2.1, R3.1, R4.1, R5.1, R6.1, R7.1
- net flags0: no longer D8.2 (A)
- net ~adder_oe: now also D3.2 (A)
- net ~and_oe: now also D1.2 (A)
- net ~exp_oe: now also D5.2 (A)
- net ~not_oe: now also D8.2 (A)
- net ~or_oe: now also D2.2 (A)
- net ~shl_oe: now also D6.2 (A)
- net ~shr_oe: now also D7.2 (A)
- net ~xor_oe: now also D4.2 (A)
- new net: D3.1 (K), R3.2
- new net: D4.1 (K), R4.2
- new net: D6.1 (K), R6.2
- new net: D7.1 (K), R7.2
- new net: D5.1 (K), R5.2
- new net: D2.1 (K), R2.2
- new net: D1.1 (K), R1.2
Other:
- moved on the sheet: D8, R8
