File: boards/alu/alu.sch (KiCad schematic (older format))
At the start: 49 parts, among them U1 SN74ACT08PW, U10 74ACT244MTC, U11 74ACT32MTCX, U12 MC74ACT138DTR2G, U13 SN74ACT08PW, U14 MC74ACT02DTR2G, U15 SN74ACT08PW, U16 74ACT244MTC, U17 74ACT244MTC, U18 74ACT244MTC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

Commit message: ALU board: change capacitor footprint, show labels
Parts:
- C3: footprint Capacitor_SMD:CP_Elec_4x4.5 -> Capacitor_Tantalum_SMD:CP_EIA-3528-21_Kemet-B_Pad1.50x2.35mm_HandSolder
Changed lines of the file:
@@
 F 0 "C3" H 22318 14046 50  0000 L CNN
 F 1 "10u x 6.3V" H 22318 13955 50  0000 L CNN
-F 2 "Capacitor_SMD:CP_Elec_4x4.5" H 22238 13850 50  0001 C CNN
+F 2 "Capacitor_Tantalum_SMD:CP_EIA-3528-21_Kemet-B_Pad1.50x2.35mm_HandSolder" H 22238 13850 50  0001 C CNN
 F 3 "~" H 22200 14000 50  0001 C CNN
 	1    22200 14000
@@
 Text Label 3600 10300 2    50   ~ 0
 ~and_oe
-Wire Bus Line
-	11450 2600 11450 6600
-Wire Bus Line
-	7800 6600 7800 9750
-Wire Bus Line
-	7800 1950 7800 5300
-Wire Bus Line
-	5350 1650 5350 5700
-Wire Wire Line
-	5450 2100 6350 2100
-Wire Wire Line
-	5450 2400 6350 2400
-Wire Wire Line
-	5450 2700 6350 2700
-Wire Wire Line
-	5450 3000 6350 3000
-Wire Wire Line
-	5450 4300 6350 4300
-Wire Wire Line
-	5450 4600 6350 4600
-Wire Wire Line
-	5450 4900 6350 4900
-Wire Bus Line
-	5850 1500 5850 5500
-Wire Wire Line
-	5450 5200 6350 5200
-Wire Bus Line
-	5350 6000 5350 9550
-Wire Wire Line
-	5450 6550 6350 6550
-Wire Wire Line
-	5450 6850 6350 6850
-Wire Wire Line
-	5450 7150 6350 7150
-Wire Wire Line
-	5450 7450 6350 7450
-Wire Wire Line
-	5450 8750 6350 8750
-Wire Wire Line
-	5450 9050 6350 9050
-Wire Bus Line
-	5850 5700 5850 9650
-Wire Wire Line
-	5450 9350 6350 9350
-Wire Wire Line
-	5450 9650 6350 9650
-Wire Bus Line
-	12350 2900 14550 2900
-Wire Bus Line
-	12350 2900 12350 6650
-Wire Bus Line
-	1250 3200 1250 4000
-Wire Bus Line
-	1250 1500 1250 3050
-Wire Bus Line
-	1900 1650 1900 2950
-Wire Bus Line
-	3450 2050 3450 2950
-Wire Bus Line
-	3450 3050 3450 3550
 $Comp
 L Device:R R8
@@
 	0    1    1    0
 $EndComp
+Wire Wire Line
+	5450 2100 6350 2100
+Wire Wire Line
+	5450 2400 6350 2400
+Wire Wire Line
+	5450 2700 6350 2700
+Wire Wire Line
+	5450 3000 6350 3000
+Wire Wire Line
+	5450 4300 6350 4300
+Wire Wire Line
+	5450 4600 6350 4600
+Wire Wire Line
+	5450 4900 6350 4900
+Wire Wire Line
+	5450 5200 6350 5200
+Wire Wire Line
+	5450 6550 6350 6550
+Wire Wire Line
+	5450 6850 6350 6850
+Wire Wire Line
+	5450 7150 6350 7150
+Wire Wire Line
+	5450 7450 6350 7450
+Wire Wire Line
+	5450 8750 6350 8750
+Wire Wire Line
+	5450 9050 6350 9050
+Wire Wire Line
+	5450 9350 6350 9350
+Wire Wire Line
+	5450 9650 6350 9650
+Wire Bus Line
+	12350 2900 14550 2900
+Wire Bus Line
+	1250 3200 1250 4000
+Wire Bus Line
+	3450 3050 3450 3550
+Wire Bus Line
+	12350 2900 12350 6650
+Wire Bus Line
+	11450 2600 11450 6600
+Wire Bus Line
+	7800 6600 7800 9750
+Wire Bus Line
+	7800 1950 7800 5300
+Wire Bus Line
+	5350 6000 5350 9550
+Wire Bus Line
+	5850 5700 5850 9650
+Wire Bus Line
+	1900 1650 1900 2950
+Wire Bus Line
+	3450 2050 3450 2950
+Wire Bus Line
+	1250 1500 1250 3050
+Wire Bus Line
+	5850 1500 5850 5500
+Wire Bus Line
+	5350 1650 5350 5700
 $EndSCHEMATC
