File: boards/vga/vga.sch (KiCad schematic (older format))
At the start: 39 parts, among them J1 Conn_02x20_Odd_Even, Q1 Q_PMOS_DGS, U1 74LS161, U10 62256-TSOP, U11 74LS161, U12 74LS161, U13 74HC244, U14 SN74LV20APWR, U15 74LV32APWJ, U16 74LV08APWJ, U17 AT28C256-PLCC32, U18 74HC273, U19 74HC273, U2 74LS161, U20 74LS151, U21 74LS157, U22 SN74LV10APWR, U23 SN74LV74APWR, U24 SN74LV00APW, U25 74LV32APWJ, U26 SN74LV21APWR, U27 SN74AHC1G86DBVR, U28 74LV32APWJ, U29 74LV08APWJ, U3 74LS157, U30 SN74LV74APWR, U4 74LS157, U5 74LS157, U6 74LS161, U7 74LS161, U8 74HC244, U9 62256-TSOP, X1 MXO45HS-3C-25M1750

Commit message: VGA: select chips and packages
Parts:
- U1, U11, U12, U2, U6, U7: value 74LS161 -> SN74LV161APW; footprint (none) -> Package_SO:TSSOP-16_4.4x5mm_P0.65mm
- U13, U8: value 74HC244 -> SN74LV244APW; footprint (none) -> Package_SO:TSSOP-20_4.4x6.5mm_P0.65mm
- U14: value SN74LV20APWR -> SN74LV20APW
- U18, U19: value 74HC273 -> SN74LV273APW; footprint (none) -> Package_SO:TSSOP-20_4.4x6.5mm_P0.65mm
- U20: value 74LS151 -> CD74AC151M96; footprint (none) -> Package_SO:SOIC-16_3.9x9.9mm_P1.27mm
- U21, U3, U4, U5: value 74LS157 -> SN74LV157APW; footprint (none) -> Package_SO:TSSOP-16_4.4x5mm_P0.65mm
- U22: value SN74LV10APWR -> SN74LV10APW
- U23, U30: value SN74LV74APWR -> SN74LV74APW
- U26: value SN74LV21APWR -> SN74LV21APW

Commit message: VGA: decoupling capacitors
Parts:
- added C1, C10, C11, C12, C13, C14, C15, C16, C17, C18, C19, C2, C20, C21, C22, C23, C24, C25, C26, C27, C28, C29, C3, C30, C4, C5, C6, C7, C8, C9: 0.1, Capacitor_SMD:C_0805_2012Metric, symbol Device:C
- added R3: 50, symbol Device:R
- gave numbers to parts that had none: 1
Connections:
- net GND: now also C1.2, C10.2, C11.2, C12.2, C13.2, C14.2, C15.2, C16.2, C17.2, C18.2, C19.2, C2.2, C20.2, C21.2, C22.2, C23.2, C24.2, C25.2, C26.2, C27.2, C28.2, C29.2, C3.2, C30.2, C4.2, C5.2, C6.2, C7.2, C8.2, C9.2
- net VCC: now also C1.1, C10.1, C11.1, C12.1, C13.1, C14.1, C15.1, C16.1, C17.1, C18.1, C19.1, C2.1, C20.1, C21.1, C22.1, C23.1, C24.1, C25.1, C26.1, C27.1, C28.1, C29.1, C3.1, C30.1, C4.1, C5.1, C6.1, C7.1, C8.1, C9.1
- net pixel_out: now also R3.2; no longer U21.1 (S)
- new net: R3.1, U21.1 (S)

Commit message: VGA: P-MOSFET
Parts:
- Q1: value Q_PMOS_DGS -> BSS84AK; footprint (none) -> Package_TO_SOT_SMD:SOT-23; symbol Device:Q_PMOS_DGS -> Device:Q_PMOS_GSD
- R1, R2, R3: footprint (none) -> Resistor_SMD:R_0805_2012Metric
Connections:
- net VCC: now also Q1.2 (S); no longer Q1.3 (S)
- net rdy_out: now also Q1.1 (G); no longer Q1.2 (G)
- net ~rdy: now also Q1.3 (D); no longer Q1.1 (D)
Changed lines of the file:
@@
 F 0 "R1" V 13807 11250 50  0000 C CNN
 F 1 "50" V 13716 11250 50  0000 C CNN
-F 2 "" V 13530 11250 50  0001 C CNN
+F 2 "Resistor_SMD:R_0805_2012Metric" V 13530 11250 50  0001 C CNN
 F 3 "~" H 13600 11250 50  0001 C CNN
 	1    13600 11250
@@
 ext_sel
 $Comp
-L Device:Q_PMOS_DGS Q1
+L Device:Q_PMOS_GSD Q1
 U 1 1 5FD7375C
 P 21800 13800
 F 0 "Q1" H 22005 13754 50  0000 L CNN
-F 1 "Q_PMOS_DGS" H 22005 13845 50  0000 L CNN
-F 2 "" H 22000 13900 50  0001 C CNN
+F 1 "BSS84AK" H 22005 13845 50  0000 L CNN
+F 2 "Package_TO_SOT_SMD:SOT-23" H 22000 13900 50  0001 C CNN
 F 3 "~" H 21800 13800 50  0001 C CNN
 	1    21800 13800
@@
 F 0 "R2" V 4557 13000 50  0000 C CNN
 F 1 "50" V 4466 13000 50  0000 C CNN
-F 2 "" V 4280 13000 50  0001 C CNN
+F 2 "Resistor_SMD:R_0805_2012Metric" V 4280 13000 50  0001 C CNN
 F 3 "~" H 4350 13000 50  0001 C CNN
 	1    4350 13000
@@
 F 0 "R3" V 16907 5250 50  0000 C CNN
 F 1 "50" V 16816 5250 50  0000 C CNN
-F 2 "" V 16630 5250 50  0001 C CNN
+F 2 "Resistor_SMD:R_0805_2012Metric" V 16630 5250 50  0001 C CNN
 F 3 "~" H 16700 5250 50  0001 C CNN
 	1    16700 5250
