File: boards/io/io.sch (KiCad schematic (older format))
At the start: 127 parts, among them J1 61304021021, J2 SSW-120-02-G-D-RA, J3 Conn_01x09, J4 694106301002, J5 Conn_01x09, J6 SSW-120-02-G-D-RA, U1 74LV32APWJ, U10 MC74HC151ADTR2G, U11 SN74LV273APW, U12 74LV32APWJ, U13 IS61C256AL-12TLI, U14 74LV32APWJ, U2 SN74LV04APWR, U4 AT28C256-PLCC32, U5 IS61C256AL-12TLI, U6 SSW-116-01-T-S, U7 SN74LV273APW, U8 SN74LV244APW, U9 74HC30D

Commit message: IO: delete LCD module, add IO port
Parts:
- removed C10: 0.1u, Capacitor_SMD:C_0805_2012Metric, symbol Device:C
- removed J5: Conn_01x09, Connector_PinHeader_2.54mm:PinHeader_1x09_P2.54mm_Vertical, symbol Connector_Generic:Conn_01x09
- removed RV1: BOURNS 3296Y-1-203LF, Potentiometer_THT:Potentiometer_Bourns_3296Z_Horizontal, symbol Device:R_POT
- removed U14: 74LV32APWJ, Package_SO:TSSOP-14_4.4x5mm_P0.65mm, symbol 74xx:74LS32
- removed U2: SN74LV04APWR, Package_SO:TSSOP-14_4.4x5mm_P0.65mm, symbol 74xx:74HC04
- removed U6: SSW-116-01-T-S, Connector_PinSocket_2.54mm:PinSocket_1x16_P2.54mm_Vertical, symbol Display_Character:RC1602A
- added C1, C15, C16: 0.1u, Capacitor_SMD:C_0805_2012Metric, symbol Device:C
- added J5, J7: Conn_01x08, symbol Connector_Generic:Conn_01x08
- added J8: Conn_01x09, Connector_PinHeader_2.54mm:PinHeader_1x09_P2.54mm_Vertical, symbol Connector_Generic:Conn_01x09
- added R54, R55, R56, R57, R58, R59, R60, R61: 10k, Resistor_SMD:R_0805_2012Metric, symbol Device:R
- added U14: 74LS139, symbol 74xx:74LS139
- added U2: 74LS00, symbol 74xx:74LS00
- added U3: SN74LV273APW, Package_SO:TSSOP-20_4.4x6.5mm_P0.65mm, symbol 74xx:74HC273
- added U6: SN74LV244APW, Package_SO:TSSOP-20_4.4x6.5mm_P0.65mm, symbol 74xx:74HC244
Connections:
- net ~a2 is gone; now on net VCC: U12.13
- net GND: now also J3.1 (Pin_1), C1.2, C15.2, C16.2, R54.2, R55.2, R56.2, R57.2, R58.2, R59.2, R60.2, R61.2, U14.8 (GND), U2.7 (GND), U3.10 (GND), U6.10 (GND); no longer J3.9 (Pin_9)
- net VCC: now also U12.10, U12.12, U12.9, C1.1, C15.1, C16.1, J8.1 (Pin_1), U14.13 (A1), U14.14 (A0), U14.15 (E), U14.16 (VCC), U2.10, U2.12, U2.13, U2.14 (VCC), U2.9, U3.20 (VCC), U6.20 (VCC)
- net a1: now also U14.2 (A0); no longer U1.2, U12.12
- net a15: now also U2.1, U2.2
- net a2: now also U14.3 (A1); no longer U1.1
- net d0: now also U3.3 (D0), U6.18 (1Y0)
- net d1: now also U3.4 (D1), U6.16 (1Y1)
- net d2: now also U3.7 (D2), U6.14 (1Y2)
- net d3: now also U3.8 (D3), U6.12 (1Y3)
- net d4: now also U3.13 (D4), U6.3 (2Y0)
- net d5: now also U3.14 (D5), U6.5 (2Y1)
- net d6: now also U3.17 (D6), U6.7 (2Y2)
- net d7: now also U3.18 (D7), U6.9 (2Y3)
- net raml_ena: now also U2.5
- net ~a15: now also U2.3, U2.4
- net ~cr_cs: now also U14.6 (O2); no longer U12.8
- net ~io_cs: now also U14.1 (E); no longer U1.5, U12.9
- net ~kb_cs: now also U14.4 (O0); no longer U1.6
- net ~oe: now also U1.2
- net ~raml_cs: now also U2.6
- net ~rst: now also U3.1 (~Mr)
- net ~we: now also U1.5
- net at R46.1, U8.11 (2A3): now also J7.1 (Pin_1)
- net at R45.1, U8.13 (2A2): now also J7.2 (Pin_2)
- net at R44.1, U8.15 (2A1): now also J7.3 (Pin_3)
- net at R43.1, U8.17 (2A0): now also J7.4 (Pin_4)
- net at R39.1, U8.2 (1A0): now also J7.8 (Pin_8)
- net at R40.1, U8.4 (1A1): now also J7.7 (Pin_7)
- net at R41.1, U8.6 (1A2): now also J7.6 (Pin_6)
- net at R42.1, U8.8 (1A3): now also J7.5 (Pin_5)
- net at R7.1: now also J5.1 (Pin_1); no longer J3.1 (Pin_1)
- net at R8.1: now also J5.2 (Pin_2); no longer J3.2 (Pin_2)
- net at R9.1: now also J5.3 (Pin_3); no longer J3.3 (Pin_3)
- net at R10.1: now also J5.4 (Pin_4); no longer J3.4 (Pin_4)
- net at R11.1: now also J5.5 (Pin_5); no longer J3.5 (Pin_5)
- net at R12.1: now also J5.6 (Pin_6); no longer J3.6 (Pin_6)
- net at R13.1: now also J5.7 (Pin_7); no longer J3.7 (Pin_7)
- net at R14.1: now also J5.8 (Pin_8); no longer J3.8 (Pin_8)
- net a_or_12 renamed ~iport_oe
- net ~iport_oe: now also U6.1 (1OE), U6.19 (2OE); no longer U1.4
- net a_or_1n2: no longer names the net of U12.11
- net a_or_1n2: no longer U12.10
- new net: J3.6 (Pin_6), U3.12 (Q4)
- new net: J3.7 (Pin_7), U3.15 (Q5)
- new net: J3.8 (Pin_8), U3.16 (Q6)
- new net: J3.9 (Pin_9), U3.19 (Q7)
- new net: J3.2 (Pin_2), U3.2 (Q0)
- new net: J3.3 (Pin_3), U3.5 (Q1)
- new net: J3.4 (Pin_4), U3.6 (Q2)
- new net: J3.5 (Pin_5), U3.9 (Q3)
- new net: J8.2 (Pin_2), R61.1, U6.11 (2A3)
- new net: J8.3 (Pin_3), R60.1, U6.13 (2A2)
- new net: J8.4 (Pin_4), R59.1, U6.15 (2A1)
- new net: J8.5 (Pin_5), R58.1, U6.17 (2A0)
- new net: J8.9 (Pin_9), R54.1, U6.2 (1A0)
- new net: J8.8 (Pin_8), R55.1, U6.4 (1A1)
- new net: J8.7 (Pin_7), R56.1, U6.6 (1A2)
- new net: J8.6 (Pin_6), R57.1, U6.8 (1A3)
- new net oport_cp: U1.6, U3.11 (Cp)
- new net ~port_cs: U1.1, U1.4, U14.5 (O1)
- no-connect marks 26 -> 34
Other:
- note added: "FF00 Keyboard\nFF02 IO port\nFF04 Control register"
- note added: "IO port (0xFF02)"
- note added: "Keyboard (0xFF00)"
- note removed: "FF00 Keyboard\nFF02 LCD control\nFF03 LCD data\nFF04 Control register"
- moved on the sheet: C11, C12, C14, D35, D36, J3, R51, R52, U12B, U12C, U12D, U12E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

Commit message: IO: footprints and values
Parts:
- J5, J7: footprint (none) -> Connector_PinHeader_2.54mm:PinHeader_1x08_P2.54mm_Vertical
- U14: value 74LS139 -> SN74LV139APW; footprint (none) -> Package_SO:TSSOP-16_4.4x5mm_P0.65mm
- U2: value 74LS00 -> SN74LV00APW; footprint (none) -> Package_SO:TSSOP-14_4.4x5mm_P0.65mm
Changed lines of the file:
@@
 F 0 "J7" V 12614 3562 50  0000 R CNN
 F 1 "Conn_01x08" V 12750 4200 50  0000 R CNN
-F 2 "" H 12650 4050 50  0001 C CNN
+F 2 "Connector_PinHeader_2.54mm:PinHeader_1x08_P2.54mm_Vertical" H 12650 4050 50  0001 C CNN
 F 3 "~" H 12650 4050 50  0001 C CNN
 	1    12650 4050
@@
 F 0 "J5" H 10980 4742 50  0000 L CNN
 F 1 "Conn_01x08" H 10700 4200 50  0000 L CNN
-F 2 "" H 10900 4750 50  0001 C CNN
+F 2 "Connector_PinHeader_2.54mm:PinHeader_1x08_P2.54mm_Vertical" H 10900 4750 50  0001 C CNN
 F 3 "~" H 10900 4750 50  0001 C CNN
 	1    10900 4750
@@
 P 9300 10450
 F 0 "U14" H 9300 10817 50  0000 C CNN
-F 1 "74LS139" H 9300 10726 50  0000 C CNN
-F 2 "" H 9300 10450 50  0001 C CNN
-F 3 "http://www.ti.com/lit/ds/symlink/sn74ls139a.pdf" H 9300 10450 50  0001 C CNN
+F 1 "SN74LV139APW" H 9300 10726 50  0000 C CNN
+F 2 "Package_SO:TSSOP-16_4.4x5mm_P0.65mm" H 9300 10450 50  0001 C CNN
+F 3 "https://www.ti.com/lit/ds/symlink/sn74lv139a.pdf" H 9300 10450 50  0001 C CNN
 	1    9300 10450
 	1    0    0    -1
@@
 P 8700 13250
 F 0 "U14" H 8700 13617 50  0000 C CNN
-F 1 "74LS139" H 8700 13526 50  0000 C CNN
-F 2 "" H 8700 13250 50  0001 C CNN
-F 3 "http://www.ti.com/lit/ds/symlink/sn74ls139a.pdf" H 8700 13250 50  0001 C CNN
+F 1 "SN74LV139APW" H 8700 13526 50  0000 C CNN
+F 2 "Package_SO:TSSOP-16_4.4x5mm_P0.65mm" H 8700 13250 50  0001 C CNN
+F 3 "https://www.ti.com/lit/ds/symlink/sn74lv139a.pdf" H 8700 13250 50  0001 C CNN
 	2    8700 13250
 	1    0    0    -1
@@
 P 6750 14100
 F 0 "U14" H 6980 14146 50  0000 L CNN
-F 1 "74LS139" H 6980 14055 50  0000 L CNN
-F 2 "" H 6750 14100 50  0001 C CNN
-F 3 "http://www.ti.com/lit/ds/symlink/sn74ls139a.pdf" H 6750 14100 50  0001 C CNN
+F 1 "SN74LV139APW" H 6980 14055 50  0000 L CNN
+F 2 "Package_SO:TSSOP-16_4.4x5mm_P0.65mm" H 6750 14100 50  0001 C CNN
+F 3 "https://www.ti.com/lit/ds/symlink/sn74lv139a.pdf" H 6750 14100 50  0001 C CNN
 	3    6750 14100
 	1    0    0    -1
@@
 P 7950 8700
 F 0 "U2" H 7950 9025 50  0000 C CNN
-F 1 "74LS00" H 7950 8934 50  0000 C CNN
-F 2 "" H 7950 8700 50  0001 C CNN
-F 3 "http://www.ti.com/lit/gpn/sn74ls00" H 7950 8700 50  0001 C CNN
+F 1 "SN74LV00APW" H 7950 8934 50  0000 C CNN
+F 2 "Package_SO:TSSOP-14_4.4x5mm_P0.65mm" H 7950 8700 50  0001 C CNN
+F 3 "https://www.ti.com/lit/ds/symlink/sn74lv00a.pdf" H 7950 8700 50  0001 C CNN
 	1    7950 8700
 	1    0    0    -1
@@
 P 8900 8800
 F 0 "U2" H 8900 9125 50  0000 C CNN
-F 1 "74LS00" H 8900 9034 50  0000 C CNN
-F 2 "" H 8900 8800 50  0001 C CNN
-F 3 "http://www.ti.com/lit/gpn/sn74ls00" H 8900 8800 50  0001 C CNN
+F 1 "SN74LV00APW" H 8900 9034 50  0000 C CNN
+F 2 "Package_SO:TSSOP-14_4.4x5mm_P0.65mm" H 8900 8800 50  0001 C CNN
+F 3 "https://www.ti.com/lit/ds/symlink/sn74lv00a.pdf" H 8900 8800 50  0001 C CNN
 	2    8900 8800
 	1    0    0    -1
@@
 P 10000 14700
 F 0 "U2" H 10000 15025 50  0000 C CNN
-F 1 "74LS00" H 10000 14934 50  0000 C CNN
-F 2 "" H 10000 14700 50  0001 C CNN
-F 3 "http://www.ti.com/lit/gpn/sn74ls00" H 10000 14700 50  0001 C CNN
+F 1 "SN74LV00APW" H 10000 14934 50  0000 C CNN
+F 2 "Package_SO:TSSOP-14_4.4x5mm_P0.65mm" H 10000 14700 50  0001 C CNN
+F 3 "https://www.ti.com/lit/ds/symlink/sn74lv00a.pdf" H 10000 14700 50  0001 C CNN
 	3    10000 14700
 	1    0    0    -1
@@
 P 10000 14150
 F 0 "U2" H 10000 14475 50  0000 C CNN
-F 1 "74LS00" H 10000 14384 50  0000 C CNN
-F 2 "" H 10000 14150 50  0001 C CNN
-F 3 "http://www.ti.com/lit/gpn/sn74ls00" H 10000 14150 50  0001 C CNN
+F 1 "SN74LV00APW" H 10000 14384 50  0000 C CNN
+F 2 "Package_SO:TSSOP-14_4.4x5mm_P0.65mm" H 10000 14150 50  0001 C CNN
+F 3 "https://www.ti.com/lit/ds/symlink/sn74lv00a.pdf" H 10000 14150 50  0001 C CNN
 	4    10000 14150
 	1    0    0    -1
@@
 P 5600 14100
 F 0 "U2" H 5830 14146 50  0000 L CNN
-F 1 "74LS00" H 5830 14055 50  0000 L CNN
-F 2 "" H 5600 14100 50  0001 C CNN
-F 3 "http://www.ti.com/lit/gpn/sn74ls00" H 5600 14100 50  0001 C CNN
+F 1 "SN74LV00APW" H 5830 14055 50  0000 L CNN
+F 2 "Package_SO:TSSOP-14_4.4x5mm_P0.65mm" H 5600 14100 50  0001 C CNN
+F 3 "https://www.ti.com/lit/ds/symlink/sn74lv00a.pdf" H 5600 14100 50  0001 C CNN
 	5    5600 14100
 	1    0    0    -1

Commit message: IO: delete IO port
Parts:
- removed C1, C11, C15: 0.1u, Capacitor_SMD:C_0805_2012Metric, symbol Device:C
- removed J3, J8: Conn_01x09, Connector_PinHeader_2.54mm:PinHeader_1x09_P2.54mm_Vertical, symbol Connector_Generic:Conn_01x09
- removed R54, R55, R56, R57, R58, R59, R60, R61: 10k, Resistor_SMD:R_0805_2012Metric, symbol Device:R
- removed U12: 74LV32APWJ, Package_SO:TSSOP-14_4.4x5mm_P0.65mm, symbol 74xx:74LS32
- removed U3: SN74LV273APW, Package_SO:TSSOP-20_4.4x6.5mm_P0.65mm, symbol 74xx:74HC273
- removed U6: SN74LV244APW, Package_SO:TSSOP-20_4.4x6.5mm_P0.65mm, symbol 74xx:74HC244
Connections:
- net oport_cp is gone; now on net ~rom_cs: U1.6
- net ~iport_oe is gone; now on net cr_cp: U1.3
- net a15: now also U1.4
- net raml_ena: now also U1.5
- net ~cr_cs: now also U1.2, U14.5 (O1); no longer U14.6 (O2)
- net ~oe: no longer U1.2
- net ~we: now also U1.1; no longer U1.5
- removed net ~port_cs: U1.1, U1.4, U14.5 (O1)
Other:
- note removed: "IO port (0xFF02)"
- moved on the sheet: U1A, U1B

Commit message: IO: PCB rev. 2
Parts:
- J2, J6: footprint Connector_PinHeader_2.54mm:PinHeader_2x20_P2.54mm_Horizontal -> Connector_PinSocket_2.54mm:PinSocket_2x20_P2.54mm_Horizontal
Connections:
- net at R46.1, U8.11 (2A3): now also J7.8 (Pin_8); no longer J7.1 (Pin_1)
- net at R45.1, U8.13 (2A2): now also J7.7 (Pin_7); no longer J7.2 (Pin_2)
- net at R44.1, U8.15 (2A1): now also J7.6 (Pin_6); no longer J7.3 (Pin_3)
- net at R43.1, U8.17 (2A0): now also J7.5 (Pin_5); no longer J7.4 (Pin_4)
- net at R39.1, U8.2 (1A0): now also J7.1 (Pin_1); no longer J7.8 (Pin_8)
- net at R40.1, U8.4 (1A1): now also J7.2 (Pin_2); no longer J7.7 (Pin_7)
- net at R41.1, U8.6 (1A2): now also J7.3 (Pin_3); no longer J7.6 (Pin_6)
- net at R42.1, U8.8 (1A3): now also J7.4 (Pin_4); no longer J7.5 (Pin_5)
Changed lines of the file:
@@
 	0    1    1    0
 $EndComp
-Wire Wire Line
-	12250 4450 13050 4450
 $Comp
 L Device:R R40
@@
 	0    1    1    0
 $EndComp
-Wire Wire Line
-	12250 4550 12950 4550
 $Comp
 L Device:R R41
@@
 	0    1    1    0
 $EndComp
-Wire Wire Line
-	12250 4650 12850 4650
 $Comp
 L Device:R R42
@@
 	0    1    1    0
 $EndComp
-Wire Wire Line
-	12250 4750 12750 4750
 $Comp
 L Device:R R43
@@
 	0    1    1    0
 $EndComp
-Wire Wire Line
-	12250 4850 12650 4850
 $Comp
 L Device:R R44
@@
 	0    1    1    0
 $EndComp
-Wire Wire Line
-	12250 4950 12550 4950
 $Comp
 L Device:R R45
@@
 	0    1    1    0
 $EndComp
-Wire Wire Line
-	12250 5050 12450 5050
 $Comp
 L Device:R R46
@@
 	0    1    1    0
 $EndComp
-Wire Wire Line
-	12250 5150 12350 5150
-Wire Wire Line
-	13050 4250 13050 4450
-Connection ~ 13050 4450
-Wire Wire Line
-	13050 4450 13100 4450
-Wire Wire Line
-	12950 4250 12950 4550
-Connection ~ 12950 4550
-Wire Wire Line
-	12950 4550 13100 4550
-Wire Wire Line
-	12850 4250 12850 4650
-Connection ~ 12850 4650
-Wire Wire Line
-	12850 4650 13100 4650
-Wire Wire Line
-	12750 4250 12750 4750
-Connection ~ 12750 4750
-Wire Wire Line
-	12750 4750 13100 4750
-Wire Wire Line
-	12650 4250 12650 4850
-Connection ~ 12650 4850
-Wire Wire Line
-	12650 4850 13100 4850
-Wire Wire Line
-	12550 4250 12550 4950
-Connection ~ 12550 4950
-Wire Wire Line
-	12550 4950 13100 4950
-Wire Wire Line
-	12450 4250 12450 5050
-Connection ~ 12450 5050
-Wire Wire Line
-	12450 5050 13100 5050
-Wire Wire Line
-	12350 4250 12350 5150
-Connection ~ 12350 5150
-Wire Wire Line
-	12350 5150 13100 5150
 Wire Wire Line
 	11950 4300 11950 4450
@@
 F 0 "J2" H 1150 7517 50  0000 C CNN
 F 1 "SSW-120-02-G-D-RA" H 1150 7426 50  0000 C CNN
-F 2 "Connector_PinHeader_2.54mm:PinHeader_2x20_P2.54mm_Horizontal" H 1100 6400 50  0001 C CNN
+F 2 "Connector_PinSocket_2.54mm:PinSocket_2x20_P2.54mm_Horizontal" H 1100 6400 50  0001 C CNN
 F 3 "~" H 1100 6400 50  0001 C CNN
 	1    1100 6400
@@
 F 0 "J6" H 21550 7567 50  0000 C CNN
 F 1 "SSW-120-02-G-D-RA" H 21550 7476 50  0000 C CNN
-F 2 "Connector_PinHeader_2.54mm:PinHeader_2x20_P2.54mm_Horizontal" H 21500 6450 50  0001 C CNN
+F 2 "Connector_PinSocket_2.54mm:PinSocket_2x20_P2.54mm_Horizontal" H 21500 6450 50  0001 C CNN
 F 3 "~" H 21500 6450 50  0001 C CNN
 	1    21500 6450
@@
 L Connector_Generic:Conn_01x08 J7
 U 1 1 5FDEB6D8
-P 12650 4050
-F 0 "J7" V 12614 3562 50  0000 R CNN
-F 1 "Conn_01x08" V 12750 4200 50  0000 R CNN
-F 2 "Connector_PinHeader_2.54mm:PinHeader_1x08_P2.54mm_Vertical" H 12650 4050 50  0001 C CNN
-F 3 "~" H 12650 4050 50  0001 C CNN
-	1    12650 4050
-	0    -1   -1   0
+P 12750 4050
+F 0 "J7" V 12714 3562 50  0000 R CNN
+F 1 "Conn_01x08" V 12850 4200 50  0000 R CNN
+F 2 "Connector_PinHeader_2.54mm:PinHeader_1x08_P2.54mm_Vertical" H 12750 4050 50  0001 C CNN
+F 3 "~" H 12750 4050 50  0001 C CNN
+	1    12750 4050
+	0    1    -1   0
 $EndComp
 $Comp
@@
 NoConn ~ 7550 7200
 NoConn ~ 9800 10550
+Wire Wire Line
+	12750 4750 13100 4750
+Wire Wire Line
+	12250 4750 12750 4750
+Connection ~ 12750 4750
+Wire Wire Line
+	12750 4250 12750 4750
+Wire Wire Line
+	12650 4850 13100 4850
+Wire Wire Line
+	12250 4850 12650 4850
+Connection ~ 12650 4850
+Wire Wire Line
+	12650 4250 12650 4850
+Wire Wire Line
+	12550 4950 13100 4950
+Wire Wire Line
+	12250 4950 12550 4950
+Connection ~ 12550 4950
+Wire Wire Line
+	12550 4250 12550 4950
+Wire Wire Line
+	12450 5050 13100 5050
+Wire Wire Line
+	12250 5050 12450 5050
+Connection ~ 12450 5050
+Wire Wire Line
+	12450 4250 12450 5050
+Wire Wire Line
+	12350 5150 13100 5150
+Wire Wire Line
+	12250 5150 12350 5150
+Connection ~ 12350 5150
+Wire Wire Line
+	12350 4250 12350 5150
+Wire Wire Line
+	12850 4650 13100 4650
+Wire Wire Line
+	12250 4650 12850 4650
+Connection ~ 12850 4650
+Wire Wire Line
+	12850 4250 12850 4650
+Wire Wire Line
+	12950 4550 13100 4550
+Wire Wire Line
+	12250 4550 12950 4550
+Connection ~ 12950 4550
+Wire Wire Line
+	12950 4250 12950 4550
+Wire Wire Line
+	13050 4450 13100 4450
+Wire Wire Line
+	12250 4450 13050 4450
+Connection ~ 13050 4450
+Wire Wire Line
+	13050 4250 13050 4450
 Wire Bus Line
 	11000 1200 11000 2100
