File: boards/io/io.kicad_pcb (KiCad board)
At the start: 2 copper layers, 100 x 100 mm, 123 parts, among them J1 61304021021, J2 SSW-120-02-G-D-RA, J4 694106301002, J5 Conn_01x08, J6 SSW-120-02-G-D-RA, J7 Conn_01x08, U1 74LV32APWJ, U10 MC74HC151ADTR2G, U11 SN74LV273APW, U13 IS61C256AL-12TLI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

Commit message: IO board rev. 3
Move side connectors
Take caution against crosstalk
Parts:
- moved D35 9.65 mm to (195.8, 71.4)
- moved R51 9.55 mm to (195.8, 69.3)
- moved R52 9.51 mm to (104.0, 69.3)
- moved D36 9.41 mm to (104.0, 71.6)
- moved J6 5.82 mm to (194.8, 75.9)
- moved J2 5.82 mm to (105.2, 124.1)
Connections:
- net /~rdy renamed /rdy
Routing:
- net /r_ena: track 89.6 -> 103.5 mm
- net /~rst: track 160.4 -> 174.2 mm
- net /rdy: track 139.8 -> 153.5 mm
- net /~we: track 225.8 -> 239.5 mm
- net /l_ena: track 80.3 -> 93.5 mm, vias 2 -> 1
- net /~oe: track 210.6 -> 223.6 mm
- net /a6: track 155.6 -> 168.4 mm
- net /a3: track 146.7 -> 159.3 mm
- net /a13: track 203.3 -> 215.9 mm
- net /a2: track 162.0 -> 174.6 mm
- net /a4: track 150.2 -> 162.7 mm
- net /a12: track 202.4 -> 214.7 mm
- net /a11: track 155.4 -> 167.6 mm
- net /a5: track 158.9 -> 171.0 mm
- net /a10: track 167.1 -> 179.0 mm
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Other:
- board text added: "IO rev.3"
- board text removed: "IO rev.2"
