File: boards/vario/ps2.sch (KiCad schematic (older format))
At the start: 33 parts, among them Q1 Q_NMOS_DSG, Q2 Q_NMOS_DSG, Q3 Q_PMOS_DGS, U10 74LS161, U11 74HC244, U12 74HC74, U13 74HC74, U14 74LS08, U15 74HC74, U16 74HC74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

Commit message: PS/2: decoupling capacitors
Parts:
- added C10, C11, C12, C13, C14, C15, C16, C17, C18, C19, C20, C21, C22, C23, C24, C25, C26, C3, C4, C5, C6, C7, C8, C9: 0.1, symbol Device:C
