File: boards/vario/ps2.sch (KiCad schematic (older format))
At the start: 58 parts, among them Q3 2N7002, Q4 2N7002, Q5 2N7002, U10 74HC161PW, U11 MC74HC244ADT, U12 74HC74PW, U13 74HC74PW, U14 74HC08PW, U15 74HC74PW, U16 74HC74PW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

Commit message: Vario: kikad-rescue
Parts:
- U19, U23: symbol 74xx:74LS280 -> vario-rescue:74LS280-74xx
Changed lines of the file:
@@
 send_ena_clk
 $Comp
-L 74xx:74LS280 U19
+L vario-rescue:74LS280-74xx U19
 U 1 1 5FFD6EE7
 P 9850 14750
+AR Path="/5FFD6EE7" Ref="U19"  Part="1"
+AR Path="/5FE853A4/5FFD6EE7" Ref="U19"  Part="1"
 F 0 "U19" H 10250 14300 50  0000 C CNN
 F 1 "CD74HC280MT" H 10250 14150 50  0000 C CNN
@@
 data_out_ena
 $Comp
-L 74xx:74LS280 U23
+L vario-rescue:74LS280-74xx U23
 U 1 1 600222E3
 P 6100 4150
+AR Path="/600222E3" Ref="U23"  Part="1"
+AR Path="/5FE853A4/600222E3" Ref="U23"  Part="1"
 F 0 "U23" H 6500 3700 50  0000 C CNN
 F 1 "CD74HC280MT" H 6500 3550 50  0000 C CNN

Commit message: Vario: exact RC values
Parts:
- C1: value C -> 10n
- C2: value C -> 100
- R3: value R -> 16k
- R4: value R -> 10k
Changed lines of the file:
@@
 P 3550 10450
 F 0 "R3" V 3757 10450 50  0000 C CNN
-F 1 "R" V 3666 10450 50  0000 C CNN
+F 1 "16k" V 3666 10450 50  0000 C CNN
 F 2 "Resistor_SMD:R_0805_2012Metric" V 3480 10450 50  0001 C CNN
 F 3 "~" H 3550 10450 50  0001 C CNN
@@
 P 3700 10600
 F 0 "C1" H 3815 10646 50  0000 L CNN
-F 1 "C" H 3815 10555 50  0000 L CNN
+F 1 "10n" H 3815 10555 50  0000 L CNN
 F 2 "Capacitor_SMD:C_0805_2012Metric" H 3738 10450 50  0001 C CNN
 F 3 "~" H 3700 10600 50  0001 C CNN
@@
 P 9200 8700
 F 0 "R4" V 9407 8700 50  0000 C CNN
-F 1 "R" V 9316 8700 50  0000 C CNN
+F 1 "10k" V 9316 8700 50  0000 C CNN
 F 2 "Resistor_SMD:R_0805_2012Metric" V 9130 8700 50  0001 C CNN
 F 3 "~" H 9200 8700 50  0001 C CNN
@@
 P 9350 8850
 F 0 "C2" H 9465 8896 50  0000 L CNN
-F 1 "C" H 9465 8805 50  0000 L CNN
+F 1 "100" H 9465 8805 50  0000 L CNN
 F 2 "Capacitor_SMD:C_0805_2012Metric" H 9388 8700 50  0001 C CNN
 F 3 "~" H 9350 8850 50  0001 C CNN
