File: boards/vario/vario.sch (KiCad schematic (older format))
At the start: 39 parts, among them J1 Conn_02x20_Odd_Even, J2 SD_Card, J3 Mini-DIN-6, U34 74LS273, U35 74HC244, U36 IFX54441EJV33

Commit message: Vario: status LEDs
Parts:
- added D1, D4: LED, symbol Device:LED
- added H1, H2, H3, H4: MountingHole, symbol Mechanical:MountingHole
- added R18, R21: 620, symbol Device:R
- gave numbers to parts that had none: 7
Connections:
- net GND: now also R18.1
- net VCC: now also R21.1
- net en_3v3: now also D1.2 (A)
- net at U37.1 (E), U37.11 (O1): now also D4.1 (K)
- new net: D1.1 (K), R18.2
- new net: D4.2 (A), R21.2
Changed lines of the file:
@@
 	9250 10150 9250 10250
 $Comp
-L Device:Q_NMOS_GSD Q?
+L Device:Q_NMOS_GSD Q1
 U 1 1 6021BDC6
 P 6000 7550
-F 0 "Q?" H 6205 7596 50  0000 L CNN
+F 0 "Q1" H 6205 7596 50  0000 L CNN
 F 1 "Q_NMOS_GSD" H 6205 7505 50  0000 L CNN
 F 2 "" H 6200 7650 50  0001 C CNN
@@
 Connection ~ 5900 7350
 $Comp
-L 74xx:74LS30 U?
+L 74xx:74LS30 U27
 U 1 1 6022739C
 P 1250 7600
-F 0 "U?" H 1250 8125 50  0000 C CNN
+F 0 "U27" H 1250 8125 50  0000 C CNN
 F 1 "74LS30" H 1250 8034 50  0000 C CNN
 F 2 "" H 1250 7600 50  0001 C CNN
@@
 $EndComp
 $Comp
-L 74xx:74LS30 U?
+L 74xx:74LS30 U27
 U 2 1 602286DA
 P 2650 13600
-F 0 "U?" H 2880 13646 50  0000 L CNN
+F 0 "U27" H 2880 13646 50  0000 L CNN
 F 1 "74LS30" H 2880 13555 50  0000 L CNN
 F 2 "" H 2650 13600 50  0001 C CNN
@@
 $EndComp
 $Comp
-L 74xx:74LS139 U?
+L 74xx:74LS139 U37
 U 1 1 602FAA53
 P 3550 7200
-F 0 "U?" H 3550 7567 50  0000 C CNN
+F 0 "U37" H 3550 7567 50  0000 C CNN
 F 1 "74LS139" H 3550 7476 50  0000 C CNN
 F 2 "" H 3550 7200 50  0001 C CNN
@@
 $EndComp
 $Comp
-L 74xx:74LS139 U?
+L 74xx:74LS139 U37
 U 2 1 602FCA57
 P 2200 7400
-F 0 "U?" H 2200 7767 50  0000 C CNN
+F 0 "U37" H 2200 7767 50  0000 C CNN
 F 1 "74LS139" H 2200 7676 50  0000 C CNN
 F 2 "" H 2200 7400 50  0001 C CNN
@@
 $EndComp
 $Comp
-L 74xx:74LS139 U?
+L 74xx:74LS139 U37
 U 3 1 602FD784
 P 3650 13600
-F 0 "U?" H 3880 13646 50  0000 L CNN
+F 0 "U37" H 3880 13646 50  0000 L CNN
 F 1 "74LS139" H 3880 13555 50  0000 L CNN
 F 2 "" H 3650 13600 50  0001 C CNN
@@
 	1700 7600 1550 7600
 $Comp
-L power:VCC #PWR?
+L power:VCC #PWR072
 U 1 1 6031DFFE
 P 950 8000
-F 0 "#PWR?" H 950 7850 50  0001 C CNN
+F 0 "#PWR072" H 950 7850 50  0001 C CNN
 F 1 "VCC" V 965 8128 50  0000 L CNN
 F 2 "" H 950 8000 50  0001 C CNN
@@
 ~oe
 $Comp
-L Device:C C?
+L Device:C C25
 U 1 1 6034577B
 P 2600 15200
-F 0 "C?" H 2715 15246 50  0000 L CNN
+F 0 "C25" H 2715 15246 50  0000 L CNN
 F 1 "0.1" H 2715 15155 50  0000 L CNN
 F 2 "" H 2638 15050 50  0001 C CNN
@@
 $EndComp
 $Comp
-L power:GND #PWR?
+L power:GND #PWR0147
 U 1 1 60345781
 P 2600 15350
-F 0 "#PWR?" H 2600 15100 50  0001 C CNN
+F 0 "#PWR0147" H 2600 15100 50  0001 C CNN
 F 1 "GND" H 2605 15177 50  0000 C CNN
 F 2 "" H 2600 15350 50  0001 C CNN
@@
 $EndComp
 $Comp
-L power:VCC #PWR?
+L power:VCC #PWR0146
 U 1 1 60345787
 P 2600 15050
-F 0 "#PWR?" H 2600 14900 50  0001 C CNN
+F 0 "#PWR0146" H 2600 14900 50  0001 C CNN
 F 1 "VCC" H 2615 15223 50  0000 C CNN
 F 2 "" H 2600 15050 50  0001 C CNN
@@
 $EndComp
 $Comp
-L Device:C C?
+L Device:C C44
 U 1 1 60347585
 P 3600 15150
-F 0 "C?" H 3715 15196 50  0000 L CNN
+F 0 "C44" H 3715 15196 50  0000 L CNN
 F 1 "0.1" H 3715 15105 50  0000 L CNN
 F 2 "" H 3638 15000 50  0001 C CNN
@@
 $EndComp
 $Comp
-L power:GND #PWR?
+L power:GND #PWR0180
 U 1 1 6034758B
 P 3600 15300
-F 0 "#PWR?" H 3600 15050 50  0001 C CNN
+F 0 "#PWR0180" H 3600 15050 50  0001 C CNN
 F 1 "GND" H 3605 15127 50  0000 C CNN
 F 2 "" H 3600 15300 50  0001 C CNN
@@
 $EndComp
 $Comp
-L power:VCC #PWR?
+L power:VCC #PWR0165
 U 1 1 60347591
 P 3600 15000
-F 0 "#PWR?" H 3600 14850 50  0001 C CNN
+F 0 "#PWR0165" H 3600 14850 50  0001 C CNN
 F 1 "VCC" H 3615 15173 50  0000 C CNN
 F 2 "" H 3600 15000 50  0001 C CNN
@@
 $EndComp
 $Comp
-L Device:C C?
+L Device:C C45
 U 1 1 60349401
 P 4450 15200
-F 0 "C?" H 4565 15246 50  0000 L CNN
+F 0 "C45" H 4565 15246 50  0000 L CNN
 F 1 "0.1" H 4565 15155 50  0000 L CNN
 F 2 "" H 4488 15050 50  0001 C CNN
@@
 $EndComp
 $Comp
-L power:GND #PWR?
+L power:GND #PWR0219
 U 1 1 60349407
 P 4450 15350
-F 0 "#PWR?" H 4450 15100 50  0001 C CNN
+F 0 "#PWR0219" H 4450 15100 50  0001 C CNN
 F 1 "GND" H 4455 15177 50  0000 C CNN
 F 2 "" H 4450 15350 50  0001 C CNN
@@
 $EndComp
 $Comp
-L power:VCC #PWR?
+L power:VCC #PWR0218
 U 1 1 6034940D
 P 4450 15050
-F 0 "#PWR?" H 4450 14900 50  0001 C CNN
+F 0 "#PWR0218" H 4450 14900 50  0001 C CNN
 F 1 "VCC" H 4465 15223 50  0000 C CNN
 F 2 "" H 4450 15050 50  0001 C CNN
@@
 $EndComp
 $Comp
-L power:GND #PWR?
+L power:GND #PWR0149
 U 1 1 6034AA58
 P 2650 14100
-F 0 "#PWR?" H 2650 13850 50  0001 C CNN
+F 0 "#PWR0149" H 2650 13850 50  0001 C CNN
 F 1 "GND" H 2655 13927 50  0000 C CNN
 F 2 "" H 2650 14100 50  0001 C CNN
@@
 $EndComp
 $Comp
-L power:GND #PWR?
+L power:GND #PWR0217
 U 1 1 6034B314
 P 3650 14100
-F 0 "#PWR?" H 3650 13850 50  0001 C CNN
+F 0 "#PWR0217" H 3650 13850 50  0001 C CNN
 F 1 "GND" H 3655 13927 50  0000 C CNN
 F 2 "" H 3650 14100 50  0001 C CNN
@@
 $EndComp
 $Comp
-L power:VCC #PWR?
+L power:VCC #PWR0148
 U 1 1 6034B7EC
 P 2650 13100
-F 0 "#PWR?" H 2650 12950 50  0001 C CNN
+F 0 "#PWR0148" H 2650 12950 50  0001 C CNN
 F 1 "VCC" H 2665 13273 50  0000 C CNN
 F 2 "" H 2650 13100 50  0001 C CNN
@@
 $EndComp
 $Comp
-L power:VCC #PWR?
+L power:VCC #PWR0216
 U 1 1 6034BF31
 P 3650 13100
-F 0 "#PWR?" H 3650 12950 50  0001 C CNN
+F 0 "#PWR0216" H 3650 12950 50  0001 C CNN
 F 1 "VCC" H 3665 13273 50  0000 C CNN
 F 2 "" H 3650 13100 50  0001 C CNN
@@
 $EndComp
 $Comp
-L 74xx:74LS32 U?
+L 74xx:74LS32 U38
 U 1 1 6034E6D8
 P 4250 10150
-F 0 "U?" H 4250 10475 50  0000 C CNN
+F 0 "U38" H 4250 10475 50  0000 C CNN
 F 1 "74LS32" H 4250 10384 50  0000 C CNN
 F 2 "" H 4250 10150 50  0001 C CNN
@@
 $EndComp
 $Comp
-L 74xx:74LS32 U?
+L 74xx:74LS32 U38
 U 2 1 603503BA
 P 8600 10850
-F 0 "U?" H 8600 11175 50  0000 C CNN
+F 0 "U38" H 8600 11175 50  0000 C CNN
 F 1 "74LS32" H 8600 11084 50  0000 C CNN
 F 2 "" H 8600 10850 50  0001 C CNN
@@
 $EndComp
 $Comp
-L 74xx:74LS32 U?
+L 74xx:74LS32 U38
 U 3 1 6035209C
 P 11700 12600
-F 0 "U?" H 11700 12925 50  0000 C CNN
+F 0 "U38" H 11700 12925 50  0000 C CNN
 F 1 "74LS32" H 11700 12834 50  0000 C CNN
 F 2 "" H 11700 12600 50  0001 C CNN
@@
 $EndComp
 $Comp
-L 74xx:74LS32 U?
+L 74xx:74LS32 U38
 U 4 1 6035479B
 P 11100 12600
-F 0 "U?" H 11100 12925 50  0000 C CNN
+F 0 "U38" H 11100 12925 50  0000 C CNN
 F 1 "74LS32" H 11100 12834 50  0000 C CNN
 F 2 "" H 11100 12600 50  0001 C CNN
@@
 $EndComp
 $Comp
-L 74xx:74LS32 U?
+L 74xx:74LS32 U38
 U 5 1 60357EA2
 P 4850 13600
-F 0 "U?" H 5080 13646 50  0000 L CNN
+F 0 "U38" H 5080 13646 50  0000 L CNN
 F 1 "74LS32" H 5080 13555 50  0000 L CNN
 F 2 "" H 4850 13600 50  0001 C CNN
@@
 $EndComp
 $Comp
-L power:GND #PWR?
+L power:GND #PWR0221
 U 1 1 6035EB9D
 P 4850 14100
-F 0 "#PWR?" H 4850 13850 50  0001 C CNN
+F 0 "#PWR0221" H 4850 13850 50  0001 C CNN
 F 1 "GND" H 4855 13927 50  0000 C CNN
 F 2 "" H 4850 14100 50  0001 C CNN
@@
 $EndComp
 $Comp
-L power:VCC #PWR?
+L power:VCC #PWR0220
 U 1 1 6035F03D
 P 4850 13100
-F 0 "#PWR?" H 4850 12950 50  0001 C CNN
+F 0 "#PWR0220" H 4850 12950 50  0001 C CNN
 F 1 "VCC" H 4865 13273 50  0000 C CNN
 F 2 "" H 4850 13100 50  0001 C CNN
@@
 NoConn ~ 12000 12600
 $Comp
-L power:VCC #PWR?
+L power:VCC #PWR0222
 U 1 1 6036380A
 P 10800 12600
-F 0 "#PWR?" H 10800 12450 50  0001 C CNN
+F 0 "#PWR0222" H 10800 12450 50  0001 C CNN
 F 1 "VCC" H 10815 12773 50  0000 C CNN
 F 2 "" H 10800 12600 50  0001 C CNN
@@
 ~card_cs
 Wire Wire Line
-	3050 7400 2700 7400
+	3050 7400 2950 7400
 NoConn ~ 2300 3050
 NoConn ~ 1800 3050
@@
 NoConn ~ 2300 2850
 NoConn ~ 1800 2850
+Text Label 950  7900 2    50   ~ 0
+ena
+$Comp
+L Mechanical:MountingHole H1
+U 1 1 60387703
+P 19400 600
+F 0 "H1" H 19500 646 50  0000 L CNN
+F 1 "MountingHole" H 19500 555 50  0000 L CNN
+F 2 "" H 19400 600 50  0001 C CNN
+F 3 "~" H 19400 600 50  0001 C CNN
+	1    19400 600
+	1    0    0    -1
+$EndComp
+$Comp
+L Mechanical:MountingHole H2
+U 1 1 60387DC7
+P 19400 850
+F 0 "H2" H 19500 896 50  0000 L CNN
+F 1 "MountingHole" H 19500 805 50  0000 L CNN
+F 2 "" H 19400 850 50  0001 C CNN
+F 3 "~" H 19400 850 50  0001 C CNN
+	1    19400 850
+	1    0    0    -1
+$EndComp
+$Comp
+L Mechanical:MountingHole H3
+U 1 1 60387F65
+P 19400 1150
+F 0 "H3" H 19500 1196 50  0000 L CNN
+F 1 "MountingHole" H 19500 1105 50  0000 L CNN
+F 2 "" H 19400 1150 50  0001 C CNN
+F 3 "~" H 19400 1150 50  0001 C CNN
+	1    19400 1150
+	1    0    0    -1
+$EndComp
+$Comp
+L Mechanical:MountingHole H4
+U 1 1 60388301
+P 19400 1400
+F 0 "H4" H 19500 1446 50  0000 L CNN
+F 1 "MountingHole" H 19500 1355 50  0000 L CNN
+F 2 "" H 19400 1400 50  0001 C CNN
+F 3 "~" H 19400 1400 50  0001 C CNN
+	1    19400 1400
+	1    0    0    -1
+$EndComp
+$Comp
+L Device:LED D1
+U 1 1 6038A92B
+P 12350 2950
+F 0 "D1" H 12343 2695 50  0000 C CNN
+F 1 "LED" H 12343 2786 50  0000 C CNN
+F 2 "" H 12350 2950 50  0001 C CNN
+F 3 "~" H 12350 2950 50  0001 C CNN
+	1    12350 2950
+	-1   0    0    1
+$EndComp
+Text Label 12200 2950 2    50   ~ 0
+en_3v3
+$Comp
+L Device:R R18
+U 1 1 6038DD0A
+P 12650 2950
+F 0 "R18" V 12443 2950 50  0000 C CNN
+F 1 "620" V 12534 2950 50  0000 C CNN
+F 2 "" V 12580 2950 50  0001 C CNN
+F 3 "~" H 12650 2950 50  0001 C CNN
+	1    12650 2950
+	0    1    1    0
+$EndComp
+$Comp
+L power:GND #PWR0223
+U 1 1 6038E61B
+P 12800 2950
+F 0 "#PWR0223" H 12800 2700 50  0001 C CNN
+F 1 "GND" H 12805 2777 50  0000 C CNN
+F 2 "" H 12800 2950 50  0001 C CNN
+F 3 "" H 12800 2950 50  0001 C CNN
+	1    12800 2950
+	0    -1   -1   0
+$EndComp
+$Comp
+L Device:LED D4
+U 1 1 603BA214
+P 3350 8000
+F 0 "D4" H 3343 8217 50  0000 C CNN
+F 1 "LED" H 3343 8126 50  0000 C CNN
+F 2 "" H 3350 8000 50  0001 C CNN
+F 3 "~" H 3350 8000 50  0001 C CNN
+	1    3350 8000
+	1    0    0    -1
+$EndComp
+$Comp
+L Device:R R21
+U 1 1 603BA21A
+P 3650 8000
+F 0 "R21" V 3443 8000 50  0000 C CNN
+F 1 "620" V 3534 8000 50  0000 C CNN
+F 2 "" V 3580 8000 50  0001 C CNN
+F 3 "~" H 3650 8000 50  0001 C CNN
+	1    3650 8000
+	0    1    1    0
+$EndComp
+Wire Wire Line
+	3200 8000 2950 8000
+Wire Wire Line
+	2950 8000 2950 7400
+Connection ~ 2950 7400
+Wire Wire Line
+	2950 7400 2700 7400
 Wire Bus Line
 	4200 2150 4200 5750
-Text Label 950  7900 2    50   ~ 0
-ena
+$Comp
+L power:VCC #PWR0228
+U 1 1 603C0A6B
+P 3800 8000
+F 0 "#PWR0228" H 3800 7850 50  0001 C CNN
+F 1 "VCC" H 3815 8173 50  0000 C CNN
+F 2 "" H 3800 8000 50  0001 C CNN
+F 3 "" H 3800 8000 50  0001 C CNN
+	1    3800 8000
+	0    1    1    0
+$EndComp
 $EndSCHEMATC

Commit message: Vario: component names and footprints
Parts:
- added 33.0x10v: CP, Capacitor_Tantalum_SMD:CP_EIA-3528-21_Kemet-B_Pad1.50x2.35mm_HandSolder, symbol Device:CP
- 33.0x10v: renamed from C41; footprint (none) -> Capacitor_Tantalum_SMD:CP_EIA-3528-21_Kemet-B_Pad1.50x2.35mm_HandSolder
- C25, C37, C38, C39, C40, C42, C43, C44, C45: footprint (none) -> Capacitor_SMD:C_0805_2012Metric
- D1, D4: footprint (none) -> LED_SMD:LED_0805_2012Metric
- H1, H2, H3, H4: footprint (none) -> MountingHole:MountingHole_3.2mm_M3
- J1: footprint (none) -> Connector_PinHeader_2.54mm:PinHeader_2x20_P2.54mm_Horizontal
- J2: footprint (none) -> Connector_Card:SD_Kyocera_145638009211859+
- J3: footprint (none) -> vario:Connector-MiniDIN-6
- Q1: footprint (none) -> Package_TO_SOT_SMD:SOT-23
- R10, R11, R12, R13, R14, R15, R16, R17, R18, R21, R6, R7, R8, R9: footprint (none) -> Resistor_SMD:R_0805_2012Metric
- U27: value 74LS30 -> 74HC30D; footprint (none) -> Package_SO:SOIC-14_3.9x8.7mm_P1.27mm
- U34: value 74LS273 -> 74HC273PW; footprint (none) -> Package_SO:TSSOP-20_4.4x6.5mm_P0.65mm
- U35: value 74HC244 -> MC74HC244ADT; footprint (none) -> Package_SO:TSSOP-20_4.4x6.5mm_P0.65mm
- U37: value 74LS139 -> SN74HC139PW; footprint (none) -> Package_SO:TSSOP-16_4.4x5mm_P0.65mm
- U38: value 74LS32 -> SN74HC32PWR; footprint (none) -> Package_SO:TSSOP-14_4.4x5mm_P0.65mm
Connections:
- net GND: now also 33.0x10v.2
- net VCC: now also 33.0x10v.1
