File: boards/vario/vario.sch (KiCad schematic (older format))
At the start: 41 parts, among them J1 Conn_02x20_Odd_Even, J2 SD_Card, J3 Mini-DIN-6, Q1 Q_NMOS_GSD, U27 74HC30D, U34 74HC273PW, U35 MC74HC244ADT, U36 IFX54441EJV33, U37 SN74HC139PW, U38 SN74HC32PWR

Commit message: Vario: transistors and capacitors
Parts:
- C41, C46: renamed from 33.0x10v; value CP -> 33.0x10v
- Q1: value Q_NMOS_GSD -> 2N7002
Changed lines of the file:
@@
 	13150 1650 13050 1650
 $Comp
-L Device:CP 33.0x10v
+L Device:CP C46
 U 1 1 5FF0EBC2
 P 13800 1800
-F 0 "33.0x10v" H 13918 1846 50  0000 L CNN
-F 1 "CP" H 13918 1755 50  0000 L CNN
+F 0 "C46" H 13918 1846 50  0000 L CNN
+F 1 "33.0x10v" H 13918 1755 50  0000 L CNN
 F 2 "Capacitor_Tantalum_SMD:CP_EIA-3528-21_Kemet-B_Pad1.50x2.35mm_HandSolder" H 13838 1650 50  0001 C CNN
 F 3 "~" H 13800 1800 50  0001 C CNN
@@
 P 6000 7550
 F 0 "Q1" H 6205 7596 50  0000 L CNN
-F 1 "Q_NMOS_GSD" H 6205 7505 50  0000 L CNN
+F 1 "2N7002" H 6205 7505 50  0000 L CNN
 F 2 "Package_TO_SOT_SMD:SOT-23" H 6200 7650 50  0001 C CNN
 F 3 "~" H 6000 7550 50  0001 C CNN
@@
 $EndComp
 $Comp
-L Device:CP 33.0x10v
+L Device:CP C41
 U 1 1 60223FDB
 P 750 1850
-F 0 "33.0x10v" H 868 1896 50  0000 L CNN
-F 1 "CP" H 868 1805 50  0000 L CNN
+F 0 "C41" H 868 1896 50  0000 L CNN
+F 1 "33.0x10v" H 868 1805 50  0000 L CNN
 F 2 "Capacitor_Tantalum_SMD:CP_EIA-3528-21_Kemet-B_Pad1.50x2.35mm_HandSolder" H 788 1700 50  0001 C CNN
 F 3 "~" H 750 1850 50  0001 C CNN
@@
 $EndComp
 $Comp
-L power:GND #PWR?
+L power:GND #PWR0230
 U 1 1 60223FE1
 P 750 2000
-F 0 "#PWR?" H 750 1750 50  0001 C CNN
+F 0 "#PWR0230" H 750 1750 50  0001 C CNN
 F 1 "GND" H 755 1827 50  0000 C CNN
 F 2 "" H 750 2000 50  0001 C CNN
@@
 	4200 2150 4200 5750
 $Comp
-L power:VCC #PWR?
+L power:VCC #PWR0229
 U 1 1 602257F4
 P 750 1700
-F 0 "#PWR?" H 750 1550 50  0001 C CNN
+F 0 "#PWR0229" H 750 1550 50  0001 C CNN
 F 1 "VCC" V 765 1828 50  0000 L CNN
 F 2 "" H 750 1700 50  0001 C CNN

Commit message: Vario: board, delete redundant 7474
Connections:
- net a0: now also U37.2 (A0); no longer U37.3 (A1)
- net a1: now also U37.3 (A1); no longer U37.2 (A0)
- net a8: now also U37.14 (A0); no longer U37.13 (A1)
- net a9: now also U37.13 (A1); no longer U37.14 (A0)
Changed lines of the file:
@@
 Text Label 4550 6100 2    50   ~ 0
 ~spi_data_sel
+Text Label 3050 7200 2    50   ~ 0
+a0
 Text Label 3050 7100 2    50   ~ 0
-a0
-Text Label 3050 7200 2    50   ~ 0
 a1
+Text Label 1700 7400 2    50   ~ 0
+a8
 Text Label 1700 7300 2    50   ~ 0
-a8
-Text Label 1700 7400 2    50   ~ 0
 a9
 Text Label 950  7300 2    50   ~ 0
