File: boards/stack/stack.sch (KiCad schematic (older format))
At the start: 27 parts, among them J1 SSW-120-02-G-D-RA, J2 61304021021, J3 SSW-120-02-G-D-RA, J4 SSW-120-02-G-D-RA, U1 74LS139, U11 74HC74, U12 74LS32, U13 74LS32, U14 74HC00, U15 74AHC1G86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

Commit message: Stack: values and footprints
Parts:
- added C17: TPSB336K010T0425, Capacitor_Tantalum_SMD:CP_EIA-3528-15_AVX-H_Pad1.50x2.35mm_HandSolder, symbol Device:CP
- added D18: LED, LED_SMD:LED_0805_2012Metric, symbol Device:LED
- added R18: R, Resistor_SMD:R_0805_2012Metric, symbol Device:R
- C10, C11, C12, C13, C14, C15, C16, C9: footprint (none) -> Capacitor_SMD:C_0805_2012Metric
- D17: renamed from D?; footprint (none) -> LED_SMD:LED_0805_2012Metric
- H1, H2, H3, H4: footprint (none) -> MountingHole:MountingHole_3.2mm_M3
- J1, J3, J4: footprint (none) -> Connector_PinSocket_2.54mm:PinSocket_2x20_P2.54mm_Horizontal
- J2: footprint (none) -> Connector_PinHeader_2.54mm:PinHeader_2x20_P2.54mm_Horizontal
- R17: renamed from R?; footprint (none) -> Resistor_SMD:R_0805_2012Metric
- U1: value 74LS139 -> 74HC139; footprint (none) -> Package_SO:TSSOP-16_4.4x5mm_P0.65mm
- U11, U14: footprint (none) -> Package_SO:TSSOP-14_4.4x5mm_P0.65mm
- U12, U13, U16, U17: value 74LS32 -> 74HC32; footprint (none) -> Package_SO:TSSOP-14_4.4x5mm_P0.65mm
- U15: footprint (none) -> Package_TO_SOT_SMD:SOT-23-5
Connections:
- net GND: now also U11.11 (C), U11.12 (D), U11.13 (~R), C17.2, R18.1
- net VCC: now also C17.1; no longer U11.10 (~S), U11.11 (C), U11.12 (D), U11.13 (~R)
- net ena: now also D18.2 (A)
- net rst: now also U11.9 (Q)
- net ~rst: now also U11.10 (~S)
- net down0 renamed down_0
- net down1 renamed down_1
- net ia11 renamed f0
- net ia12 renamed f1
- net ia13 renamed f2
- net ia14 renamed f3
- net ia15 renamed f4
- net ia16 renamed f5
- net ia17 renamed f6
- net ia18 renamed f7
- net up0 renamed up_0
- net up1 renamed up_1
- new net: D18.1 (K), R18.2
- no-connect marks 36 -> 35
Other:
- moved on the sheet: U11B

Commit message: Stack: more values
Parts:
- C17: value TPSB336K010T0425 -> F931C336MBAAJ6‎; footprint Capacitor_Tantalum_SMD:CP_EIA-3528-15_AVX-H_Pad1.50x2.35mm_HandSolder -> Capacitor_Tantalum_SMD:CP_EIA-3528-21_Kemet-B_Pad1.50x2.35mm_HandSolder
- D17, D18: value LED -> APT2012CGCK
- R17, R18: value R -> 160
Other:
- note added: "access"
- note added: "enabled"
Changed lines of the file:
@@
 U 1 1 61D42B93
 P 7300 10900
-F 0 "D17" H 7293 11117 50  0000 C CNN
-F 1 "LED" H 7293 11026 50  0000 C CNN
+F 0 "D17" H 7000 11050 50  0000 C CNN
+F 1 "APT2012CGCK" H 6850 10950 50  0000 C CNN
 F 2 "LED_SMD:LED_0805_2012Metric" H 7300 10900 50  0001 C CNN
 F 3 "~" H 7300 10900 50  0001 C CNN
@@
 P 7600 10900
 F 0 "R17" V 7393 10900 50  0000 C CNN
-F 1 "R" V 7484 10900 50  0000 C CNN
+F 1 "160" V 7484 10900 50  0000 C CNN
 F 2 "Resistor_SMD:R_0805_2012Metric" V 7530 10900 50  0001 C CNN
 F 3 "~" H 7600 10900 50  0001 C CNN
@@
 U 1 1 61D54B39
 P 11350 12650
-F 0 "D18" H 11343 12395 50  0000 C CNN
-F 1 "LED" H 11343 12486 50  0000 C CNN
+F 0 "D18" H 11700 12550 50  0000 C CNN
+F 1 "APT2012CGCK" H 11800 12650 50  0000 C CNN
 F 2 "LED_SMD:LED_0805_2012Metric" H 11350 12650 50  0001 C CNN
 F 3 "~" H 11350 12650 50  0001 C CNN
@@
 P 11650 12650
 F 0 "R18" V 11443 12650 50  0000 C CNN
-F 1 "R" V 11534 12650 50  0000 C CNN
+F 1 "160" V 11534 12650 50  0000 C CNN
 F 2 "Resistor_SMD:R_0805_2012Metric" V 11580 12650 50  0001 C CNN
 F 3 "~" H 11650 12650 50  0001 C CNN
@@
 P 13700 14750
 F 0 "C17" H 13818 14796 50  0000 L CNN
-F 1 "TPSB336K010T0425" H 13818 14705 50  0000 L CNN
-F 2 "Capacitor_Tantalum_SMD:CP_EIA-3528-15_AVX-H_Pad1.50x2.35mm_HandSolder" H 13738 14600 50  0001 C CNN
+F 1 "F931C336MBAAJ6‎" H 13818 14705 50  0000 L CNN
+F 2 "Capacitor_Tantalum_SMD:CP_EIA-3528-21_Kemet-B_Pad1.50x2.35mm_HandSolder" H 13738 14600 50  0001 C CNN
 F 3 "~" H 13700 14750 50  0001 C CNN
 	1    13700 14750
@@
 Wire Bus Line
 	12900 2350 12900 5300
+Text Notes 7400 11150 2    50   ~ 0
+access
+Text Notes 11450 12850 2    50   ~ 0
+enabled
 $EndSCHEMATC

Commit message: Stack: board started
Parts:
- added C18: 0.1, Capacitor_SMD:C_0805_2012Metric, symbol Device:C
Connections:
- net GND: now also C18.2
- net VCC: now also C18.1
- net a4: now also U2.25 (A11); no longer U2.8 (A4)
- net a5: now also U2.28 (A13); no longer U2.7 (A5)
- net a6: now also U2.30 (A18); no longer U2.6 (A6)
- net a7: now also U2.31 (A15); no longer U2.5 (A7)
- net f0: now also U2.8 (A4); no longer U2.25 (A11)
- net f2: now also U2.7 (A5); no longer U2.28 (A13)
- net f4: now also U2.5 (A7); no longer U2.31 (A15)
- net f7: now also U2.6 (A6); no longer U2.30 (A18)
Changed lines of the file:
@@
 	8900 2350 10000 2350
 Connection ~ 10000 2350
-Entry Wire Line
-	12900 5500 13000 5600
-Entry Wire Line
-	12900 5400 13000 5500
-Entry Wire Line
-	12900 5600 13000 5700
-Entry Wire Line
-	12900 5700 13000 5800
-Entry Wire Line
-	12900 5800 13000 5900
-Entry Wire Line
-	12900 5900 13000 6000
-Entry Wire Line
-	12900 6000 13000 6100
-Entry Wire Line
-	12900 6100 13000 6200
 Wire Wire Line
 	13150 6200 13000 6200
@@
 Wire Wire Line
 	13000 5500 13150 5500
-Text Label 13000 5500 0    50   ~ 0
+Text Label 13000 4800 0    50   ~ 0
 f0
 Text Label 13000 5600 0    50   ~ 0
 f1
-Text Label 13000 5700 0    50   ~ 0
+Text Label 13000 4900 0    50   ~ 0
 f2
 Text Label 13000 5800 0    50   ~ 0
 f3
-Text Label 13000 5900 0    50   ~ 0
+Text Label 13000 5100 0    50   ~ 0
 f4
 Text Label 13000 6000 0    50   ~ 0
@@
 Text Label 13000 6100 0    50   ~ 0
 f6
-Text Label 13000 6200 0    50   ~ 0
+Text Label 13000 5000 0    50   ~ 0
 f7
-Wire Bus Line
-	12900 5350 9000 5350
-Wire Bus Line
-	9000 5350 9000 6900
-Wire Bus Line
-	9000 4700 9000 5350
-Connection ~ 9000 5350
-Entry Wire Line
-	12900 5300 13000 5400
-Entry Wire Line
-	12900 5200 13000 5300
-Entry Wire Line
-	12900 5100 13000 5200
-Entry Wire Line
-	12900 5000 13000 5100
-Entry Wire Line
-	12900 4900 13000 5000
-Entry Wire Line
-	12900 4800 13000 4900
-Entry Wire Line
-	12900 4700 13000 4800
-Entry Wire Line
-	12900 4600 13000 4700
-Entry Wire Line
-	12900 4500 13000 4600
-Entry Wire Line
-	12900 4400 13000 4500
-Entry Wire Line
-	12900 4300 13000 4400
 Wire Wire Line
 	13000 4400 13150 4400
@@
 Text Label 13000 5200 0    50   ~ 0
 a8
-Text Label 13000 5100 0    50   ~ 0
+Text Label 13000 5900 0    50   ~ 0
 a7
-Text Label 13000 5000 0    50   ~ 0
+Text Label 13000 6200 0    50   ~ 0
 a6
-Text Label 13000 4900 0    50   ~ 0
+Text Label 13000 5700 0    50   ~ 0
 a5
-Text Label 13000 4800 0    50   ~ 0
+Text Label 13000 5500 0    50   ~ 0
 a4
 Text Label 13000 4700 0    50   ~ 0
@@
 Wire Bus Line
 	12900 1200 12900 2350
-Connection ~ 12900 2350
 Text Label 14350 4400 0    50   ~ 0
 d0
@@
 	1    0    0    -1
 $EndComp
-Text Label 12900 2500 3    50   ~ 0
+Text Label 12900 2350 3    50   ~ 0
 a[0..15]
 Text Label 10850 1200 2    50   ~ 0
 d[0..7]
-Text Label 11050 5350 2    50   ~ 0
+Text Label 9000 5300 3    50   ~ 0
 f[0..7]
 Wire Bus Line
@@
 	1    0    0    -1
 $EndComp
+Text Notes 7400 11150 2    50   ~ 0
+access
+Text Notes 11450 12850 2    50   ~ 0
+enabled
+Wire Bus Line
+	9000 4700 9000 6900
+$Comp
+L Device:C C18
+U 1 1 61FBFFD0
+P 14800 5950
+F 0 "C18" H 14915 5996 50  0000 L CNN
+F 1 "0.1" H 14915 5905 50  0000 L CNN
+F 2 "Capacitor_SMD:C_0805_2012Metric" H 14838 5800 50  0001 C CNN
+F 3 "~" H 14800 5950 50  0001 C CNN
+	1    14800 5950
+	1    0    0    -1
+$EndComp
+$Comp
+L power:GND #PWR0105
+U 1 1 61FBFFD6
+P 14800 6100
+F 0 "#PWR0105" H 14800 5850 50  0001 C CNN
+F 1 "GND" H 14805 5927 50  0000 C CNN
+F 2 "" H 14800 6100 50  0001 C CNN
+F 3 "" H 14800 6100 50  0001 C CNN
+	1    14800 6100
+	1    0    0    -1
+$EndComp
+$Comp
+L power:VCC #PWR0104
+U 1 1 61FBFFDC
+P 14800 5800
+F 0 "#PWR0104" H 14800 5650 50  0001 C CNN
+F 1 "VCC" H 14815 5973 50  0000 C CNN
+F 2 "" H 14800 5800 50  0001 C CNN
+F 3 "" H 14800 5800 50  0001 C CNN
+	1    14800 5800
+	1    0    0    -1
+$EndComp
 Wire Bus Line
 	10000 1200 11400 1200
@@
 	11900 2350 12900 2350
 Wire Bus Line
-	12900 5350 12900 6100
-Wire Bus Line
 	11700 1200 12900 1200
 Wire Bus Line
 	14650 3050 14650 5200
-Wire Bus Line
-	12900 2350 12900 5300
-Text Notes 7400 11150 2    50   ~ 0
-access
-Text Notes 11450 12850 2    50   ~ 0
-enabled
 $EndSCHEMATC
