File: boards/eth/eth.kicad_pcb (KiCad board)
At the start: 4 copper layers, 100 x 100 mm, 88 parts, among them J1 Conn_02x20_Odd_Even, J2 eth-phy-shield-conn, U1 74HC04, U10 74HC74, U11 74HC74, U12 74HC161, U13 74HC157, U14 74HC4040, U15 74HC157, U16 74HC157, U17 74HC157, U18 74HC157, U19 74HC157, U2 74HC21, U20 6116, U21 74HC244, U22 6116, U23 74HC244, U24 74HC273, U25 74HC244, U26 74HC244, U27 74HC244, U28 74HC165, U29 74HC74, U3 74HC74, U30 74HC161, U31 74HC4040, U32 74HC164, U33 74HC86, U34 74HC21, U35 74HC21, U36 74HC74, U4 74HC139, U5 74HC32, U6 74HC08, U7 74HC32, U8 74HC08, U9 74HC04, X1 20 MHz

Commit message: Eth: board
Parts:
- added C39: 0.1, Capacitor_SMD:C_0805_2012Metric, F.Cu at (115.8, 42.5)
- added D5: LED, LED_SMD:LED_0805_2012Metric, F.Cu at (108.1, 108.9)
- added D6: LED, LED_SMD:LED_0805_2012Metric, F.Cu at (108.1, 111.0)
- added D7: BAT74, Package_TO_SOT_SMD:SOT-143, F.Cu at (175.8, 32.9)
- added R4: 500, Resistor_SMD:R_0805_2012Metric, F.Cu at (104.5, 111.0)
- added R5: 500, Resistor_SMD:R_0805_2012Metric, F.Cu at (104.5, 108.9)
- added R6: 1k, Resistor_SMD:R_0805_2012Metric, F.Cu at (179.7, 31.8)
- added REF**: OSHW-Logo2_7.3x6mm_Copper, Symbol:OSHW-Logo2_7.3x6mm_Copper, F.Cu at (104.3, 44.5)
- added TP1: GND, TestPoint:TestPoint_THTPad_D2.0mm_Drill1.0mm, F.Cu at (103.2, 117.4)
- added TP2: GND, TestPoint:TestPoint_THTPad_D2.0mm_Drill1.0mm, F.Cu at (140.0, 37.9)
- added TP3: GND, TestPoint:TestPoint_THTPad_D2.0mm_Drill1.0mm, F.Cu at (197.4, 68.9)
- added TP4: GND, TestPoint:TestPoint_THTPad_D2.0mm_Drill1.0mm, F.Cu at (187.8, 127.7)
- added U37: 74HC04, Package_SO:TSSOP-14_4.4x5mm_P0.65mm, F.Cu at (111.7, 46.6)
- C1: value C_Polarized -> 33.0x10v; footprint Capacitor_Tantalum_SMD:CP_EIA-2012-12_Kemet-R -> Capacitor_SMD:C_1210_3225Metric
- X1: value 20 MHz -> CB3-3C-20M; footprint Oscillator:Oscillator_SMD_EuroQuartz_XO32-4Pin_3.2x2.5mm -> Oscillator:Oscillator_SMD_EuroQuartz_XO91-4Pin_7.0x5.0mm
- moved C38 322.7 mm to (111.0, 119.3), turned to 90 degrees
- moved C37 309.0 mm to (126.5, 120.4), turned to 90 degrees
- moved C36 307.3 mm to (124.7, 105.2)
- moved C35 299.4 mm to (139.7, 123.2)
- moved C1 298.3 mm to (108.8, 52.1), turned to 180 degrees
- moved R1 293.3 mm to (114.8, 114.8), turned to 90 degrees
- moved X1 293.3 mm to (114.7, 124.9)
- moved C34 291.2 mm to (146.3, 114.3)
- moved R2 282.0 mm to (126.0, 115.6)
- moved R3 275.8 mm to (131.8, 116.1)
- moved C28 271.2 mm to (122.8, 51.3)
- moved D4 269.9 mm to (122.9, 118.9)
- moved D1 265.8 mm to (113.8, 111.0)
- moved C21 263.8 mm to (124.7, 94.7)
- moved D2 261.9 mm to (122.2, 114.6)
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Connections:
- U1 pad 1: /~{recv_ss} -> GND
- U1 pad 12: /~{rearm_sched} -> unconnected-(U1-Pad12)
- U1 pad 13: /rearm_sched -> VCC
- U1 pad 2: /recv_ss -> unconnected-(U1-Pad2)
- U22 pad 10: /tx_d1 -> /tx_d5
- U22 pad 11: /tx_d2 -> /tx_d6
- U22 pad 13: /tx_d3 -> /tx_d7
- U22 pad 14: /tx_d4 -> /tx_d0
- U22 pad 15: /tx_d5 -> /tx_d1
- U22 pad 16: /tx_d6 -> /tx_d2
- U22 pad 17: /tx_d7 -> /tx_d3
- U22 pad 9: /tx_d0 -> /tx_d4
- U24 pad 13: /tx_d3 -> /tx_d0
- U24 pad 14: /tx_d2 -> /tx_d1
- U24 pad 17: /tx_d1 -> /tx_d2
- U24 pad 18: /tx_d0 -> /tx_d3
- U24 pad 2: /tx_buf_d0 -> /tx_buf_d3
- U24 pad 5: /tx_buf_d1 -> /tx_buf_d2
- U24 pad 6: /tx_buf_d2 -> /tx_buf_d1
- U24 pad 9: /tx_buf_d3 -> /tx_buf_d0
- U5 pad 1: /filter/d_4320_mac -> GND
- U5 pad 2: /filter/d_4320_set -> GND
- U5 pad 3: /filter/d_4320_ok -> unconnected-(U5-Pad3)
- U6 pad 10: /~{rearm} -> /~{clr_frame_received}
- U6 pad 11: /~{recv_rst} -> /~{clr_frame_received}
- U6 pad 12: /~{clr_frame_received} -> /~{rst}
- U6 pad 13: /~{inhibit} -> /~{rearm}
- U6 pad 8: /~{clr_frame_received} -> /~{recv_rst}
- U6 pad 9: /~{rst} -> /~{inhibit}
- U7 pad 12: GND -> VCC
- U7 pad 13: GND -> VCC
- U9 pad 1: /~{recv_rst} -> GND
- U9 pad 2: /receiver/rst -> unconnected-(U9-Pad2)
- U9 pad 3: /receiver/bit_count2 -> /rearm_sched
- U9 pad 4: /receiver/~{bit_count_2} -> /~{rearm_sched}
Routing:
- net /recv_ss: track 0.00 -> 288.3 mm, vias 0 -> 22
- net /recv_sck_ena: track 0.00 -> 179.5 mm, vias 0 -> 8
- net /recv_byte_cnt2: track 0.00 -> 158.1 mm, vias 0 -> 11
- net VCC: track 0.00 -> 152.6 mm, vias 0 -> 59
- net /~{tx_buf_we}: track 0.00 -> 150.2 mm, vias 0 -> 12
- net /~{tx_halt}: track 0.00 -> 147.4 mm, vias 0 -> 8
- net /recv_byte_cnt0: track 0.00 -> 144.0 mm, vias 0 -> 9
- net /~{rearm}: track 0.00 -> 142.8 mm, vias 0 -> 8
- net GND: track 0.00 -> 141.2 mm, vias 0 -> 103
- net /~{oe}: track 0.00 -> 140.3 mm, vias 0 -> 7
- net /~{we}: track 0.00 -> 136.3 mm, vias 0 -> 8
- net /~{recv_ss}: track 0.00 -> 131.7 mm, vias 0 -> 9
- net /~{a_buf_sel}: track 0.00 -> 129.5 mm, vias 0 -> 11
- net /~{inhibit}: track 0.00 -> 128.1 mm, vias 0 -> 11
- net /recv_byte_cnt1: track 0.00 -> 124.2 mm, vias 0 -> 7
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- added copper zone on In1.Cu, net GND
- added copper zone on In2.Cu, net VCC
Other:
- board text added: "+"
- board text added: "Eth rev.1"
- board text added: "Licensed under the TAPR Open Hardware License (www.tapr.org/OHL)"
