File: boards/eth/eth.kicad_sch (KiCad schematic)
At the start: 9 parts, among them J1 partial-nucleo64, U1 74HC4040, U2 74HC157, U3 74HC157, U4 74HC164, U5 74HC157, U6 6116, U7 74HC244, U8 74HC244

Commit message: Eth: test normal operation
Parts:
- added U10, U9: 74HC244, symbol 74xx:74HC244
Connections:
- net D0: now also U10.18 (1Y0), U10.3 (2Y0), U9.18 (1Y0)
- net D1: now also U10.16 (1Y1), U10.5 (2Y1), U9.16 (1Y1)
- net D2: now also U10.14 (1Y2), U9.14 (1Y2)
- net D3: now also U9.12 (1Y3)
- net D4: now also U9.3 (2Y0)
- net D5: now also U9.5 (2Y1)
- net D6: now also U9.7 (2Y2)
- net D7: now also U9.9 (2Y3)
- net GND: now also J1.GND, U10.10 (GND), U10.11 (2A3), U10.13 (2A2), U10.8 (1A3), U9.10 (GND)
- net VCC: now also J1.+5V, U10.20 (VCC), U9.20 (VCC)
- net recv_byte_cnt0: now also U9.2 (1A0)
- net recv_byte_cnt1: now also U9.4 (1A1)
- net recv_byte_cnt10: now also U10.6 (1A2)
- net recv_byte_cnt2: now also U9.6 (1A2)
- net recv_byte_cnt3: now also U9.8 (1A3)
- net recv_byte_cnt4: now also U9.17 (2A0)
- net recv_byte_cnt5: now also U9.15 (2A1)
- net recv_byte_cnt6: now also U9.13 (2A2)
- net recv_byte_cnt7: now also U9.11 (2A3)
- net recv_byte_cnt8: now also U10.2 (1A0)
- net recv_byte_cnt9: now also U10.4 (1A1)

Commit message: Eth: receiver schematic
Parts:
- removed J1: partial-nucleo64, schield:partial-nucleo64, symbol shield:partial-nucleo64
- removed U1: 74HC4040, symbol eth:74HC4040
- removed U4: 74HC164, symbol 74xx:74HC164
- added C10, C11, C12, C13, C14, C15, C16, C17, C18, C19, C20, C21, C22, C23, C24, C25, C27: 0.1, symbol Device:C_Small
- added C26: C_Polarized, symbol Device:C_Polarized
- added D1, D2, D3, D4: D, symbol Device:D
- added J1: Conn_02x20_Odd_Even, symbol Connector_Generic:Conn_02x20_Odd_Even
- added J2: eth-phy-shield-conn, schield:partial-nucleo64, symbol shield:partial-nucleo64
- added R1, R2: 1k, symbol Device:R
- added U1, U17: 74HC04, symbol 74xx:74HC04
- added U2: 74HC21, symbol 74xx:74LS21
- added U25, U7: 74HC08, symbol 74xx:74LS08
- added U26, U3: 74HC32, symbol 74xx:74LS32
- added U4: 74HC139, symbol 74xx:74LS139
- added U5, U6: 74HC74, symbol 74xx:74HC74
- renumbered U5 to U10, U6 to U11, U7 to U12, U8 to U13, U9 to U14, U10 to U15, U2 to U8, U3 to U9
Connections:
- net GND: now also U11.18 (~{CS}), C10.2, C11.2, C12.2, C13.2, C14.2, C15.2, C16.2, C17.2, C18.2, C19.2, C20.2, C21.2, C22.2, C23.2, C24.2, C25.2, C26.2, C27.2, J1.2 (Pin_2), J1.39 (Pin_39), J2.GND, U1.7 (GND), U17.11, U17.13, U17.5, U17.7 (GND), U17.9, U2.7 (GND), U25.10, U25.12, U25.13, U25.4, U25.5, U25.7 (GND), U25.9, U26.10, U26.12, U26.13, U26.7 (GND), U26.9, U3.12, U3.13, U3.7 (GND), U4.8 (GND), U5.10 (~{S}), U5.11 (C), U5.12 (D), U5.13 (~{R}), U5.2 (D), U5.3 (C), U5.7 (GND), U7.7 (GND)
- net VCC: now also C10.1, C11.1, C12.1, C13.1, C14.1, C15.1, C16.1, C17.1, C18.1, C19.1, C20.1, C21.1, C22.1, C23.1, C24.1, C25.1, C26.1, C27.1, J1.1 (Pin_1), J1.40 (Pin_40), J2.+5V, R1.1, R2.2, U1.14 (VCC), U17.14 (VCC), U2.14 (VCC), U25.14 (VCC), U26.14 (VCC), U3.14 (VCC), U4.16 (VCC), U5.14 (VCC), U6.10 (~{S}), U7.14 (VCC)
- net a0: now also J1.23 (Pin_23), U4.14 (A0), U4.2 (A0)
- net a1: now also J1.24 (Pin_24), U4.3 (A1)
- net a10: now also J1.33 (Pin_33), U1.3
- net a2: now also J1.25 (Pin_25)
- net a3: now also J1.26 (Pin_26)
- net a4: now also J1.27 (Pin_27)
- net a5: now also J1.28 (Pin_28)
- net a6: now also J1.29 (Pin_29)
- net a7: now also J1.30 (Pin_30)
- net a8: now also J1.31 (Pin_31), U2.12
- net a9: now also J1.32 (Pin_32), U2.10
- net recv_mosi: now also J2.PB13
- net recv_sck: now also J2.PB15
- net send_mosi: now also J2.PC12
- net send_sck: now also J2.PC10
- net ~{recv_ss}: now also U12.1 (1OE), U12.19 (2OE), J2.PC6, U1.1, U6.11 (C)
- net recv_a_sel: now reaches U10.1 (S)
- net recv_a_sel: now also U8.1 (S), U9.1 (S), U25.3, U26.5
- net ~{recv_byte_cnt_hi_oe}: now reaches U15.1 (1OE)
- net ~{recv_byte_cnt_hi_oe}: now also U4.7 (O3)
- net buf_full: now reaches U15.17 (2A0)
- net buf_full: now also U6.9 (Q)
- net ~{oe_cr_to_d}: now reaches U15.19 (2OE)
- net ~{oe_cr_to_d}: now also U4.4 (O0)
- net ~{recv_buf_oe}: now reaches U11.20 (~{OE})
- net ~{recv_buf_oe}: now also U26.6
- net ~{recv_buf_we}: now reaches U11.21 (~{WE})
- net ~{recv_byte_cnt_lo_oe}: now reaches U14.1 (1OE)
- net ~{recv_byte_cnt_lo_oe}: now also U14.19 (2OE), U4.6 (O2)
- net ~{recv_d_oe}: now reaches U13.1 (1OE)
- net ~{recv_d_oe}: now also U13.19 (2OE), U26.3, U26.4
- net D0 renamed d0
- net d0: now also J1.11 (Pin_11)
- net D1 renamed d1
- net d1: now also J1.12 (Pin_12)
- net D2 renamed d2
- net d2: now also J1.13 (Pin_13)
- net D3 renamed d3
- net d3: now also J1.14 (Pin_14)
- net D4 renamed d4
- net d4: now also J1.15 (Pin_15)
- net D5 renamed d5
- net d5: now also J1.16 (Pin_16)
- net D6 renamed d6
- net d6: now also J1.17 (Pin_17)
- net D7 renamed d7
- net d7: now also J1.18 (Pin_18)
- new net: D1.2 (A), D2.2 (A), R1.2, U1.5
- new net: D3.2 (A), D4.2 (A), R2.1, U1.11
- new net: U3.6, U4.1 (E)
- new net a11: J1.34 (Pin_34), U1.9, U2.9
- new net a12: J1.35 (Pin_35), U2.5
- new net a13: J1.36 (Pin_36), U2.4
- new net a14: J1.37 (Pin_37), U2.2
- new net a15: J1.38 (Pin_38), U2.1
- new net a_89nab_set: D1.1 (K), U2.8
- new net a_cdef_set: D2.1 (K), D3.1 (K), U2.6
- new net rdy: J1.5 (Pin_5)
- new net rearm_sched: U1.13, U5.5 (Q)
- new net recv_sck_ena: U25.2, U6.8 (~{Q})
- new net recv_ss: U1.2, U25.1, U3.10, U5.1 (~{R})
- new net ~{a10}: U1.4, U2.13
- new net ~{a11}: D4.1 (K), U1.8
- new net ~{a_buf_sel}: U1.10, U26.1
- new net ~{a_fbxx}: U1.6, U3.4, U4.13 (A1)
- new net ~{clr_frame_received}: U6.13 (~{R}), U7.12, U7.8
- new net ~{inhibit}: U6.12 (D), U7.13
- new net ~{oe}: J1.7 (Pin_7), U26.2, U3.5
- new net ~{rearm_req}: U4.12 (O0), U5.4 (~{S})
- new net ~{rearm_sched}: U1.12, U3.9
- new net ~{rearm}: U3.8, U7.10
- new net ~{recv_rst}: U7.11
- new net ~{rst}: J1.4 (Pin_4), U7.9
- new net ~{we}: J1.8 (Pin_8), U4.15 (E)
- no-connect marks 1 -> 29
Other:
- added sheet filter (filter.kicad_sch)
- added sheet receiver (receiver.kicad_sch)
- moved on the sheet: U10, U11, U12, U13, U14, U15, U8, U9

Commit message: Eth: begin transmission
Parts:
- added U19: 74HC4040, symbol eth:74HC4040
- added U27: 6116, symbol eth:6116
- added U28, U29, U30: 74HC157, symbol 74xx:74LS157
- added U31: 74HC244, symbol 74xx:74HC244
- added U33: 74HC165, symbol 74xx:74HC165
Connections:
- net GND: now also U19.8 (GND), U27.12 (GND), U27.18 (~{CS}), U27.19 (A10), U28.15 (E), U28.8 (GND), U29.15 (E), U29.8 (GND), U30.10 (I1c), U30.11 (I0c), U30.13 (I1d), U30.14 (I0d), U30.15 (E), U30.8 (GND), U31.10 (GND), U33.8 (GND)
- net VCC: now also U19.16 (VCC), U27.24 (VCC), U28.16 (VCC), U29.16 (VCC), U30.16 (VCC), U31.20 (VCC), U33.16 (VCC)
- net a0: now also U28.2 (I0a)
- net a1: now also U28.5 (I0b)
- net a2: now also U28.11 (I0c)
- net a3: now also U28.14 (I0d)
- net a4: now also U29.2 (I0a)
- net a5: now also U29.5 (I0b)
- net a6: now also U29.11 (I0c)
- net a7: now also U29.14 (I0d)
- net a8: now also U30.2 (I0a)
- net a9: now also U30.5 (I0b)
- net d0: now also U31.2 (1A0)
- net d1: now also U31.4 (1A1)
- net d2: now also U31.6 (1A2)
- net d3: now also U31.8 (1A3)
- net d4: now also U31.17 (2A0)
- net d5: now also U31.15 (2A1)
- net d6: now also U31.13 (2A2)
- net d7: now also U31.11 (2A3)
- new net tx_a0: U27.8 (A0), U28.4 (Za)
- new net tx_a1: U27.7 (A1), U28.7 (Zb)
- new net tx_a2: U27.6 (A2), U28.9 (Zc)
- new net tx_a3: U27.5 (A3), U28.12 (Zd)
- new net tx_a4: U27.4 (A4), U29.4 (Za)
- new net tx_a5: U27.3 (A5), U29.7 (Zb)
- new net tx_a6: U27.2 (A6), U29.9 (Zc)
- new net tx_a7: U27.1 (A7), U29.12 (Zd)
- new net tx_a8: U27.23 (A8), U30.4 (Za)
- new net tx_a9: U27.22 (A9), U30.7 (Zb)
- new net tx_byte_cnt0: U19.9 (Q0), U28.3 (I1a)
- new net tx_byte_cnt1: U19.7 (Q1), U28.6 (I1b)
- new net tx_byte_cnt2: U19.6 (Q2), U28.10 (I1c)
- new net tx_byte_cnt3: U19.5 (Q3), U28.13 (I1d)
- new net tx_byte_cnt4: U19.3 (Q4), U29.3 (I1a)
- new net tx_byte_cnt5: U19.2 (Q5), U29.6 (I1b)
- new net tx_byte_cnt6: U19.4 (Q6), U29.10 (I1c)
- new net tx_byte_cnt7: U19.13 (Q7), U29.13 (I1d)
- new net tx_byte_cnt8: U19.12 (Q8), U30.3 (I1a)
- new net tx_byte_cnt9: U19.14 (Q9), U30.6 (I1b)
- new net tx_d0: U27.9 (D0), U31.18 (1Y0), U33.6 (D7)
- new net tx_d1: U27.10 (D1), U31.16 (1Y1), U33.5 (D6)
- new net tx_d2: U27.11 (D2), U31.14 (1Y2), U33.4 (D5)
- new net tx_d3: U27.13 (D3), U31.12 (1Y3), U33.3 (D4)
- new net tx_d4: U27.14 (D4), U31.3 (2Y0), U33.14 (D3)
- new net tx_d5: U27.15 (D5), U31.5 (2Y1), U33.13 (D2)
- new net tx_d6: U27.16 (D6), U31.7 (2Y2), U33.12 (D1)
- new net tx_d7: U27.17 (D7), U31.9 (2Y3), U33.11 (D0)
- no-connect marks 29 -> 31
Other:
- moved on the sheet: U17C, U17D, U17E, U17F, U25B, U25C, U25D, U26C, U26D, U3D, U5B

Commit message: Eth: transmitter schematics finished
Parts:
- added C28, C29, C30, C31, C32, C33, C34, C35, C36, C37, C38: 0.1, symbol Device:C_Small
- added D5, D6, D7, D8: D, symbol Device:D_Small
- added H1, H2, H3, H4: MountingHole, symbol Mechanical:MountingHole
- added R3: 1k, symbol Device:R_Small
- added U34: 74HC161, symbol 74xx:74LS161
- added U35: 74HC273, symbol 74xx:74HC273
- added U36: 74HC74, symbol 74xx:74HC74
- added X1: 20 MHz, Oscillator:Oscillator_SMD_EuroQuartz_XO32-4Pin_3.2x2.5mm, symbol Oscillator:XO32
Connections:
- net send_sck is gone; now on net tx_sck: J2.PC10
- net GND: now also U33.10 (DS), U33.15 (~{CE}), C28.2, C29.2, C30.2, C31.2, C32.2, C33.2, C34.2, C35.2, C36.2, C37.2, C38.2, R3.2, U34.3 (D0), U34.4 (D1), U34.5 (D2), U34.6 (D3), U34.8 (GND), U35.10 (GND), U36.7 (GND), X1.2 (GND); no longer U17.11, U17.5, U17.9, U25.10, U25.12, U25.13, U25.4, U25.5, U25.9, U26.10, U26.9, U5.10 (~{S}), U5.11 (C), U5.13 (~{R})
- net VCC: now also U5.13 (~{R}), C28.1, C29.1, C30.1, C31.1, C32.1, C33.1, C34.1, C35.1, C36.1, C37.1, C38.1, U34.10 (CET), U34.16 (VCC), U34.7 (CEP), U34.9 (~{PE}), U35.1 (~{Mr}), U35.20 (VCC), U36.10 (~{S}), U36.12 (D), U36.14 (VCC), U36.4 (~{S}), X1.1 (EN), X1.4 (V+)
- net tx_byte_cnt0: now also U36.11 (C)
- net tx_d0: now also U35.18 (D7); no longer U33.6 (D7)
- net tx_d1: now also U35.17 (D6); no longer U33.5 (D6)
- net tx_d2: now also U35.14 (D5); no longer U33.4 (D5)
- net tx_d3: now also U35.13 (D4); no longer U33.3 (D4)
- net tx_d4: now also U35.8 (D3); no longer U33.14 (D3)
- net tx_d5: now also U35.7 (D2); no longer U33.13 (D2)
- net tx_d6: now also U35.4 (D1); no longer U33.12 (D1)
- net tx_d7: now also U35.3 (D0); no longer U33.11 (D0)
- net ~{a_buf_sel}: now also U26.9
- net ~{rst}: now also U25.13
- net ~{we}: now also U26.10
- net ~{tx_halt_set}: now reaches U25.11
- net ~{tx_halt_set}: now also U5.10 (~{S})
- net ~{tx_buf_oe}: now reaches U17.8
- net ~{tx_buf_oe}: now also U27.20 (~{OE})
- net ~{tx_buf_we}: now reaches U30.1 (S)
- net ~{tx_buf_we}: now also U17.9, U26.8, U27.21 (~{WE}), U28.1 (S), U29.1 (S), U31.1 (1OE), U31.19 (2OE)
- net ~{tx_byte_clk}: now reaches U19.10 (CP)
- net ~{tx_byte_clk}: now also U25.9, U34.15 (TC)
- net tx_halt: now reaches U19.11 (MR)
- net tx_halt: now also U5.9 (Q)
- net tx_byte_cnt10: now reaches U19.15 (Q10)
- net tx_byte_cnt10: now also U25.10
- net ~{n_reg_oe_ena}: now reaches U3.6, U4.1 (E)
- net ~{tx_halt}: now reaches U15.15 (2A1)
- net ~{tx_halt}: now also U5.8 (~{Q}), U34.1 (~{MR}), U36.13 (~{R})
- net tx_finish: now reaches U25.8
- net tx_finish: now also U17.11
- net ~{tx_req}: now reaches U4.11 (O1)
- net ~{tx_req}: now also U5.11 (C)
- net ~{tx_shift_pl}: now reaches U33.1 (~{PL})
- net ~{tx_shift_pl}: now also D5.1 (K), D6.1 (K), D7.1 (K), D8.1 (K), R3.1
- net tx_shift_cp: now reaches U33.2 (CP)
- net tx_shift_cp: now also U17.6
- net tx_shift_q7: now reaches U33.9 (Q7)
- net tx_shift_q7: now also U36.2 (D)
- net ~{tx_finish}: now reaches U17.10
- net ~{tx_finish}: now also U25.12
- net tx_sck: now reaches U25.6
- net send_mosi renamed tx_mosi
- net tx_mosi: now also U36.5 (Q)
- new net tx_buf_d0: U33.11 (D0), U35.2 (Q0)
- new net tx_buf_d1: U33.12 (D1), U35.5 (Q1)
- new net tx_buf_d2: U33.13 (D2), U35.6 (Q2)
- new net tx_buf_d3: U33.14 (D3), U35.9 (Q3)
- new net tx_buf_d4: U33.3 (D4), U35.12 (Q4)
- new net tx_buf_d5: U33.4 (D5), U35.15 (Q5)
- new net tx_buf_d6: U33.5 (D6), U35.16 (Q6)
- new net tx_buf_d7: U33.6 (D7), U35.19 (Q7)
- new net tx_cnt0: D5.2 (A), U17.5, U25.4, U34.14 (Q0), U36.3 (C)
- new net tx_cnt1: D6.2 (A), U34.13 (Q1)
- new net tx_cnt2: D7.2 (A), U34.12 (Q2)
- new net tx_cnt3: D8.2 (A), U34.11 (Q3), U35.11 (Cp)
- new net tx_cp_in: U34.2 (CP), X1.3 (OUT)
- new net tx_oe: U25.5, U36.1 (~{R}), U36.9 (Q)
- no-connect marks 31 -> 26
Other:
- note added: "bus bits in reverse order"
- note added: "shift"
- note added: "tx_halt"
- note added: "tx_oe"
- moved on the sheet: C11, U17C, U17D, U17E, U17F, U25B, U25C, U25D, U26A, U26B, U26C, U26D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

Commit message: Eth: schematics checked
Parts:
- removed D1, D2, D3, D4: D, symbol Device:D
- removed D5, D6, D7, D8: D, symbol Device:D_Small
- added D1, D2, D3, D4: BAT74, Package_TO_SOT_SMD:SOT-143, symbol eth:BAT74
- C1: renamed from C26; footprint (none) -> Capacitor_Tantalum_SMD:CP_EIA-2012-12_Kemet-R
- C10: renamed from C29; footprint (none) -> Capacitor_SMD:C_0805_2012Metric
- C11: renamed from C27; footprint (none) -> Capacitor_SMD:C_0805_2012Metric
- C12: renamed from C28; footprint (none) -> Capacitor_SMD:C_0805_2012Metric
- C13: renamed from C30; footprint (none) -> Capacitor_SMD:C_0805_2012Metric
- C14: renamed from C11; footprint (none) -> Capacitor_SMD:C_0805_2012Metric
- C15: renamed from C31; footprint (none) -> Capacitor_SMD:C_0805_2012Metric
- C16: renamed from C38; footprint (none) -> Capacitor_SMD:C_0805_2012Metric
- C17: renamed from C10; footprint (none) -> Capacitor_SMD:C_0805_2012Metric
- C18: renamed from C37; footprint (none) -> Capacitor_SMD:C_0805_2012Metric
- C19: renamed from C12; footprint (none) -> Capacitor_SMD:C_0805_2012Metric
- C2: renamed from C18; footprint (none) -> Capacitor_SMD:C_0805_2012Metric
- C20: renamed from C36; footprint (none) -> Capacitor_SMD:C_0805_2012Metric
- C21: renamed from C13; footprint (none) -> Capacitor_SMD:C_0805_2012Metric
- C22: renamed from C35; footprint (none) -> Capacitor_SMD:C_0805_2012Metric
- C23: renamed from C14; footprint (none) -> Capacitor_SMD:C_0805_2012Metric
- C24: renamed from C34; footprint (none) -> Capacitor_SMD:C_0805_2012Metric
- C25: renamed from C15; footprint (none) -> Capacitor_SMD:C_0805_2012Metric
- C26: renamed from C33; footprint (none) -> Capacitor_SMD:C_0805_2012Metric
- C27: renamed from C16; footprint (none) -> Capacitor_SMD:C_0805_2012Metric
- C28: renamed from C17; footprint (none) -> Capacitor_SMD:C_0805_2012Metric
- C29: renamed from C32; footprint (none) -> Capacitor_SMD:C_0805_2012Metric
- C3: renamed from C19; footprint (none) -> Capacitor_SMD:C_0805_2012Metric
- C4: renamed from C20; footprint (none) -> Capacitor_SMD:C_0805_2012Metric
- C5: renamed from C21; footprint (none) -> Capacitor_SMD:C_0805_2012Metric
- C6: renamed from C22; footprint (none) -> Capacitor_SMD:C_0805_2012Metric
- C7: renamed from C23; footprint (none) -> Capacitor_SMD:C_0805_2012Metric
- C8: renamed from C24; footprint (none) -> Capacitor_SMD:C_0805_2012Metric
- C9: renamed from C25; footprint (none) -> Capacitor_SMD:C_0805_2012Metric
- H1, H4: footprint (none) -> MountingHole:MountingHole_3.2mm_M3
- H2: renamed from H3; footprint (none) -> MountingHole:MountingHole_3.2mm_M3
- H3: renamed from H2; footprint (none) -> MountingHole:MountingHole_3.2mm_M3
- J1: footprint (none) -> Connector_PinHeader_2.54mm:PinHeader_2x20_P2.54mm_Horizontal
- R1, R2, R3: footprint (none) -> Resistor_SMD:R_0805_2012Metric
- U1, U2: footprint (none) -> Package_SO:TSSOP-14_4.4x5mm_P0.65mm
- U10: renamed from U6; footprint (none) -> Package_SO:TSSOP-14_4.4x5mm_P0.65mm
- U11: renamed from U36; footprint (none) -> Package_SO:TSSOP-14_4.4x5mm_P0.65mm
- U12: renamed from U34; footprint (none) -> Package_SO:TSSOP-16_4.4x5mm_P0.65mm
- U13: renamed from U8; footprint (none) -> Package_SO:TSSOP-16_4.4x5mm_P0.65mm
- U15: renamed from U28; footprint (none) -> Package_SO:TSSOP-16_4.4x5mm_P0.65mm
- U16: renamed from U9; footprint (none) -> Package_SO:TSSOP-16_4.4x5mm_P0.65mm
- U17: renamed from U29; footprint (none) -> Package_SO:TSSOP-16_4.4x5mm_P0.65mm
- U18: renamed from U10; footprint (none) -> Package_SO:TSSOP-16_4.4x5mm_P0.65mm
- U19: renamed from U30; footprint (none) -> Package_SO:TSSOP-16_4.4x5mm_P0.65mm
- U19, U4: footprint (none) -> Package_SO:TSSOP-16_4.4x5mm_P0.65mm
- U20: renamed from U11; footprint (none) -> Package_SO:SOIC-24W_7.5x15.4mm_P1.27mm
- U21: renamed from U12; footprint (none) -> Package_SO:TSSOP-20_4.4x6.5mm_P0.65mm
- U22: renamed from U27; footprint (none) -> Package_SO:SOIC-24W_7.5x15.4mm_P1.27mm
- U23: renamed from U31; footprint (none) -> Package_SO:TSSOP-20_4.4x6.5mm_P0.65mm
- U24: renamed from U35; footprint (none) -> Package_SO:TSSOP-20_4.4x6.5mm_P0.65mm
- U25: renamed from U13; footprint (none) -> Package_SO:TSSOP-20_4.4x6.5mm_P0.65mm
- U26: renamed from U14; footprint (none) -> Package_SO:TSSOP-20_4.4x6.5mm_P0.65mm
- U27: renamed from U15; footprint (none) -> Package_SO:TSSOP-20_4.4x6.5mm_P0.65mm
- U28: renamed from U33; footprint (none) -> Package_SO:TSSOP-16_4.4x5mm_P0.65mm
- U3: renamed from U5; footprint (none) -> Package_SO:TSSOP-14_4.4x5mm_P0.65mm
- U5: renamed from U3; footprint (none) -> Package_SO:TSSOP-14_4.4x5mm_P0.65mm
- U6: renamed from U7; footprint (none) -> Package_SO:TSSOP-14_4.4x5mm_P0.65mm
- U7: renamed from U26; footprint (none) -> Package_SO:TSSOP-14_4.4x5mm_P0.65mm
- U8: renamed from U25; footprint (none) -> Package_SO:TSSOP-14_4.4x5mm_P0.65mm
- U9: renamed from U17; footprint (none) -> Package_SO:TSSOP-14_4.4x5mm_P0.65mm
Connections:
- net a_89nab_set: now also D1.1 (C1)
- net a_cdef_set: now also D1.2 (C2), D2.1 (C1)
- net tx_cnt0: now also D3.4 (A1)
- net tx_cnt1: now also D3.3 (A2)
- net tx_cnt2: now also D4.3 (A2)
- net tx_cnt3: now also D4.4 (A1)
- net ~{a11}: now also D2.2 (C2)
- net ~{tx_shift_pl}: now also D3.1 (C1), D3.2 (C2), D4.1 (C1), D4.2 (C2)
- net at R1.2, U1.5: now also D1.3 (A2), D1.4 (A1)
- net at R2.1, U1.11: now also D2.3 (A2), D2.4 (A1)
- net ~{n_reg_oe_ena} renamed ~{reg_oe_ena}
Other:
- moved on the sheet: R3

Commit message: Eth: board dimensions
Parts:
- J2: footprint schield:partial-nucleo64 -> eth:partial-nucleo64
Changed lines of the file:
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@@
       (effects (font (size 1.27 1.27)))
     )
-    (property "Footprint" "schield:partial-nucleo64" (at 55.88 47.625 0)
+    (property "Footprint" "eth:partial-nucleo64" (at 55.88 47.625 0)
       (effects (font (size 1.27 1.27)) hide)
     )

Commit message: Eth: untangle schematic
Parts:
- added D5, D6: LED, LED_SMD:LED_0805_2012Metric, symbol Device:LED
- added R4, R5: 500, Resistor_SMD:R_0805_2012Metric, symbol Device:R
- added U37: 74HC04, Package_SO:TSSOP-14_4.4x5mm_P0.65mm, symbol 74xx:74HC04
- added unit 2 of U9
- added unit 1 of U9
- C1: value C_Polarized -> 33.0x10v; footprint Capacitor_Tantalum_SMD:CP_EIA-2012-12_Kemet-R -> Capacitor_SMD:C_1210_3225Metric
- X1: value 20 MHz -> CB3-3C-20M; footprint Oscillator:Oscillator_SMD_EuroQuartz_XO32-4Pin_3.2x2.5mm -> Oscillator:Oscillator_SMD_EuroQuartz_XO91-4Pin_7.0x5.0mm
Connections:
- net GND: now also U1.1, U9.1; no longer U7.12, U7.13
- net VCC: now also U1.13, U7.12, U7.13, R4.1, R5.2
- net rearm_sched: now also U9.3; no longer U1.13
- net recv_ss: now also U37.6; no longer U1.2
- net tx_buf_d0: now also U24.9 (Q3); no longer U24.2 (Q0)
- net tx_buf_d1: now also U24.6 (Q2); no longer U24.5 (Q1)
- net tx_buf_d2: now also U24.5 (Q1); no longer U24.6 (Q2)
- net tx_buf_d3: now also U24.2 (Q0); no longer U24.9 (Q3)
- net tx_d0: now also U22.14 (D4), U24.13 (D4); no longer U22.9 (D0), U24.18 (D7)
- net tx_d1: now also U22.15 (D5), U24.14 (D5); no longer U22.10 (D1), U24.17 (D6)
- net tx_d2: now also U22.16 (D6), U24.17 (D6); no longer U22.11 (D2), U24.14 (D5)
- net tx_d3: now also U22.17 (D7), U24.18 (D7); no longer U22.13 (D3), U24.13 (D4)
- net tx_d4: now also U22.9 (D0); no longer U22.14 (D4)
- net tx_d5: now also U22.10 (D1); no longer U22.15 (D5)
- net tx_d6: now also U22.11 (D2); no longer U22.16 (D6)
- net tx_d7: now also U22.13 (D3); no longer U22.17 (D7)
- net ~{a_buf_sel}: now also D6.1 (K)
- net ~{a_fbxx}: now also D5.1 (K)
- net ~{clr_frame_received}: now also U6.10, U6.11; no longer U6.12, U6.8
- net ~{inhibit}: now also U6.9; no longer U6.13
- net ~{rearm_sched}: now also U9.4; no longer U1.12
- net ~{rearm}: now also U6.13; no longer U6.10
- net ~{recv_rst}: now also U6.8; no longer U6.11
- net ~{recv_ss}: now also U37.5; no longer U1.1
- net ~{rst}: now also U6.12; no longer U6.9
- new net: D6.2 (A), R4.2
- new net: D5.2 (A), R5.1
- no-connect marks 26 -> 29
Other:
- moved on the sheet: U1A, U1F, U6C, U6D
