File: boards/eth/eth.kicad_sch (KiCad schematic)
At the start: 76 parts, among them J1 Conn_02x20_Odd_Even, J2 eth-phy-shield-conn, U1 74HC04, U10 74HC74, U11 74HC74, U12 74HC161, U13 74HC157, U15 74HC157, U16 74HC157, U17 74HC157, U18 74HC157, U19 74HC157, U19 74HC4040, U2 74HC21, U20 6116, U21 74HC244, U22 6116, U23 74HC244, U24 74HC273, U25 74HC244, U26 74HC244, U27 74HC244, U28 74HC165, U3 74HC74, U37 74HC04, U4 74HC139, U5 74HC32, U6 74HC08, U7 74HC32, U8 74HC08, U9 74HC04, X1 CB3-3C-20M

Commit message: Eth: board
Parts:
- added TP1, TP2, TP3, TP4: GND, TestPoint:TestPoint_THTPad_D2.0mm_Drill1.0mm, symbol Connector:TestPoint
Connections:
- net GND: now also TP1.1, TP2.1, TP3.1, TP4.1
Changed lines of the file:
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@@
     (date "2023-10-14")
     (rev "1")
+    (comment 1 "Licensed under the TAPR Open Hardware License (www.tapr.org/OHL)")
+    (comment 2 "Copyright 2023 Ivan Mikhailov")
   )
   (junction (at 144.145 148.59) (diameter 0) (color 0 0 0 0)
@@
     )
   )
+  (symbol (lib_id "Connector:TestPoint") (at 798.83 88.265 0) (unit 1)
+    (in_bom yes) (on_board yes) (dnp no)
+    (property "Reference" "TP4" (at 796.925 78.105 0)
+      (effects (font (size 1.27 1.27)) (justify left))
+    )
+    (property "Value" "GND" (at 796.925 81.28 0)
+      (effects (font (size 1.27 1.27)) (justify left))
+    )
+    (property "Footprint" "TestPoint:TestPoint_THTPad_D2.0mm_Drill1.0mm" (at 803.91 88.265 0)
+      (effects (font (size 1.27 1.27)) hide)
+    )
+    (property "Datasheet" "~" (at 803.91 88.265 0)
+      (effects (font (size 1.27 1.27)) hide)
+    )
+    (pin "1")
+    (instances
+      (project "eth"
+        (path "/25b810b6-8afb-4eb4-8eaf-dfe3b666cbdb"
+          (reference "TP4") (unit 1)
+        )
+      )
+    )
+  )
   (symbol (lib_id "power:VCC") (at 45.72 42.545 90) (unit 1)
     (in_bom yes) (on_board yes) (dnp no) (fields_autoplaced)
@@
     )
   )
+  (symbol (lib_id "power:GND") (at 778.51 88.265 0) (unit 1)
+    (in_bom yes) (on_board yes) (dnp no) (fields_autoplaced)
+    (property "Reference" "#PWR0156" (at 778.51 94.615 0)
+      (effects (font (size 1.27 1.27)) hide)
+    )
+    (property "Value" "GND" (at 778.51 93.345 0)
+      (effects (font (size 1.27 1.27)))
+    )
+    (property "Footprint" "" (at 778.51 88.265 0)
+      (effects (font (size 1.27 1.27)) hide)
+    )
+    (property "Datasheet" "" (at 778.51 88.265 0)
+      (effects (font (size 1.27 1.27)) hide)
+    )
+    (pin "1")
+    (instances
+      (project "eth"
+        (path "/25b810b6-8afb-4eb4-8eaf-dfe3b666cbdb"
+          (reference "#PWR0156") (unit 1)
+        )
+      )
+    )
+  )
   (symbol (lib_id "power:VCC") (at 393.7 542.925 90) (unit 1)
     (in_bom yes) (on_board yes) (dnp no) (fields_autoplaced)
@@
     )
   )
+  (symbol (lib_id "Connector:TestPoint") (at 785.495 88.265 0) (unit 1)
+    (in_bom yes) (on_board yes) (dnp no)
+    (property "Reference" "TP2" (at 783.59 78.105 0)
+      (effects (font (size 1.27 1.27)) (justify left))
+    )
+    (property "Value" "GND" (at 783.59 81.28 0)
+      (effects (font (size 1.27 1.27)) (justify left))
+    )
+    (property "Footprint" "TestPoint:TestPoint_THTPad_D2.0mm_Drill1.0mm" (at 790.575 88.265 0)
+      (effects (font (size 1.27 1.27)) hide)
+    )
+    (property "Datasheet" "~" (at 790.575 88.265 0)
+      (effects (font (size 1.27 1.27)) hide)
+    )
+    (pin "1")
+    (instances
+      (project "eth"
+        (path "/25b810b6-8afb-4eb4-8eaf-dfe3b666cbdb"
+          (reference "TP2") (unit 1)
+        )
+      )
+    )
+  )
   (symbol (lib_id "74xx:74LS161") (at 300.355 380.365 0) (unit 1)
     (in_bom yes) (on_board yes) (dnp no) (fields_autoplaced)
@@
     )
   )
+  (symbol (lib_id "Connector:TestPoint") (at 778.51 88.265 0) (unit 1)
+    (in_bom yes) (on_board yes) (dnp no)
+    (property "Reference" "TP1" (at 776.605 78.105 0)
+      (effects (font (size 1.27 1.27)) (justify left))
+    )
+    (property "Value" "GND" (at 776.605 81.28 0)
+      (effects (font (size 1.27 1.27)) (justify left))
+    )
+    (property "Footprint" "TestPoint:TestPoint_THTPad_D2.0mm_Drill1.0mm" (at 783.59 88.265 0)
+      (effects (font (size 1.27 1.27)) hide)
+    )
+    (property "Datasheet" "~" (at 783.59 88.265 0)
+      (effects (font (size 1.27 1.27)) hide)
+    )
+    (pin "1")
+    (instances
+      (project "eth"
+        (path "/25b810b6-8afb-4eb4-8eaf-dfe3b666cbdb"
+          (reference "TP1") (unit 1)
+        )
+      )
+    )
+  )
   (symbol (lib_id "Device:C_Small") (at 520.7 276.225 0) (unit 1)
     (in_bom yes) (on_board yes) (dnp no) (fields_autoplaced)
@@
     )
   )
+  (symbol (lib_id "power:GND") (at 792.48 88.265 0) (unit 1)
+    (in_bom yes) (on_board yes) (dnp no) (fields_autoplaced)
+    (property "Reference" "#PWR0220" (at 792.48 94.615 0)
+      (effects (font (size 1.27 1.27)) hide)
+    )
+    (property "Value" "GND" (at 792.48 93.345 0)
+      (effects (font (size 1.27 1.27)))
+    )
+    (property "Footprint" "" (at 792.48 88.265 0)
+      (effects (font (size 1.27 1.27)) hide)
+    )
+    (property "Datasheet" "" (at 792.48 88.265 0)
+      (effects (font (size 1.27 1.27)) hide)
+    )
+    (pin "1")
+    (instances
+      (project "eth"
+        (path "/25b810b6-8afb-4eb4-8eaf-dfe3b666cbdb"
+          (reference "#PWR0220") (unit 1)
+        )
+      )
+    )
+  )
   (symbol (lib_id "power:GND") (at 612.775 335.28 0) (unit 1)
     (in_bom yes) (on_board yes) (dnp no) (fields_autoplaced)
@@
     )
   )
+  (symbol (lib_id "Connector:TestPoint") (at 792.48 88.265 0) (unit 1)
+    (in_bom yes) (on_board yes) (dnp no)
+    (property "Reference" "TP3" (at 790.575 78.105 0)
+      (effects (font (size 1.27 1.27)) (justify left))
+    )
+    (property "Value" "GND" (at 790.575 81.28 0)
+      (effects (font (size 1.27 1.27)) (justify left))
+    )
+    (property "Footprint" "TestPoint:TestPoint_THTPad_D2.0mm_Drill1.0mm" (at 797.56 88.265 0)
+      (effects (font (size 1.27 1.27)) hide)
+    )
+    (property "Datasheet" "~" (at 797.56 88.265 0)
+      (effects (font (size 1.27 1.27)) hide)
+    )
+    (pin "1")
+    (instances
+      (project "eth"
+        (path "/25b810b6-8afb-4eb4-8eaf-dfe3b666cbdb"
+          (reference "TP3") (unit 1)
+        )
+      )
+    )
+  )
   (symbol (lib_id "power:VCC") (at 381.635 276.86 0) (unit 1)
     (in_bom yes) (on_board yes) (dnp no) (fields_autoplaced)
@@
     )
   )
+  (symbol (lib_id "power:GND") (at 798.83 88.265 0) (unit 1)
+    (in_bom yes) (on_board yes) (dnp no) (fields_autoplaced)
+    (property "Reference" "#PWR0221" (at 798.83 94.615 0)
+      (effects (font (size 1.27 1.27)) hide)
+    )
+    (property "Value" "GND" (at 798.83 93.345 0)
+      (effects (font (size 1.27 1.27)))
+    )
+    (property "Footprint" "" (at 798.83 88.265 0)
+      (effects (font (size 1.27 1.27)) hide)
+    )
+    (property "Datasheet" "" (at 798.83 88.265 0)
+      (effects (font (size 1.27 1.27)) hide)
+    )
+    (pin "1")
+    (instances
+      (project "eth"
+        (path "/25b810b6-8afb-4eb4-8eaf-dfe3b666cbdb"
+          (reference "#PWR0221") (unit 1)
+        )
+      )
+    )
+  )
   (symbol (lib_id "power:VCC") (at 572.135 118.745 0) (unit 1)
     (in_bom yes) (on_board yes) (dnp no) (fields_autoplaced)
@@
         )
       )
+    )
+  )
+  (symbol (lib_id "power:GND") (at 785.495 88.265 0) (unit 1)
+    (in_bom yes) (on_board yes) (dnp no) (fields_autoplaced)
+    (property "Reference" "#PWR0219" (at 785.495 94.615 0)
+      (effects (font (size 1.27 1.27)) hide)
+    )
+    (property "Value" "GND" (at 785.495 93.345 0)
+      (effects (font (size 1.27 1.27)))
+    )
+    (property "Footprint" "" (at 785.495 88.265 0)
+      (effects (font (size 1.27 1.27)) hide)
+    )
+    (property "Datasheet" "" (at 785.495 88.265 0)
+      (effects (font (size 1.27 1.27)) hide)
+    )
+    (pin "1")
+    (instances
+      (project "eth"
+        (path "/25b810b6-8afb-4eb4-8eaf-dfe3b666cbdb"
+          (reference "#PWR0219") (unit 1)
+        )
+      )
