File: boards/eth/eth.kicad_sch (KiCad schematic)
At the start: 80 parts, among them J1 Conn_02x20_Odd_Even, J2 eth-phy-shield-conn, U1 74HC04, U10 74HC74, U11 74HC74, U12 74HC161, U13 74HC157, U15 74HC157, U16 74HC157, U17 74HC157, U18 74HC157, U19 74HC157, U19 74HC4040, U2 74HC21, U20 6116, U21 74HC244, U22 6116, U23 74HC244, U24 74HC273, U25 74HC244, U26 74HC244, U27 74HC244, U28 74HC165, U3 74HC74, U37 74HC04, U4 74HC139, U5 74HC32, U6 74HC08, U7 74HC32, U8 74HC08, U9 74HC04, X1 CB3-3C-20M

Commit message: Eth: doc and errata
Parts:
- U11: value 74HC74 -> 74LV74A
Changed lines of the file:
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@@
       (effects (font (size 1.27 1.27)) (justify left))
     )
-    (property "Value" "74HC74" (at 278.13 540.385 0)
+    (property "Value" "74LV74A" (at 278.13 540.385 0)
       (effects (font (size 1.27 1.27)) (justify left))
     )
@@
       (effects (font (size 1.27 1.27)) (justify left))
     )
-    (property "Value" "74HC74" (at 648.6241 377.19 0)
+    (property "Value" "74LV74A" (at 648.6241 377.19 0)
       (effects (font (size 1.27 1.27)) (justify left))
     )
@@
       (effects (font (size 1.27 1.27)) (justify left))
     )
-    (property "Value" "74HC74" (at 648.6241 342.265 0)
+    (property "Value" "74LV74A" (at 648.6241 342.265 0)
       (effects (font (size 1.27 1.27)) (justify left))
     )
